File: Amazing All-Band Receiver.brd (EAGLE design)
At the start: 38.1 x 20.3 mm, 20 parts, among them T1 BC547, T2 BC547

Commit message: ...
Parts:
- D1: value OA79-10 -> OA79
Changed lines of the file:
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@@
 <element name="C4" library="c" package="C050-025X075" value="10n" x="17.78" y="10.16" rot="R180"/>
 <element name="C5" library="c" package="C050-025X075" value="1n" x="5.08" y="15.24" rot="R270"/>
-<element name="D1" library="d" package="DO34-7V" value="OA79-10" x="27.94" y="8.89"/>
+<element name="D1" library="d" package="DO34-7V" value="OA79" x="27.94" y="8.89"/>
 <element name="EAR+" library="pad" package="SPAD" value="SPAD" x="5.08" y="10.16" rot="R90"/>
 <element name="EAR-" library="pad" package="SPAD" value="SPAD" x="2.54" y="10.16" rot="R90"/>
