File: eagle/FM-Super-Regen.brd (EAGLE design)
At the start: 53.3 x 20.3 mm, 15 parts, among them Q1 BF245B

Commit message: ...
Parts:
- C5, C6: device c:C050-020X036 -> c:C050-020X044
- L1: device l:L-08/10-TAP1 -> l:L-08/10-X-TAP1
- moved ANT 8.03 mm to (2.54, 17.8)
- moved C3 2.54 mm to (25.4, 5.08)
- moved C4 2.54 mm to (25.4, 15.2)
- moved Q1 2.54 mm to (25.4, 12.7)
- moved L1 2.54 mm to (11.4, 15.2)
- moved R1 2.54 mm to (12.7, 5.08)
- moved AOUT+ 2.54 mm to (50.8, 5.08)
- moved C1 2.54 mm to (17.8, 5.08)
- moved C5 2.54 mm to (35.6, 5.08), turned to 0 degrees
- moved C6 2.54 mm to (43.2, 5.08), turned to 180 degrees
- moved L2 2.54 mm to (36.8, 15.2)
- moved R2 2.54 mm to (35.6, 7.62)
Routing:
- net N$3: track 35.6 -> 30.5 mm
- net N$1: track 7.62 -> 5.08 mm
Changed lines of the file:
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@@
 <elements>
 <element name="9V" library="pad" package="SPAD" value="SPAD" x="5.08" y="7.62"/>
-<element name="ANT" library="pad" package="SPAD" value="ANT" x="5.08" y="10.16"/>
-<element name="AOUT+" library="pad" package="SPAD" value="SPAD" x="50.8" y="7.62" rot="R180"/>
+<element name="ANT" library="pad" package="SPAD" value="ANT" x="2.54" y="17.78"/>
+<element name="AOUT+" library="pad" package="SPAD" value="SPAD" x="50.8" y="5.08" rot="R180"/>
 <element name="AOUT-" library="pad" package="SPAD" value="SPAD" x="50.8" y="2.54" rot="R180"/>
-<element name="C1" library="c" package="C050-020X036/V" value="1n" x="20.32" y="5.08" smashed="yes">
-<attribute name="NAME" x="19.304" y="5.08" size="1.016" layer="25" align="center-right"/>
-<attribute name="VALUE" x="20.066" y="1.27" size="1.016" layer="27" align="center-left"/>
+<element name="C1" library="c" package="C050-020X036/V" value="1n" x="17.78" y="5.08" smashed="yes">
+<attribute name="NAME" x="16.764" y="5.08" size="1.016" layer="25" align="center-right"/>
+<attribute name="VALUE" x="17.526" y="1.27" size="1.016" layer="27" align="center-left"/>
 </element>
-<element name="C3" library="cap-trim" package="TRIM-2222-808" value="15p" x="27.94" y="5.08" rot="R270"/>
-<element name="C4" library="c" package="C050-020X036" value="4.7pF" x="27.94" y="15.24"/>
-<element name="C5" library="c" package="C050-020X036" value="4.7n" x="38.1" y="5.08" rot="R180"/>
-<element name="C6" library="c" package="C050-020X036" value="100n" x="45.72" y="5.08"/>
+<element name="C3" library="cap-trim" package="TRIM-2222-808" value="15p" x="25.4" y="5.08" rot="R270"/>
+<element name="C4" library="c" package="C050-020X036" value="4.7pF" x="25.4" y="15.24"/>
+<element name="C5" library="c" package="C050-020X044" value="4.7n" x="35.56" y="5.08"/>
+<element name="C6" library="c" package="C050-020X044" value="100n" x="43.18" y="5.08" rot="R180"/>
 <element name="GND" library="pad" package="SPAD" value="SPAD" x="5.08" y="5.08"/>
-<element name="L2" library="l" package="L-BODY" value="3.3uH" x="39.37" y="15.24"/>
-<element name="Q1" library="t" package="TO92" value="BF245B" x="27.94" y="12.7" rot="R180"/>
-<element name="R1" library="r" package="POT-V" value="1k" x="15.24" y="5.08" rot="R180"/>
-<element name="R2" library="r" package="0204/10" value="10k" x="38.1" y="7.62"/>
-<element name="L1" library="l" package="L-08/10-TAP1" value="0.22uH" x="13.97" y="15.24"/>
+<element name="L2" library="l" package="L-BODY" value="3.3uH" x="36.83" y="15.24"/>
+<element name="Q1" library="t" package="TO92" value="BF245B" x="25.4" y="12.7" rot="R180"/>
+<element name="R1" library="r" package="POT-V" value="1k" x="12.7" y="5.08" rot="R180"/>
+<element name="R2" library="r" package="0204/10" value="10k" x="35.56" y="7.62"/>
+<element name="L1" library="l" package="L-08/10-X-TAP1" value="0.22uH" x="11.43" y="15.24"/>
 </elements>
 <signals>
@@
 <contactref element="AOUT-" pad="1"/>
 <contactref element="GND" pad="1"/>
-<wire x1="30.48" y1="5.08" x2="20.32" y2="5.08" width="0.6096" layer="16"/>
-<wire x1="17.78" y1="7.62" x2="17.78" y2="6.35" width="0.6096" layer="16"/>
-<wire x1="17.78" y1="5.08" x2="5.08" y2="5.08" width="0.6096" layer="16"/>
-<wire x1="30.48" y1="5.08" x2="30.48" y2="7.62" width="0.6096" layer="16"/>
-<wire x1="50.8" y1="2.54" x2="35.56" y2="2.54" width="0.6096" layer="16"/>
-<wire x1="35.56" y1="2.54" x2="35.56" y2="5.08" width="0.6096" layer="16"/>
-<wire x1="33.02" y1="7.62" x2="35.56" y2="7.62" width="0.6096" layer="16"/>
-<wire x1="35.56" y1="7.62" x2="35.56" y2="5.08" width="0.6096" layer="16"/>
-<wire x1="30.48" y1="12.7" x2="30.48" y2="7.62" width="0.6096" layer="16"/>
+<wire x1="27.94" y1="5.08" x2="17.78" y2="5.08" width="0.6096" layer="16"/>
+<wire x1="15.24" y1="7.62" x2="15.24" y2="6.35" width="0.6096" layer="16"/>
+<wire x1="15.24" y1="5.08" x2="5.08" y2="5.08" width="0.6096" layer="16"/>
+<wire x1="27.94" y1="5.08" x2="27.94" y2="7.62" width="0.6096" layer="16"/>
+<wire x1="50.8" y1="2.54" x2="33.02" y2="2.54" width="0.6096" layer="16"/>
+<wire x1="33.02" y1="2.54" x2="33.02" y2="5.08" width="0.6096" layer="16"/>
 <wire x1="30.48" y1="7.62" x2="33.02" y2="7.62" width="0.6096" layer="16"/>
-<wire x1="17.78" y1="7.62" x2="17.78" y2="5.08" width="0.6096" layer="16"/>
-<wire x1="17.78" y1="5.08" x2="20.32" y2="5.08" width="0.6096" layer="16"/>
-<wire x1="20.32" y1="5.08" x2="20.32" y2="7.62" width="0.6096" layer="16"/>
+<wire x1="33.02" y1="7.62" x2="33.02" y2="5.08" width="0.6096" layer="16"/>
+<wire x1="27.94" y1="12.7" x2="27.94" y2="7.62" width="0.6096" layer="16"/>
+<wire x1="27.94" y1="7.62" x2="30.48" y2="7.62" width="0.6096" layer="16"/>
+<wire x1="15.24" y1="7.62" x2="15.24" y2="5.08" width="0.6096" layer="16"/>
+<wire x1="15.24" y1="5.08" x2="17.78" y2="5.08" width="0.6096" layer="16"/>
+<wire x1="17.78" y1="5.08" x2="17.78" y2="7.62" width="0.6096" layer="16"/>
 </signal>
 <signal name="N$2">
@@
 <contactref element="C4" pad="1"/>
 <contactref element="C3" pad="2"/>
-<wire x1="25.4" y1="7.62" x2="25.4" y2="12.7" width="0.6096" layer="16"/>
-<wire x1="25.4" y1="12.7" x2="25.4" y2="15.24" width="0.6096" layer="16"/>
+<wire x1="22.86" y1="7.62" x2="22.86" y2="12.7" width="0.6096" layer="16"/>
+<wire x1="22.86" y1="12.7" x2="22.86" y2="15.24" width="0.6096" layer="16"/>
 <contactref element="L1" pad="2"/>
-<wire x1="20.32" y1="15.24" x2="25.4" y2="15.24" width="0.6096" layer="16"/>
+<wire x1="17.78" y1="15.24" x2="22.86" y2="15.24" width="0.6096" layer="16"/>
 </signal>
 <signal name="N$3">
 <contactref element="C1" pad="1"/>
 <contactref element="R1" pad="S"/>
-<wire x1="20.32" y1="2.54" x2="15.24" y2="2.54" width="0.6096" layer="16"/>
-<wire x1="15.24" y1="2.54" x2="2.54" y2="2.54" width="0.6096" layer="16"/>
+<wire x1="17.78" y1="2.54" x2="12.7" y2="2.54" width="0.6096" layer="16"/>
+<wire x1="12.7" y1="2.54" x2="2.54" y2="2.54" width="0.6096" layer="16"/>
 <contactref element="L1" pad="1"/>
 <wire x1="2.54" y1="2.54" x2="2.54" y2="15.24" width="0.6096" layer="16"/>
-<wire x1="2.54" y1="15.24" x2="7.62" y2="15.24" width="0.6096" layer="16"/>
+<wire x1="2.54" y1="15.24" x2="5.08" y2="15.24" width="0.6096" layer="16"/>
 </signal>
 <signal name="N$4">
 <contactref element="ANT" pad="1"/>
 <contactref element="L1" pad="3"/>
-<wire x1="5.08" y1="10.16" x2="10.16" y2="10.16" width="0.6096" layer="16"/>
+<wire x1="2.54" y1="17.78" x2="7.62" y2="17.78" width="0.6096" layer="16"/>
 </signal>
 <signal name="N$5">
@@
 <contactref element="Q1" pad="2"/>
 <contactref element="L2" pad="3"/>
-<wire x1="27.94" y1="12.7" x2="27.94" y2="15.24" width="0.6096" layer="16"/>
-<wire x1="27.94" y1="15.24" x2="30.48" y2="15.24" width="0.6096" layer="16"/>
-<wire x1="30.48" y1="15.24" x2="35.56" y2="15.24" width="0.6096" layer="16"/>
-<wire x1="35.56" y1="15.24" x2="35.56" y2="12.7" width="0.6096" layer="16"/>
+<wire x1="25.4" y1="12.7" x2="25.4" y2="15.24" width="0.6096" layer="16"/>
+<wire x1="25.4" y1="15.24" x2="27.94" y2="15.24" width="0.6096" layer="16"/>
+<wire x1="27.94" y1="15.24" x2="33.02" y2="15.24" width="0.6096" layer="16"/>
+<wire x1="33.02" y1="15.24" x2="33.02" y2="12.7" width="0.6096" layer="16"/>
 </signal>
 <signal name="N$6">
@@
 <contactref element="C5" pad="1"/>
 <contactref element="C6" pad="1"/>
-<wire x1="43.18" y1="17.78" x2="40.64" y2="17.78" width="0.6096" layer="16"/>
-<wire x1="40.64" y1="17.78" x2="40.64" y2="7.62" width="0.6096" layer="16"/>
-<wire x1="40.64" y1="5.08" x2="40.64" y2="7.62" width="0.6096" layer="16"/>
-<wire x1="40.64" y1="7.62" x2="43.18" y2="7.62" width="0.6096" layer="16"/>
-<wire x1="43.18" y1="5.08" x2="43.18" y2="7.62" width="0.6096" layer="16"/>
+<wire x1="40.64" y1="17.78" x2="38.1" y2="17.78" width="0.6096" layer="16"/>
+<wire x1="38.1" y1="17.78" x2="38.1" y2="7.62" width="0.6096" layer="16"/>
+<wire x1="40.64" y1="5.08" x2="38.1" y2="5.08" width="0.6096" layer="16"/>
+<wire x1="38.1" y1="5.08" x2="38.1" y2="7.62" width="0.6096" layer="16"/>
+<wire x1="38.1" y1="7.62" x2="40.64" y2="7.62" width="0.6096" layer="16"/>
 </signal>
 <signal name="N$8">
 <contactref element="AOUT+" pad="1"/>
 <contactref element="C6" pad="2"/>
-<wire x1="48.26" y1="5.08" x2="48.26" y2="7.62" width="0.6096" layer="16"/>
-<wire x1="48.26" y1="7.62" x2="50.8" y2="7.62" width="0.6096" layer="16"/>
+<wire x1="45.72" y1="5.08" x2="50.8" y2="5.08" width="0.6096" layer="16"/>
 </signal>
 <signal name="N$1">
 <contactref element="9V" pad="1"/>
 <contactref element="R1" pad="E"/>
-<wire x1="5.08" y1="7.62" x2="12.7" y2="7.62" width="0.6096" layer="16"/>
+<wire x1="5.08" y1="7.62" x2="10.16" y2="7.62" width="0.6096" layer="16"/>
 </signal>
 </signals>
