File: eagle/Kosmos-X3000-FM-Superregen.brd (EAGLE design)
At the start: 35.6 x 17.8 mm, 14 parts, among them T1 BF247B

Commit message: ...
Parts:
- added AF: SPAD+-+-, pad:SPAD+-
- BATT: value SPAD+- -> SPAD+-+-
- turned C1 to 180 degrees
- turned C3 to 180 degrees
- turned C4 to 270 degrees
- turned R3 to 90 degrees
- turned T1 to 180 degrees
Connections:
- net GND: now also AF.1, R3.2; no longer R3.1
- net N$4: now also AF.2
- net N$5: now also R3.1; no longer R3.2
Routing:
- net GND: track 30.5 -> 53.3 mm
- net N$4: track 2.54 -> 7.62 mm
Changed lines of the file:
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@@
 </autorouter>
 <elements>
-<element name="C1" library="c" package="C050-020X044" value="5nF" x="12.7" y="7.62"/>
+<element name="C1" library="c" package="C050-020X044" value="5nF" x="12.7" y="7.62" rot="R180"/>
 <element name="C2" library="cap-trim" package="TRIM-2222-808" value="33pF" x="12.7" y="12.7"/>
-<element name="C3" library="c" package="C050-020X044" value="6.8nF" x="22.86" y="5.08"/>
-<element name="C4" library="c" package="C050-020X044" value="100nF" x="27.94" y="5.08" rot="R90"/>
+<element name="C3" library="c" package="C050-020X044" value="6.8nF" x="22.86" y="5.08" rot="R180"/>
+<element name="C4" library="c" package="C050-020X044" value="100nF" x="27.94" y="5.08" rot="R270"/>
 <element name="L1" library="l" package="L-04-5/5V" value="100nH" x="6.35" y="12.7"/>
 <element name="L2" library="l" package="L-04-5/5V" value="73nH" x="26.67" y="12.7"/>
@@
 <element name="R1" library="r" package="0202/7-V" value="150" x="33.02" y="11.43" rot="R180"/>
 <element name="R2" library="r" package="0202/7" value="10k" x="21.59" y="7.62" rot="R90"/>
-<element name="R3" library="r" package="0202/7" value="3.3k" x="13.97" y="5.08" rot="R270"/>
-<element name="T1" library="t" package="TO92" value="BF247B" x="20.32" y="12.7" rot="R90"/>
-<element name="BATT" library="pad" package="SPAD+-" value="SPAD+-" x="33.02" y="3.81"/>
+<element name="R3" library="r" package="0202/7" value="3.3k" x="13.97" y="5.08" rot="R90"/>
+<element name="T1" library="t" package="TO92" value="BF247B" x="20.32" y="12.7" rot="R180"/>
+<element name="BATT" library="pad" package="SPAD+-" value="SPAD+-+-" x="33.02" y="3.81"/>
 <element name="C5" library="c" package="C025-015X024" value="15p" x="2.54" y="8.89" rot="R180"/>
 <element name="ANT" library="pad" package="SPAD" value="ANT" x="2.54" y="15.24"/>
+<element name="AF" library="pad" package="SPAD+-" value="SPAD+-+-" x="30.48" y="3.81"/>
 </elements>
 <signals>
@@
 <signal name="GND">
 <contactref element="L3" pad="1"/>
-<contactref element="R3" pad="1"/>
+<contactref element="R3" pad="2"/>
 <contactref element="C3" pad="2"/>
 <contactref element="C4" pad="2"/>
@@
 <wire x1="20.32" y1="2.54" x2="17.78" y2="2.54" width="0.6096" layer="16"/>
 <wire x1="17.78" y1="2.54" x2="7.62" y2="2.54" width="0.6096" layer="16"/>
-<wire x1="33.02" y1="2.54" x2="27.94" y2="2.54" width="0.6096" layer="16"/>
+<wire x1="33.02" y1="2.54" x2="30.48" y2="2.54" width="0.6096" layer="16"/>
+<wire x1="30.48" y1="2.54" x2="27.94" y2="2.54" width="0.6096" layer="16"/>
 <wire x1="20.32" y1="5.08" x2="20.32" y2="2.54" width="0.6096" layer="16"/>
 <wire x1="20.32" y1="2.54" x2="27.94" y2="2.54" width="0.6096" layer="16"/>
 <wire x1="17.78" y1="5.08" x2="17.78" y2="2.54" width="0.6096" layer="16"/>
+<contactref element="AF" pad="1"/>
+<wire x1="30.48" y1="2.54" x2="7.62" y2="2.54" width="0.6096" layer="16"/>
 </signal>
 <signal name="N$4">
@@
 <contactref element="R2" pad="2"/>
 <wire x1="25.4" y1="5.08" x2="25.4" y2="7.62" width="0.6096" layer="16"/>
+<contactref element="AF" pad="2"/>
+<wire x1="25.4" y1="5.08" x2="30.48" y2="5.08" width="0.6096" layer="16"/>
 </signal>
 <signal name="N$5">
 <contactref element="R2" pad="1"/>
-<contactref element="R3" pad="2"/>
+<contactref element="R3" pad="1"/>
 <contactref element="C1" pad="1"/>
 <contactref element="T1" pad="2"/>
