File: eagle/Simple-Charger-LiIon-OpampBased-LM324.sch (EAGLE design)
At the start: 21 parts, among them IC1 LM324N, T1 BC327

Commit message: ...
Parts:
- R10: device r:R-H0204/10 -> r:R-H0204/2V
- R2: device r:R-H0204/10-V -> r:R-H0204/7-V
- R5: device r:R-H0204/10 -> r:R-H0204/10-V
- R7: device r:R-H0204/10 -> r:R-H0204/7-V
- R8: device r:R0204/10-V -> r:R0204/10
- R9: device r:R0204/7-V -> r:R0204/10-V
Connections:
- net GND: now also IC1A.+IN, IC1A.-IN, IC1B.+IN, IC1B.-IN
Other:
- moved on the sheet: IC1A, IC1B

Commit message: ...
Parts:
- C1: device c:CPOLE2.5-5 -> c:CPOLE2,5-5/V
- R2, R7: device r:R-H0204/7-V -> r:R-H0204/10-V
Changed lines of the file:
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@@
 <part name="IC1" library="ic" deviceset="LM324" device="N"/>
 <part name="R1" library="r" deviceset="R-H" device="0204/10" value="1"/>
-<part name="R2" library="r" deviceset="R-H" device="0204/7-V" value="2.7k"/>
+<part name="R2" library="r" deviceset="R-H" device="0204/10-V" value="2.7k"/>
 <part name="R3" library="r" deviceset="R" device="0204/10-V" value="2.2k"/>
 <part name="R4" library="r" deviceset="R" device="0204/10-V" value="220"/>
 <part name="R5" library="r" deviceset="R-H" device="0204/10-V" value="470"/>
 <part name="R6" library="r" deviceset="R" device="0204/10-V" value="4.7k"/>
-<part name="R7" library="r" deviceset="R-H" device="0204/7-V" value="3.6k"/>
+<part name="R7" library="r" deviceset="R-H" device="0204/10-V" value="3.6k"/>
 <part name="R8" library="r" deviceset="R" device="0204/10" value="680"/>
 <part name="R9" library="r" deviceset="R" device="0204/10-V" value="1k"/>
 <part name="R10" library="r" deviceset="R-H" device="0204/2V" value="680k"/>
-<part name="C1" library="c" deviceset="CPOL" device="E2.5-5" value="100uF/16V"/>
+<part name="C1" library="c" deviceset="CPOL" device="E2,5-5/V" value="100uF/16V"/>
 <part name="C2" library="c" deviceset="C-H" device="050-020X044" value="68nF"/>
 <part name="R11" library="r" deviceset="R" device="0204/10-V" value="470"/>

Commit message: ...
Parts:
- C2: device c:C-H050-020X044 -> c:C-H050-020X044/V
- LI-ION: value SPAD+-+- -> (none)
- R1: device r:R-H0204/10 -> r:R-H0204/10-V
- R4: device r:R0204/10-V -> r:R0204/10
- R5: device r:R-H0204/10-V -> r:R-H0204/10
- USB: value SPAD+--+ -> (none)
Connections:
- net N$11: now also T1.E; no longer T1.C
- net V+: now also T1.C; no longer T1.E
Other:
- moved on the sheet: IC1A, IC1B, IC1D, LI-ION+, LI-ION-, R1, R11, R2, R3, R4, R6, T1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
