File: eagle/VCO-555-Thomas-Henry.brd (EAGLE design)
At the start: 160 x 100 mm, 86 parts, among them IC1 TL074P, IC2 TL074P, IC3 LM13700N, IC4 NE555N, T1 BC847, U1 BC857BS-7-F

Commit message: ...
Parts:
- removed U1: BC857BS-7-F, Diodes_Inc_By_element14_Batch_1:SOT65P210X100-6N
- added T2, T3: 2N3904, t:TO92
- C1, C2, C3, C4, C5, C6: device resistor:C0805K -> c:C050-020X044
- R46, R51, R52: device resistor:0207/10 -> r:0204/10
- R7, R8: device resistor:R1206 -> r:0204/10
- moved X7 244.7 mm to (162.6, 86.4)
- moved X8 237.8 mm to (152.4, 58.4)
- moved R44 237.5 mm to (154.9, 88.9)
- moved R49 221.5 mm to (149.9, 61.0)
- moved R43 217.7 mm to (147.3, 99.1)
- moved R50 213.3 mm to (129.5, 66.0)
- moved R37 212.3 mm to (129.5, 88.9)
- moved X5 210.9 mm to (144.8, 40.6)
- moved R48 206.0 mm to (147.3, 63.5)
- moved R41 201.9 mm to (144.8, 81.3)
- moved R42 201.8 mm to (144.8, 76.2)
- moved R28 200.5 mm to (127.0, 35.6)
- moved IC2 196.0 mm to (128.3, 52.1), turned to 90 degrees
- moved IC4 195.4 mm to (111.8, 45.7)
- moved R27 195.3 mm to (132.1, 25.4)
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Connections:
- removed net N$3: R12.1, R13.2, U1.6
- new net N$57: R12.1, R13.2, T3.3
- net GND: now also T3.2; no longer U1.2
- net N$20: now also T2.2; no longer U1.5
- net N$21: now also T2.1, T3.1; no longer U1.1, U1.4
- net N$4: now also T2.3; no longer U1.3

Commit message: ...
Parts:
- R22, R40, R44: device resistor:0207/10 -> r:0204/10
- T1: value BC847 -> 2N3904; device transistor:SOT23 -> t:TO92
- moved T1 10.8 mm to (101.6, 7.62)
Connections:
- net GND: now also T1.1; no longer T1.2
- net N$40: now also T1.2; no longer T1.1
Changed lines of the file:
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@@
 <element name="R20" library="resistor" package="0207/10" value="20k" x="81.28" y="55.88"/>
 <element name="R21" library="resistor" package="0207/10" value="20k" x="91.44" y="58.42"/>
-<element name="R22" library="resistor" package="0207/10" value="2k" x="96.52" y="71.12"/>
+<element name="R22" library="r" package="0204/10" value="2k" x="96.52" y="71.12"/>
 <element name="R23" library="resistor" package="0207/10" value="2k" x="99.06" y="68.58"/>
 <element name="R24" library="resistor" package="0207/10" value="10k" x="81.28" y="60.96"/>
@@
 <element name="R39" library="resistor" package="0207/10" value="100k" x="132.08" y="93.98"/>
 <element name="R4" library="resistor" package="0207/10" value="100k" x="10.16" y="45.72"/>
-<element name="R40" library="resistor" package="0207/10" value="39k" x="139.7" y="96.52"/>
+<element name="R40" library="r" package="0204/10" value="39k" x="139.7" y="96.52"/>
 <element name="R41" library="resistor" package="0207/10" value="39k" x="144.78" y="81.28"/>
 <element name="R42" library="resistor" package="RTRIM3296W" value="25k" x="144.78" y="76.2"/>
 <element name="R43" library="resistor" package="0207/10" value="300k" x="147.32" y="99.06"/>
-<element name="R44" library="resistor" package="0207/10" value="5.6k" x="154.94" y="88.9"/>
+<element name="R44" library="r" package="0204/10" value="5.6k" x="154.94" y="88.9"/>
 <element name="R45" library="resistor" package="0207/10" value="1k" x="157.48" y="91.44"/>
 <element name="R46" library="r" package="0204/10" value="2.2k" x="134.62" y="71.12"/>
@@
 <attribute name="MPN" value="" x="30.48" y="5.08" size="1.778" layer="27" display="off"/>
 </element>
-<element name="T1" library="transistor" package="SOT23" value="BC847" x="93.98" y="15.24"/>
+<element name="T1" library="t" package="TO92" value="2N3904" x="101.6" y="7.62"/>
 <element name="U$1" library="gm-caps-electro-pol" package="063_025" value="47uF" x="20.32" y="7.62"/>
 <element name="U$2" library="gm-caps-electro-pol" package="063_025" value="47uF" x="20.32" y="2.54"/>
@@
 <contactref element="X5" pad="2"/>
 <contactref element="IC2" pad="5"/>
-<contactref element="T1" pad="2"/>
+<contactref element="T1" pad="1"/>
 <contactref element="D2" pad="A"/>
 <contactref element="X6" pad="2"/>
@@
 <wire x1="80.01" y1="10.16" x2="55.88" y2="11.43" width="0" layer="19" extent="1-1"/>
 <wire x1="92.71" y1="12.7" x2="80.01" y2="10.16" width="0" layer="19" extent="1-1"/>
-<wire x1="94.93" y1="14.14" x2="92.71" y2="12.7" width="0" layer="19" extent="1-1"/>
+<wire x1="101.6" y1="10.16" x2="92.71" y2="12.7" width="0" layer="19" extent="1-1"/>
 <wire x1="82.55" y1="25.4" x2="80.01" y2="10.16" width="0" layer="19" extent="1-1"/>
 <wire x1="6.35" y1="55.88" x2="6.35" y2="22.86" width="0" layer="19" extent="1-1"/>
@@
 <contactref element="IC4" pad="4"/>
 <wire x1="99.06" y1="20.32" x2="115.57" y2="41.91" width="0" layer="19" extent="1-1"/>
-<wire x1="93.98" y1="16.34" x2="99.06" y2="20.32" width="0" layer="19" extent="1-1"/>
+<wire x1="101.6" y1="5.08" x2="99.06" y2="20.32" width="0" layer="19" extent="1-1"/>
 </signal>
 <signal name="N$40">
-<contactref element="T1" pad="1"/>
+<contactref element="T1" pad="2"/>
 <contactref element="D2" pad="C"/>
 <contactref element="R35" pad="2"/>
-<wire x1="93.03" y1="14.14" x2="91.44" y2="15.24" width="0" layer="19" extent="1-1"/>
+<wire x1="101.6" y1="7.62" x2="91.44" y2="15.24" width="0" layer="19" extent="1-1"/>
 <wire x1="85.09" y1="12.7" x2="91.44" y2="15.24" width="0" layer="19" extent="1-1"/>
 </signal>
