File: eagle/OpAmp-Inverting-3Transistor.sch (EAGLE design)
At the start: 19 parts, among them IC1 LM324

Commit message: ...
Parts:
- removed AUDIO_IN+: AUDIO_IN, pad:SPAD
- removed AUDIO_IN-, AUDIO_OUT-: SPAD, pad:SPAD
- removed AUDIO_OUT+: AUDIO_OUT, pad:SPAD
- removed C1: 100nF, c:C050-024X044
- removed C4: 1uF, c:CPOLE2,5-3
- removed CV_IN: CV_IN, pad:SPAD
- removed IC1: LM324, ic:LM324N
- removed R7: 1k, r:R0202/7
- removed R8: 100k, r:POT-P5
- removed _R5: 100k, r:R0202/7
- added IN, OUT: SPAD+-, pad:SPAD+-
- added R5: 4.7k, r:R0204/10
- added T1, T2: 2N3904, t:2N3904
- added T3: 2N3906, t:2N3906
- C2: value 100nF -> 33nF; device c:C050-024X044 -> c:C050-020X044
- C3: value 1uF -> 3.3uF; device c:CPOLE2,5-3 -> c:CPOLE2,5-4
- D1: value 1N4148 -> 1N4728; device d:1N414834-7 -> d:Z-DIODE34Z5V
- R1: value 470k -> 100k; device r:R0202/7 -> r:R-H0204/10
- R2: value 100k -> 1M; device r:R0202V -> r:R-H0204/10
- R3: value 10k -> 75k; device r:POT-P5 -> r:R-H0204/10
- R4: value 100k -> 7.5k; device r:R0202V -> r:R0204/10
- R6: device r:R0202/10 -> r:R0204/10
Connections:
- removed net N$10: C4.-, R1.1
- removed net VCC: IC1P.V+, R4.1, R8.E
- new net 9V: R4.2, R5.2, R6.2, T3.E
- net GND: now also D1.A, IN-.P$1, OUT-.P$1, T2.E; no longer AUDIO_IN-.P$1, AUDIO_OUT-.P$1, D1.C, IC1P.V-, R8.A, _R5.1
- net N$1: now also D1.C, R5.1, T1.E; no longer AUDIO_IN+.P$1, C4.+
- net N$2: now also R3.1, R4.1, T1.C; no longer C1.1, IC1A.-IN, R1.2, R2.1
- net N$3: now also T2.B, T3.C; no longer C2.2, R3.E
- net N$4: now also C2.2, IN+.P$1; no longer C3.+, IC1A.OUT, R2.2, R3.S
- net N$5: now also C2.1, R1.1; no longer R6.2, R8.S
- net N$6: now also R1.2, R2.1, T1.B; no longer AUDIO_OUT+.P$1, C3.-
- net N$7: now also R3.2, T3.B; no longer IC1A.+IN, R4.2, _R5.2
- net N$8: now also C3.+, R2.2, R6.1, T2.C; no longer CV_IN.P$1, R7.2
- net N$9: now also C3.-, OUT+.P$1; no longer C1.2, C2.1, D1.A, R6.1, R7.1
Other:
- moved on the sheet: R1, R2, R4, R6

Commit message: ...
Parts:
- IN, OUT: value SPAD+- -> SPAD+-+-; device pad:SPAD+- -> pad:SPAD+-+-
- R3: device r:R-H0204/10 -> r:R-H0204/10-V
- R4, R5, R6: device r:R0204/10 -> r:R0204/10-V
- T1: device t:2N3904 -> t:2SC9014
- T2: device t:2N3904 -> t:2N3904EBC
- T3: device t:2N3906 -> t:2SC9015-TO92-EBC
Connections:
- net 9V: now also R4.1, R5.1, R6.1; no longer R4.2, R5.2, R6.2
- net N$1: now also R5.2; no longer R5.1
- net N$2: now also R4.2; no longer R4.1
- net N$8: now also R6.2; no longer R6.1
Other:
- moved on the sheet: T2

Commit message: ...
Parts:
- added J1: (no value), pad:VCC_GNDPWR-R
- D1: value 1N4728 -> Z=3.3V
- IN: value SPAD+-+- -> SPAD+--+; device pad:SPAD+-+- -> pad:SPAD+--+
- T1: value 2N3904 -> BC547; device t:2SC9014 -> t:BC547CBE
- T2: value 2N3904 -> BC547; device t:2N3904EBC -> t:BC547CBE
- T3: value 2N3906 -> BC557; device t:2SC9015-TO92-EBC -> t:BC557CBE
Connections:
- removed net 9V: R4.1, R5.1, R6.1, T3.E
- new net VCC: J1G$1.VCC, R4.1, R5.1, R6.1, T3.E
- net GND: now also J1G$2.GND
Changed lines of the file:
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@@
 </classes>
 <parts>
-<part name="T1" library="t" deviceset="2SC9014" device="" value="2N3904"/>
-<part name="T2" library="t" deviceset="2N3904" device="EBC" value="2N3904"/>
-<part name="T3" library="t" deviceset="2SC9015" device="-TO92-EBC" value="2N3906"/>
+<part name="T1" library="t" deviceset="BC547" device="CBE" value="BC547"/>
+<part name="T2" library="t" deviceset="BC547" device="CBE" value="BC547"/>
+<part name="T3" library="t" deviceset="BC557" device="CBE" value="BC557"/>
 <part name="R1" library="r" deviceset="R-H" device="0204/10" value="100k"/>
 <part name="R2" library="r" deviceset="R-H" device="0204/10" value="1M"/>
@@
 <part name="R5" library="r" deviceset="R" device="0204/10-V" value="4.7k"/>
 <part name="R6" library="r" deviceset="R" device="0204/10-V" value="1k"/>
-<part name="D1" library="d" deviceset="Z-DIODE" device="34Z5V" value="1N4728"/>
-<part name="U$2" library="pad" deviceset="V+" device="" value="9V"/>
-<part name="S1" library="pad" deviceset="GND" device=""/>
+<part name="D1" library="d" deviceset="Z-DIODE" device="34Z5V" value="Z=3.3V"/>
 <part name="C2" library="c" deviceset="C" device="050-020X044" value="33nF"/>
-<part name="IN" library="pad" deviceset="SPAD+-" device="+-"/>
+<part name="IN" library="pad" deviceset="SPAD+-" device="-+" value="SPAD+--+"/>
 <part name="OUT" library="pad" deviceset="SPAD+-" device="+-"/>
 <part name="C3" library="c" deviceset="CPOL" device="E2,5-4" value="3.3uF"/>
 <part name="S2" library="pad" deviceset="GND" device=""/>
 <part name="S3" library="pad" deviceset="GND" device=""/>
+<part name="J1" library="pad" deviceset="VCC_GND" device="PWR-R"/>
 </parts>
 <sheets>
@@
 <instance part="R6" gate="G$1" x="58.42" y="45.72"/>
 <instance part="D1" gate="G$1" x="27.94" y="17.78"/>
-<instance part="U$2" gate="G$1" x="38.1" y="55.88"/>
-<instance part="S1" gate="1" x="27.94" y="7.62"/>
 <instance part="C2" gate="1" x="-7.62" y="30.48" smashed="yes" rot="R270">
 <attribute name="NAME" x="-7.62" y="33.02" size="1.27" layer="95" align="bottom-center"/>
@@
 <instance part="S2" gate="1" x="-10.16" y="15.24"/>
 <instance part="S3" gate="1" x="71.12" y="22.86"/>
+<instance part="J1" gate="G$1" x="38.1" y="55.88"/>
+<instance part="J1" gate="G$2" x="27.94" y="10.16"/>
 </instances>
 <busses>
@@
 <nets>
 <net name="GND" class="0">
-<segment>
-<pinref part="D1" gate="G$1" pin="A"/>
-<wire x1="27.94" y1="12.7" x2="27.94" y2="15.24" width="0.1524" layer="91"/>
-<pinref part="S1" gate="1" pin="GND"/>
-<wire x1="27.94" y1="12.7" x2="27.94" y2="10.16" width="0.1524" layer="91"/>
-<junction x="27.94" y="12.7"/>
-<pinref part="T2" gate="G$1" pin="E"/>
-<wire x1="58.42" y1="22.86" x2="58.42" y2="12.7" width="0.1524" layer="91"/>
-<wire x1="58.42" y1="12.7" x2="27.94" y2="12.7" width="0.1524" layer="91"/>
-</segment>
 <segment>
 <pinref part="IN" gate="-" pin="P$1"/>
@@
 <wire x1="76.2" y1="30.48" x2="71.12" y2="30.48" width="0.1524" layer="91"/>
 <wire x1="71.12" y1="30.48" x2="71.12" y2="25.4" width="0.1524" layer="91"/>
+</segment>
+<segment>
+<pinref part="D1" gate="G$1" pin="A"/>
+<wire x1="27.94" y1="12.7" x2="27.94" y2="15.24" width="0.1524" layer="91"/>
+<wire x1="27.94" y1="12.7" x2="27.94" y2="10.16" width="0.1524" layer="91"/>
+<junction x="27.94" y="12.7"/>
+<pinref part="T2" gate="G$1" pin="E"/>
+<wire x1="58.42" y1="22.86" x2="58.42" y2="12.7" width="0.1524" layer="91"/>
+<wire x1="58.42" y1="12.7" x2="27.94" y2="12.7" width="0.1524" layer="91"/>
+<pinref part="J1" gate="G$2" pin="GND"/>
 </segment>
 </net>
@@
 </segment>
 </net>
-<net name="9V" class="0">
+<net name="VCC" class="0">
 <segment>
 <wire x1="17.78" y1="53.34" x2="27.94" y2="53.34" width="0.1524" layer="91"/>
@@
 <wire x1="48.26" y1="43.18" x2="48.26" y2="53.34" width="0.1524" layer="91"/>
 <junction x="48.26" y="53.34"/>
-<pinref part="U$2" gate="G$1" pin="+12V"/>
 <wire x1="38.1" y1="55.88" x2="38.1" y2="53.34" width="0.1524" layer="91"/>
 <junction x="38.1" y="53.34"/>
@@
 <pinref part="R6" gate="G$1" pin="1"/>
 <wire x1="58.42" y1="50.8" x2="58.42" y2="53.34" width="0.1524" layer="91"/>
+<pinref part="J1" gate="G$1" pin="VCC"/>
 </segment>
 </net>

Commit message: ...
Parts:
- C3: device c:CPOLE2,5-4 -> c:CPOLE2,5-4/V
- D1: device d:Z-DIODE34Z5V -> d:Z-DIODE34Z2,5
- R1: device r:R-H0204/10 -> r:R-H0202/10-V
- R2: device r:R-H0204/10 -> r:R-H0202/10
- R3: device r:R-H0204/10-V -> r:R-H0202/7
- R4, R5: device r:R0204/10-V -> r:R0202/7
- R6: device r:R0204/10-V -> r:R0202/10-V
Changed lines of the file:
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@@
 <part name="T2" library="t" deviceset="BC547" device="CBE" value="BC547"/>
 <part name="T3" library="t" deviceset="BC557" device="CBE" value="BC557"/>
-<part name="R1" library="r" deviceset="R-H" device="0204/10" value="100k"/>
-<part name="R2" library="r" deviceset="R-H" device="0204/10" value="1M"/>
-<part name="R3" library="r" deviceset="R-H" device="0204/10-V" value="75k"/>
-<part name="R4" library="r" deviceset="R" device="0204/10-V" value="7.5k"/>
-<part name="R5" library="r" deviceset="R" device="0204/10-V" value="4.7k"/>
-<part name="R6" library="r" deviceset="R" device="0204/10-V" value="1k"/>
-<part name="D1" library="d" deviceset="Z-DIODE" device="34Z5V" value="Z=3.3V"/>
+<part name="R1" library="r" deviceset="R-H" device="0202/10-V" value="100k"/>
+<part name="R2" library="r" deviceset="R-H" device="0202/10" value="1M"/>
+<part name="R3" library="r" deviceset="R-H" device="0202/7" value="75k"/>
+<part name="R4" library="r" deviceset="R" device="0202/7" value="7.5k"/>
+<part name="R5" library="r" deviceset="R" device="0202/7" value="4.7k"/>
+<part name="R6" library="r" deviceset="R" device="0202/10-V" value="1k"/>
+<part name="D1" library="d" deviceset="Z-DIODE" device="34Z2,5" value="Z=3.3V"/>
 <part name="C2" library="c" deviceset="C" device="050-020X044" value="33nF"/>
 <part name="IN" library="pad" deviceset="SPAD+-" device="-+" value="SPAD+--+"/>
 <part name="OUT" library="pad" deviceset="SPAD+-" device="+-"/>
-<part name="C3" library="c" deviceset="CPOL" device="E2,5-4" value="3.3uF"/>
+<part name="C3" library="c" deviceset="CPOL" device="E2,5-4/V" value="3.3uF"/>
 <part name="S2" library="pad" deviceset="GND" device=""/>
 <part name="S3" library="pad" deviceset="GND" device=""/>

Commit message: ...
Parts:
- R3: device r:R-H0202/7 -> r:R-H0202/10
- R4, R5: device r:R0202/7 -> r:R0202/10
- R6: device r:R0202/10-V -> r:R0202/7-V
Changed lines of the file:
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@@
 <grid distance="0.05" unitdist="inch" unit="inch" style="lines" multiple="2" display="yes" altdistance="0.025" altunitdist="inch" altunit="inch"/>
 <layers>
-<layer number="1" name="Top" color="4" fill="1" visible="no" active="no"/>
-<layer number="2" name="Route2" color="1" fill="3" visible="no" active="no"/>
-<layer number="3" name="Route3" color="4" fill="3" visible="no" active="no"/>
-<layer number="4" name="Route4" color="1" fill="4" visible="no" active="no"/>
-<layer number="5" name="Route5" color="4" fill="4" visible="no" active="no"/>
-<layer number="6" name="Route6" color="1" fill="8" visible="no" active="no"/>
-<layer number="7" name="Route7" color="4" fill="8" visible="no" active="no"/>
-<layer number="8" name="Route8" color="1" fill="2" visible="no" active="no"/>
-<layer number="9" name="Route9" color="4" fill="2" visible="no" active="no"/>
-<layer number="10" name="Route10" color="1" fill="7" visible="no" active="no"/>
-<layer number="11" name="Route11" color="4" fill="7" visible="no" active="no"/>
-<layer number="12" name="Route12" color="1" fill="5" visible="no" active="no"/>
-<layer number="13" name="Route13" color="4" fill="5" visible="no" active="no"/>
-<layer number="14" name="Route14" color="1" fill="6" visible="no" active="no"/>
-<layer number="15" name="Route15" color="4" fill="6" visible="no" active="no"/>
-<layer number="16" name="Bottom" color="1" fill="1" visible="no" active="no"/>
-<layer number="17" name="Pads" color="2" fill="1" visible="no" active="no"/>
-<layer number="18" name="Vias" color="2" fill="1" visible="no" active="no"/>
-<layer number="19" name="Unrouted" color="6" fill="1" visible="no" active="no"/>
-<layer number="20" name="Dimension" color="15" fill="1" visible="no" active="no"/>
-<layer number="21" name="tPlace" color="7" fill="1" visible="no" active="no"/>
-<layer number="22" name="bPlace" color="7" fill="1" visible="no" active="no"/>
-<layer number="23" name="tOrigins" color="15" fill="1" visible="no" active="no"/>
-<layer number="24" name="bOrigins" color="15" fill="1" visible="no" active="no"/>
-<layer number="25" name="tNames" color="7" fill="1" visible="no" active="no"/>
-<layer number="26" name="bNames" color="7" fill="1" visible="no" active="no"/>
-<layer number="27" name="tValues" color="7" fill="1" visible="no" active="no"/>
-<layer number="28" name="bValues" color="7" fill="1" visible="no" active="no"/>
+<layer number="1" name="Top" color="4" fill="1" visible="yes" active="no"/>
+<layer number="2" name="Route2" color="1" fill="3" visible="yes" active="no"/>
+<layer number="3" name="Route3" color="4" fill="3" visible="yes" active="no"/>
+<layer number="4" name="Route4" color="1" fill="4" visible="yes" active="no"/>
+<layer number="5" name="Route5" color="4" fill="4" visible="yes" active="no"/>
+<layer number="6" name="Route6" color="1" fill="8" visible="yes" active="no"/>
+<layer number="7" name="Route7" color="4" fill="8" visible="yes" active="no"/>
+<layer number="8" name="Route8" color="1" fill="2" visible="yes" active="no"/>
+<layer number="9" name="Route9" color="4" fill="2" visible="yes" active="no"/>
+<layer number="10" name="Route10" color="1" fill="7" visible="yes" active="no"/>
+<layer number="11" name="Route11" color="4" fill="7" visible="yes" active="no"/>
+<layer number="12" name="Route12" color="1" fill="5" visible="yes" active="no"/>
+<layer number="13" name="Route13" color="4" fill="5" visible="yes" active="no"/>
+<layer number="14" name="Route14" color="1" fill="6" visible="yes" active="no"/>
+<layer number="15" name="Route15" color="4" fill="6" visible="yes" active="no"/>
+<layer number="16" name="Bottom" color="1" fill="1" visible="yes" active="no"/>
+<layer number="17" name="Pads" color="2" fill="1" visible="yes" active="no"/>
+<layer number="18" name="Vias" color="2" fill="1" visible="yes" active="no"/>
+<layer number="19" name="Unrouted" color="6" fill="1" visible="yes" active="no"/>
+<layer number="20" name="Dimension" color="15" fill="1" visible="yes" active="no"/>
+<layer number="21" name="tPlace" color="7" fill="1" visible="yes" active="no"/>
+<layer number="22" name="bPlace" color="7" fill="1" visible="yes" active="no"/>
+<layer number="23" name="tOrigins" color="15" fill="1" visible="yes" active="no"/>
+<layer number="24" name="bOrigins" color="15" fill="1" visible="yes" active="no"/>
+<layer number="25" name="tNames" color="7" fill="1" visible="yes" active="no"/>
+<layer number="26" name="bNames" color="7" fill="1" visible="yes" active="no"/>
+<layer number="27" name="tValues" color="7" fill="1" visible="yes" active="no"/>
+<layer number="28" name="bValues" color="7" fill="1" visible="yes" active="no"/>
 <layer number="29" name="tStop" color="7" fill="3" visible="no" active="no"/>
 <layer number="30" name="bStop" color="7" fill="6" visible="no" active="no"/>
@@
 <layer number="35" name="tGlue" color="7" fill="4" visible="no" active="no"/>
 <layer number="36" name="bGlue" color="7" fill="5" visible="no" active="no"/>
-<layer number="37" name="tTest" color="7" fill="1" visible="no" active="no"/>
-<layer number="38" name="bTest" color="7" fill="1" visible="no" active="no"/>
+<layer number="37" name="tTest" color="7" fill="1" visible="yes" active="no"/>
+<layer number="38" name="bTest" color="7" fill="1" visible="yes" active="no"/>
 <layer number="39" name="tKeepout" color="4" fill="11" visible="no" active="no"/>
 <layer number="40" name="bKeepout" color="1" fill="11" visible="no" active="no"/>
@@
 <layer number="44" name="Drills" color="7" fill="1" visible="no" active="no"/>
 <layer number="45" name="Holes" color="7" fill="1" visible="no" active="no"/>
-<layer number="46" name="Milling" color="3" fill="1" visible="no" active="no"/>
-<layer number="47" name="Measures" color="7" fill="1" visible="no" active="no"/>
-<layer number="48" name="Document" color="7" fill="1" visible="no" active="no"/>
-<layer number="49" name="Reference" color="7" fill="1" visible="no" active="no"/>
-<layer number="51" name="tDocu" color="7" fill="1" visible="no" active="no"/>
-<layer number="52" name="bDocu" color="7" fill="1" visible="no" active="no"/>
+<layer number="46" name="Milling" color="3" fill="1" visible="yes" active="no"/>
+<layer number="47" name="Measures" color="7" fill="1" visible="yes" active="no"/>
+<layer number="48" name="Document" color="7" fill="1" visible="yes" active="no"/>
+<layer number="49" name="Reference" color="7" fill="1" visible="yes" active="no"/>
+<layer number="51" name="tDocu" color="7" fill="1" visible="yes" active="no"/>
+<layer number="52" name="bDocu" color="7" fill="1" visible="yes" active="no"/>
 <layer number="90" name="Modules" color="5" fill="1" visible="yes" active="yes"/>
 <layer number="91" name="Nets" color="2" fill="1" visible="yes" active="yes"/>
@@
 <part name="R1" library="r" deviceset="R-H" device="0202/10-V" value="100k"/>
 <part name="R2" library="r" deviceset="R-H" device="0202/10" value="1M"/>
-<part name="R3" library="r" deviceset="R-H" device="0202/7" value="75k"/>
-<part name="R4" library="r" deviceset="R" device="0202/7" value="7.5k"/>
-<part name="R5" library="r" deviceset="R" device="0202/7" value="4.7k"/>
-<part name="R6" library="r" deviceset="R" device="0202/10-V" value="1k"/>
+<part name="R3" library="r" deviceset="R-H" device="0202/10" value="75k"/>
+<part name="R4" library="r" deviceset="R" device="0202/10" value="7.5k"/>
+<part name="R5" library="r" deviceset="R" device="0202/10" value="4.7k"/>
+<part name="R6" library="r" deviceset="R" device="0202/7-V" value="1k"/>
 <part name="D1" library="d" deviceset="Z-DIODE" device="34Z2,5" value="Z=3.3V"/>
 <part name="C2" library="c" deviceset="C" device="050-020X044" value="33nF"/>
