File: eagle/Handclap-TR808.brd (EAGLE design)
At the start: 134.6 x 124.5 mm, 83 parts, among them IC2 BA6110, IC4 LM339N, IC5 TL072P, T1 2N3904, T2 2N3904, T3 2N3904, T4 2N3906, T5 2N3906, T6 2N3906, T7 2N3904

Commit message: ...
Parts:
- moved R25 3.59 mm to (44.5, 45.7)
Changed lines of the file:
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@@
 <element name="R23" library="r" package="0204/10-V" value="10K" x="30.48" y="88.9" rot="R180"/>
 <element name="R24" library="r" package="0204/10-V" value="10K" x="48.26" y="76.2" rot="R180"/>
-<element name="R25" library="r" package="0204/10-V" value="15K" x="46.99" y="43.18" rot="R270"/>
+<element name="R25" library="r" package="0204/10-V" value="15K" x="44.45" y="45.72" rot="R270"/>
 <element name="R26" library="r" package="0204/10" value="150K" x="88.9" y="53.34" rot="R90"/>
 <element name="R27" library="r" package="0204/10-V" value="330" x="55.88" y="43.18" rot="R180"/>
@@
 <contactref element="T6" pad="1"/>
 <contactref element="T4" pad="1"/>
-<wire x1="41.91" y1="43.18" x2="66.04" y2="50.8" width="0" layer="19" extent="1-1"/>
-<wire x1="40.64" y1="50.8" x2="41.91" y2="43.18" width="0" layer="19" extent="1-1"/>
+<wire x1="39.37" y1="45.72" x2="66.04" y2="50.8" width="0" layer="19" extent="1-1"/>
+<wire x1="40.64" y1="50.8" x2="39.37" y2="45.72" width="0" layer="19" extent="1-1"/>
 </signal>
 <signal name="N$69">
@@
 <contactref element="T7" pad="3"/>
 <contactref element="PWR1" pad="VCC"/>
-<wire x1="52.07" y1="43.18" x2="104.14" y2="50.8" width="0" layer="19" extent="1-1"/>
-<wire x1="48.26" y1="71.12" x2="52.07" y2="43.18" width="0" layer="19" extent="1-1"/>
+<wire x1="49.53" y1="45.72" x2="104.14" y2="50.8" width="0" layer="19" extent="1-1"/>
+<wire x1="48.26" y1="71.12" x2="49.53" y2="45.72" width="0" layer="19" extent="1-1"/>
 <wire x1="25.4" y1="68.58" x2="48.26" y2="71.12" width="0" layer="19" extent="1-1"/>
 <wire x1="6.35" y1="68.58" x2="25.4" y2="68.58" width="0" layer="19" extent="1-1"/>
