File: eagle/VCF-LM324-Stereo+LFO-POT2x3.brd (EAGLE design)
At the start: 55.9 x 61 mm, 50 parts, among them IC1 LM324, J1 CONN-3P-3P, J2 CONN-3P-3P, J3 CONN-2P2P/H

Commit message: ...
Parts:
- D1: device d:DO34-5 -> d:DO34-7V
- D2: device d:DO34-7V -> d:DO35-2_54
- R10: device r:0204/10 -> r:0204/7
- R14: device r:0204/7-V -> r:0204V
- R16: device r:0204/7 -> r:0204/10
- R19: device r:0204/7-V -> r:0204/10-V
- R2: device r:0204/10-V -> r:0204V
- R3, R9: device r:0204/7-V -> r:0204/7
- moved RIGHT_OUT 23.9 mm to (30.5, 58.4)
- moved CV_IN 17.0 mm to (27.9, 33.0)
- moved D2 14.5 mm to (39.4, 38.1), turned to 180 degrees
- moved R9 13.1 mm to (31.8, 38.1)
- moved TRI 13.0 mm to (20.3, 5.08)
- moved R3 11.5 mm to (19.1, 33.0), turned to 0 degrees
- moved C7 11.4 mm to (38.1, 47.0)
- moved R23 10.2 mm to (22.9, 10.2), turned to 90 degrees
- moved R2 8.89 mm to (15.2, 36.8), turned to 90 degrees
- moved R7 7.41 mm to (19.1, 30.5), turned to 90 degrees
- moved J3 7.18 mm to (7.62, 7.62), turned to 180 degrees
- moved R10 6.35 mm to (34.3, 33.0)
- moved C1 5.68 mm to (10.2, 30.5), turned to 90 degrees
- moved +5V 5.68 mm to (50.8, 33.0)
- moved D1 5.24 mm to (7.62, 29.2)
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Routing:
- net N$5: track 72.5 -> 48.3 mm, vias 2 -> 0
- net RIGHT_OUT: track 37.9 -> 22.9 mm
- net GND: track 191.2 -> 176.5 mm, vias 3 -> 6
- net N$4: track 41.7 -> 53.3 mm
- net N$8: track 18.1 -> 7.62 mm, vias 1 -> 0
- net N$3: track 0.00 -> 10.2 mm
- net LEFT_IN: track 3.81 -> 11.4 mm
- net TRIM_1_A: track 5.08 -> 11.4 mm
- net N$16: track 23.9 -> 29.2 mm
- net TRIM_1_B: track 2.54 -> 7.62 mm
- net TRIM_2_A: track 5.08 -> 10.2 mm
- net LEFT_OUT: track 5.08 -> 10.2 mm
- net N$11: track 48.0 -> 43.3 mm
- net N$12: track 66.9 -> 71.2 mm, vias 3 -> 2
- net N$9: track 19.4 -> 15.2 mm
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Other:
- board text removed: "Cutoff"
- board text removed: "RES"

Commit message: ...
Parts:
- removed LEFT_IN, RIGHT_IN: AUDIO_IN, pad:SPAD
- removed LEFT_OUT, RIGHT_OUT: AUDIO_OUT, pad:SPAD
- added L_IN, R_IN: AUDIO_IN, pad:SPAD
- added L_OUT, R_OUT: AUDIO_OUT, pad:SPAD
- C1, C2: value 100nF -> 0.1uF; device c:C050-024X044 -> c:C050-020X044
- C3, C7: device c:E2,5-3 -> c:E2,5-3/V
- C5, C6: device c:C050-024X044 -> c:C050-020X044
- C9: device c:C050-024X044/V -> c:C050-020X044/V
- J1: value CONN-3P-3P -> A_IN
- J2: value CONN-3P-3P -> A_OUT
- R15: value POT-STEREO -> 10k
- R8: value POT-P5 -> (none)
- moved C7 7.62 mm to (30.5, 47.0)
- moved J3 3.59 mm to (10.2, 5.08), turned to 0 degrees
- moved C6 3.59 mm to (48.3, 40.6), turned to 90 degrees
- moved C5 2.54 mm to (53.3, 38.1)
- moved C9 2.54 mm to (43.2, 15.2)
- moved R8 1.27 mm to (5.08, 17.8)
- turned C11 to 270 degrees
- turned C4 to 180 degrees
- turned C8 to 0 degrees
- turned R11 to 90 degrees
- turned R12 to 180 degrees
- turned R14 to 270 degrees
- turned R16 to 180 degrees
- turned R19 to 180 degrees
- turned R2 to 270 degrees
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Connections:
- net LEFT_IN: now also L_IN.1; no longer LEFT_IN.1
- net LEFT_OUT: now also L_OUT.1; no longer LEFT_OUT.1
- net N$10: now also R4.2; no longer R4.1
- net N$12: now also R14.1; no longer R14.2
- net N$13: now also R12.1; no longer R12.2
- net N$14: now also R16.1, R19.2; no longer R16.2, R19.1
- net N$15: now also R16.2; no longer R16.1
- net N$17: now also R11.1, R14.2; no longer R11.2, R14.1
- net N$2: now also R4.1; no longer R4.2
- net N$20: now also R11.2; no longer R11.1
- net N$28: now also R23.1; no longer R23.2
- net N$5: now also R2.1; no longer R2.2
- net N$7: now also R5.1; no longer R5.2
- net N$8: now also R3.1; no longer R3.2
- net N$9: now also R2.2, R3.2; no longer R2.1, R3.1
- net RIGHT_IN: now also R_IN.1; no longer RIGHT_IN.1
- net RIGHT_OUT: now also R_OUT.1; no longer RIGHT_OUT.1
- net TRIM_2_B: now also R19.1; no longer R19.2
- net TRI_OUT: now also R23.2; no longer R23.1
- net VCC: now also R12.2, R5.2; no longer R12.1, R5.1
Routing:
- net RIGHT_OUT: track 22.9 -> 5.08 mm
- net N$12: track 71.2 -> 78.8 mm
- net LEFT_IN: track 11.4 -> 5.08 mm
- net N$28: track 40.6 -> 35.6 mm
- net RIGHT_IN: track 6.35 -> 2.54 mm
- net GND: track 176.5 -> 174.0 mm, vias 6 -> 8
- net N$5: track 48.3 -> 45.7 mm
- net N$17: track 30.5 -> 27.9 mm
- net N$9: track 15.2 -> 12.7 mm
- net VCC: track 78.7 -> 81.3 mm

Commit message: ...
Routing:
- net N$9: track 12.7 -> 17.8 mm
- net N$2: track 41.9 -> 39.4 mm
Changed lines of the file:
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@@
 <contactref element="R2" pad="2"/>
 <wire x1="15.24" y1="35.56" x2="15.24" y2="33.02" width="0.6096" layer="16"/>
-<wire x1="15.24" y1="35.56" x2="10.16" y2="35.56" width="0.6096" layer="16"/>
+<wire x1="15.24" y1="35.56" x2="15.24" y2="33.02" width="0.6096" layer="16"/>
+<wire x1="15.24" y1="33.02" x2="10.16" y2="33.02" width="0.6096" layer="16"/>
+<wire x1="10.16" y1="33.02" x2="10.16" y2="35.56" width="0.6096" layer="16"/>
 </signal>
 <signal name="N$2">
@@
 <contactref element="IC1" pad="2"/>
 <wire x1="30.48" y1="27.94" x2="15.24" y2="27.94" width="0.6096" layer="16"/>
-<wire x1="10.16" y1="27.94" x2="10.16" y2="30.48" width="0.6096" layer="16"/>
-<wire x1="10.16" y1="30.48" x2="15.24" y2="30.48" width="0.6096" layer="16"/>
+<wire x1="10.16" y1="27.94" x2="15.24" y2="27.94" width="0.6096" layer="16"/>
 <wire x1="15.24" y1="30.48" x2="15.24" y2="27.94" width="0.6096" layer="16"/>
 <wire x1="15.24" y1="29.21" x2="15.24" y2="30.48" width="0.6096" layer="16"/>

Commit message: ...
Parts:
- C1: device c:C050-020X044 -> c:C075-020X044/V
- C9: device c:C050-020X044/V -> c:C050-024X044
- D2: device d:DO35-2_54 -> d:DO34-7V
- R10, R17, R9: device r:0204/7 -> r:0204/10
- R14, R22, R5: device r:0204V -> r:0204/2V
- R21: device r:0204/10 -> r:0204/10-V
- moved D2 13.1 mm to (50.8, 44.5)
- moved R2 7.62 mm to (7.62, 36.8)
- moved C2 5.08 mm to (15.2, 38.1)
- moved CV_IN 3.59 mm to (25.4, 35.6)
- moved C3 2.54 mm to (15.2, 54.6)
- moved LED2 2.54 mm to (16.5, 15.2)
- moved LED1 2.54 mm to (16.5, 10.2)
- moved C9 2.54 mm to (45.7, 15.2), turned to 180 degrees
- moved R9 1.27 mm to (33.0, 38.1)
- moved C1 1.27 mm to (10.2, 31.8), turned to 180 degrees
- moved R10 1.27 mm to (33.0, 33.0)
- moved R17 1.27 mm to (35.6, 10.2)
- turned R14 to 0 degrees
- turned R21 to 0 degrees
- turned R22 to 0 degrees
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Connections:
- net OA_C_IN+: now also R21.2; no longer R21.1
- net VCC: now also R21.1; no longer R21.2
Routing:
- net N$3: track 10.2 -> 15.2 mm
- net N$9: track 17.8 -> 12.7 mm
- net N$16: track 29.2 -> 25.4 mm
- net GND: track 174.0 -> 176.5 mm, vias 8 -> 6
- net TRIM_P: track 22.9 -> 25.4 mm
- net N$15: track 27.9 -> 25.4 mm
- net LEFT_OUT: track 10.2 -> 12.7 mm
- net N$26: track 15.2 -> 17.8 mm

Commit message: ...
Parts:
- moved C3 2.54 mm to (15.2, 52.1), turned to 0 degrees
- moved C7 2.54 mm to (27.9, 47.0)
Routing:
- net RIGHT_OUT: track 5.08 -> 7.62 mm
- net N$12: track 78.8 -> 76.3 mm
- net VCC: vias 2 -> 4
Other:
- board size 55.9 x 61 mm -> 55.9 x 58.4 mm
Changed lines of the file:
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@@
 <plain>
 <wire x1="2.54" y1="0" x2="58.42" y2="0" width="0" layer="20"/>
-<wire x1="58.42" y1="0" x2="58.42" y2="60.96" width="0" layer="20"/>
-<wire x1="58.42" y1="60.96" x2="2.54" y2="60.96" width="0" layer="20"/>
-<wire x1="2.54" y1="60.96" x2="2.54" y2="0" width="0" layer="20"/>
+<wire x1="58.42" y1="0" x2="58.42" y2="58.42" width="0" layer="20"/>
+<wire x1="58.42" y1="58.42" x2="2.54" y2="58.42" width="0" layer="20"/>
+<wire x1="2.54" y1="58.42" x2="2.54" y2="0" width="0" layer="20"/>
 <dimension x1="67.31" y1="60.96" x2="67.31" y2="0" x3="63.5" y3="30.48" textsize="1.778" layer="20" visible="yes"/>
 <dimension x1="58.42" y1="63.5" x2="2.54" y2="63.5" x3="30.48" y3="66.04" textsize="1.778" layer="20" visible="yes"/>
@@
 <element name="R2" library="r" package="0204V" value="1k" x="7.62" y="36.83" rot="R270"/>
 <element name="R3" library="r" package="0204/7" value="1k" x="19.05" y="33.02" rot="R180"/>
-<element name="C3" library="c" package="E2,5-3/V" value="1uF" x="15.24" y="54.61" rot="R180"/>
+<element name="C3" library="c" package="E2,5-3/V" value="1uF" x="15.24" y="52.07"/>
 <element name="C4" library="c" package="C050-020X044" value="1uF" x="38.1" y="50.8" rot="R180"/>
 <element name="R11" library="r" package="0204/15" value="470k" x="55.88" y="43.18" rot="R90"/>
@@
 <element name="R_IN" library="pad" package="SPAD" value="AUDIO_IN" x="48.26" y="53.34" rot="R270"/>
 <element name="R_OUT" library="pad" package="SPAD" value="AUDIO_OUT" x="30.48" y="53.34" rot="R270"/>
-<element name="C7" library="c" package="E2,5-3/V" value="1uF" x="30.48" y="46.99" rot="R180"/>
+<element name="C7" library="c" package="E2,5-3/V" value="1uF" x="27.94" y="46.99" rot="R180"/>
 <element name="C8" library="c" package="C050-020X044" value="1uF" x="50.8" y="50.8"/>
 <element name="C9" library="c" package="C050-024X044" value="1uF" x="45.72" y="15.24" rot="R180"/>
@@
 <wire x1="48.26" y1="33.02" x2="50.8" y2="33.02" width="0.6096" layer="16"/>
 <wire x1="7.62" y1="12.7" x2="12.7" y2="12.7" width="0.6096" layer="16"/>
-<wire x1="12.7" y1="12.7" x2="12.7" y2="22.86" width="0.6096" layer="16"/>
+<wire x1="12.7" y1="12.7" x2="12.7" y2="22.86" width="0.6096" layer="1"/>
 <wire x1="12.7" y1="22.86" x2="22.86" y2="22.86" width="0.6096" layer="16"/>
 <wire x1="50.8" y1="30.48" x2="50.8" y2="33.02" width="0.6096" layer="16"/>
@@
 <wire x1="35.56" y1="35.56" x2="48.26" y2="35.56" width="0.6096" layer="1"/>
 <via x="48.26" y="35.56" extent="1-16" drill="0.6" shape="square"/>
+<via x="12.7" y="12.7" extent="1-16" drill="0.6" shape="square"/>
+<via x="12.7" y="22.86" extent="1-16" drill="0.6" shape="square"/>
 </signal>
 <signal name="N$4">
@@
 <contactref element="R15" pad="2-S"/>
 <wire x1="45.72" y1="30.48" x2="38.1" y2="30.48" width="0.6096" layer="16"/>
-<wire x1="45.72" y1="30.48" x2="45.72" y2="38.1" width="0.6096" layer="16"/>
-<via x="45.72" y="38.1" extent="1-16" drill="0.6" shape="square"/>
-<wire x1="45.72" y1="38.1" x2="45.72" y2="45.72" width="0.6096" layer="1"/>
-<via x="45.72" y="45.72" extent="1-16" drill="0.6" shape="square"/>
-<wire x1="45.72" y1="45.72" x2="30.48" y2="45.72" width="0.6096" layer="16"/>
-<wire x1="45.72" y1="45.72" x2="10.16" y2="45.72" width="0.6096" layer="16"/>
+<wire x1="45.72" y1="30.48" x2="40.64" y2="30.48" width="0.6096" layer="16"/>
+<wire x1="40.64" y1="30.48" x2="40.64" y2="38.1" width="0.6096" layer="16"/>
+<via x="40.64" y="38.1" extent="1-16" drill="0.6" shape="square"/>
+<wire x1="40.64" y1="38.1" x2="40.64" y2="45.72" width="0.6096" layer="1"/>
+<via x="40.64" y="45.72" extent="1-16" drill="0.6" shape="square"/>
+<wire x1="40.64" y1="45.72" x2="27.94" y2="45.72" width="0.6096" layer="16"/>
+<wire x1="40.64" y1="45.72" x2="10.16" y2="45.72" width="0.6096" layer="16"/>
 <wire x1="10.16" y1="45.72" x2="10.16" y2="48.26" width="0.6096" layer="16"/>
 <wire x1="10.16" y1="48.26" x2="7.54" y2="48.26" width="0.6096" layer="16"/>
@@
 <contactref element="C7" pad="-"/>
 <contactref element="R_OUT" pad="1"/>
+<wire x1="27.94" y1="48.26" x2="30.48" y2="48.26" width="0.6096" layer="16"/>
 <wire x1="30.48" y1="48.26" x2="30.48" y2="53.34" width="0.6096" layer="16"/>
 </signal>
@@
 <contactref element="C3" pad="-"/>
 <contactref element="L_OUT" pad="1"/>
-<wire x1="15.24" y1="55.88" x2="25.4" y2="55.88" width="0.6096" layer="16"/>
-<wire x1="25.4" y1="55.88" x2="25.4" y2="53.34" width="0.6096" layer="16"/>
+<wire x1="15.24" y1="50.8" x2="25.4" y2="50.8" width="0.6096" layer="16"/>
+<wire x1="25.4" y1="50.8" x2="25.4" y2="53.34" width="0.6096" layer="16"/>
 </signal>
 <signal name="N$1">

Commit message: ...
Parts:
- moved J3 2.54 mm to (10.2, 2.54)
- moved R8 2.54 mm to (2.54, 17.8)
Routing:
- net VCC: track 81.3 -> 91.4 mm
- net GND: track 176.5 -> 179.1 mm
- net N$5: vias 0 -> 2
Changed lines of the file:
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@@
 <element name="C11" library="c" package="C050-020X044" value="100nF" x="53.34" y="27.94" rot="R270"/>
 <element name="R15" library="r" package="POT-STEREO-2X3" value="10k" x="7.62" y="48.26" rot="R270"/>
-<element name="R8" library="r" package="POT-P5" value="" x="5.08" y="17.78" rot="R270"/>
+<element name="R8" library="r" package="POT-P5" value="" x="2.54" y="17.78" rot="R270"/>
 <element name="J1" library="pinconn" package="CONN-3P" value="A_IN" x="43.18" y="53.34"/>
 <element name="J2" library="pinconn" package="CONN-3P" value="A_OUT" x="25.4" y="53.34"/>
-<element name="J3" library="pinconn" package="CONN-2P" value="CONN-2P2P/H" x="10.16" y="5.08"/>
+<element name="J3" library="pinconn" package="CONN-2P" value="CONN-2P2P/H" x="10.16" y="2.54"/>
 </elements>
 <signals>
@@
 <wire x1="45.72" y1="22.86" x2="48.26" y2="22.86" width="0.6096" layer="16"/>
 <wire x1="10.16" y1="22.86" x2="10.16" y2="25.4" width="0.6096" layer="16"/>
-<wire x1="10.16" y1="5.08" x2="10.16" y2="10.16" width="0.6096" layer="16"/>
-<wire x1="10.16" y1="10.16" x2="10.16" y2="22.86" width="0.6096" layer="1"/>
-<wire x1="10.16" y1="22.86" x2="7.62" y2="22.86" width="0.6096" layer="16"/>
+<wire x1="10.16" y1="2.54" x2="10.16" y2="7.62" width="0.6096" layer="16"/>
+<wire x1="10.16" y1="7.62" x2="10.16" y2="22.86" width="0.6096" layer="1"/>
+<wire x1="10.16" y1="22.86" x2="5.08" y2="22.86" width="0.6096" layer="16"/>
 <wire x1="53.34" y1="22.86" x2="55.88" y2="22.86" width="0.6096" layer="16"/>
 <wire x1="55.88" y1="22.86" x2="55.88" y2="2.54" width="0.6096" layer="16"/>
 <wire x1="55.88" y1="2.54" x2="10.16" y2="2.54" width="0.6096" layer="16"/>
-<wire x1="10.16" y1="2.54" x2="10.16" y2="5.08" width="0.6096" layer="16"/>
 <wire x1="27.94" y1="53.34" x2="27.94" y2="55.88" width="0.6096" layer="16"/>
 <wire x1="27.94" y1="55.88" x2="45.72" y2="55.88" width="0.6096" layer="16"/>
@@
 <wire x1="53.34" y1="25.4" x2="53.34" y2="22.86" width="0.6096" layer="16"/>
 <wire x1="7.62" y1="25.4" x2="10.16" y2="25.4" width="0.6096" layer="16"/>
-<via x="10.16" y="10.16" extent="1-16" drill="0.6" shape="square"/>
+<via x="10.16" y="7.62" extent="1-16" drill="0.6" shape="square"/>
 <via x="10.16" y="22.86" extent="1-16" drill="0.6" shape="square"/>
 <wire x1="50.8" y1="48.26" x2="45.72" y2="48.26" width="0.6096" layer="16"/>
@@
 <wire x1="53.34" y1="30.48" x2="50.8" y2="30.48" width="0.6096" layer="16"/>
 <wire x1="30.48" y1="22.86" x2="22.86" y2="22.86" width="0.6096" layer="16"/>
-<wire x1="7.62" y1="12.7" x2="7.62" y2="5.08" width="0.6096" layer="16"/>
+<wire x1="10.16" y1="12.7" x2="10.16" y2="10.16" width="0.6096" layer="16"/>
+<wire x1="7.62" y1="10.16" x2="7.62" y2="2.54" width="0.6096" layer="16"/>
 <wire x1="48.26" y1="35.56" x2="48.26" y2="33.02" width="0.6096" layer="16"/>
 <wire x1="48.26" y1="33.02" x2="50.8" y2="33.02" width="0.6096" layer="16"/>
-<wire x1="7.62" y1="12.7" x2="12.7" y2="12.7" width="0.6096" layer="16"/>
-<wire x1="12.7" y1="12.7" x2="12.7" y2="22.86" width="0.6096" layer="1"/>
+<wire x1="5.08" y1="12.7" x2="10.16" y2="12.7" width="0.6096" layer="16"/>
+<wire x1="10.16" y1="10.16" x2="7.62" y2="10.16" width="0.6096" layer="16"/>
+<wire x1="10.16" y1="10.16" x2="12.7" y2="10.16" width="0.6096" layer="16"/>
+<wire x1="12.7" y1="10.16" x2="12.7" y2="22.86" width="0.6096" layer="1"/>
 <wire x1="12.7" y1="22.86" x2="22.86" y2="22.86" width="0.6096" layer="16"/>
 <wire x1="50.8" y1="30.48" x2="50.8" y2="33.02" width="0.6096" layer="16"/>
@@
 <wire x1="35.56" y1="35.56" x2="48.26" y2="35.56" width="0.6096" layer="1"/>
 <via x="48.26" y="35.56" extent="1-16" drill="0.6" shape="square"/>
-<via x="12.7" y="12.7" extent="1-16" drill="0.6" shape="square"/>
+<via x="12.7" y="10.16" extent="1-16" drill="0.6" shape="square"/>
 <via x="12.7" y="22.86" extent="1-16" drill="0.6" shape="square"/>
 </signal>
@@
 <contactref element="R9" pad="2"/>
 <contactref element="R8" pad="S"/>
-<wire x1="7.62" y1="17.78" x2="5.08" y2="17.78" width="0.6096" layer="16"/>
-<wire x1="5.08" y1="17.78" x2="5.08" y2="38.1" width="0.6096" layer="16"/>
+<wire x1="5.08" y1="17.78" x2="6.35" y2="17.78" width="0.6096" layer="16"/>
+<wire x1="6.35" y1="17.78" x2="6.35" y2="25.4" width="0.6096" layer="1"/>
+<wire x1="6.35" y1="25.4" x2="5.08" y2="25.4" width="0.6096" layer="1"/>
+<wire x1="5.08" y1="25.4" x2="5.08" y2="38.1" width="0.6096" layer="1"/>
 <contactref element="R2" pad="1"/>
 <wire x1="7.62" y1="38.1" x2="27.94" y2="38.1" width="0.6096" layer="16"/>
 <wire x1="7.62" y1="38.1" x2="5.08" y2="38.1" width="0.6096" layer="16"/>
+<via x="6.35" y="17.78" extent="1-16" drill="0.6" shape="square"/>
+<via x="5.08" y="38.1" extent="1-16" drill="0.6" shape="square"/>
 </signal>
 <signal name="N$8">

Commit message: ...
Routing:
- added copper zone on layer 16, net GND
Other:
- board outline removed
