File: eagle/Simple-Bug-BC547.brd (EAGLE design)
At the start: 14 parts, among them T1 BC547

Commit message: ...
Parts:
- moved C4 7.18 mm to (2.54, 12.7), turned to 90 degrees
- moved R1 2.54 mm to (14.0, 2.54)
- moved ANT1 2.54 mm to (20.3, 10.2)
- moved C2 2.54 mm to (20.3, 5.08)
- moved C5 2.54 mm to (10.2, 7.62)
- turned C3 to 270 degrees
- renumbered L2 to L1
Routing:
- net N$5: track 12.7 -> 20.3 mm
- net N$2: track 15.2 -> 10.2 mm
- net GND: track 17.8 -> 12.7 mm
- net N$3: track 5.08 -> 7.62 mm
- net +UB: track 30.5 -> 27.9 mm
Changed lines of the file:
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@@
 <?xml version="1.0" encoding="utf-8"?>
 <!DOCTYPE eagle SYSTEM "eagle.dtd">
-<eagle version="7.7.0">
+<eagle version="7.2.0">
 <drawing>
 <settings>
@@
 <layer number="21" name="tPlace" color="7" fill="1" visible="yes" active="yes"/>
 <layer number="22" name="bPlace" color="7" fill="1" visible="yes" active="yes"/>
-<layer number="23" name="tOrigins" color="15" fill="1" visible="no" active="yes"/>
-<layer number="24" name="bOrigins" color="15" fill="1" visible="no" active="yes"/>
-<layer number="25" name="tNames" color="7" fill="1" visible="no" active="yes"/>
-<layer number="26" name="bNames" color="7" fill="1" visible="no" active="yes"/>
+<layer number="23" name="tOrigins" color="15" fill="1" visible="yes" active="yes"/>
+<layer number="24" name="bOrigins" color="15" fill="1" visible="yes" active="yes"/>
+<layer number="25" name="tNames" color="7" fill="1" visible="yes" active="yes"/>
+<layer number="26" name="bNames" color="7" fill="1" visible="yes" active="yes"/>
 <layer number="27" name="tValues" color="7" fill="1" visible="yes" active="yes"/>
 <layer number="28" name="bValues" color="7" fill="1" visible="yes" active="yes"/>
@@
 </autorouter>
 <elements>
-<element name="C2" library="c" package="C050-020X036" value="4.7pF" x="17.78" y="5.08" smashed="yes" rot="R270">
-<attribute name="NAME" x="18.6055" y="5.334" size="0.8128" layer="25" rot="R270" align="bottom-right"/>
-<attribute name="VALUE" x="16.0655" y="6.096" size="0.8128" layer="27" rot="R270"/>
-</element>
-<element name="C3" library="c" package="C050-020X036" value="1nF" x="7.62" y="5.08" rot="R180"/>
+<element name="C2" library="c" package="C050-020X036" value="4.7pF" x="20.32" y="5.08" rot="R270"/>
+<element name="C3" library="c" package="C050-020X036" value="1nF" x="7.62" y="5.08" rot="R270"/>
 <element name="R2" library="r" package="0204/7-V" value="4.7k" x="5.08" y="13.97"/>
 <element name="R3" library="r" package="0204/7-V" value="33k" x="7.62" y="13.97"/>
 <element name="ECM" library="ECM" package="ECM-4" value="ECM-4" x="2.54" y="6.35"/>
 <element name="C1" library="cap-trim" package="TRIM-2222-808" value="1.6-15pF" x="12.7" y="15.24" rot="R90"/>
-<element name="R1" library="r" package="0204/7" value="4.7" x="11.43" y="2.54" rot="R180"/>
-<element name="C4" library="c" package="C050-020X044" value="330nF" x="7.62" y="7.62"/>
+<element name="R1" library="r" package="0204/7" value="4.7" x="13.97" y="2.54" rot="R180"/>
+<element name="C4" library="c" package="C050-020X044" value="330nF" x="2.54" y="12.7" rot="R90"/>
 <element name="+9V" library="pad" package="SPAD" value="SPAD" x="2.54" y="17.78"/>
 <element name="GND" library="pad" package="SPAD" value="SPAD" x="2.54" y="2.54"/>
-<element name="ANT1" library="pad" package="SPAD" value="ANT" x="20.32" y="7.62" rot="R180"/>
-<element name="C5" library="c" package="C050-020X036/V" value="22nF" x="12.7" y="7.62" rot="R180"/>
+<element name="ANT1" library="pad" package="SPAD" value="ANT" x="20.32" y="10.16" rot="R180"/>
+<element name="C5" library="c" package="C050-020X036/V" value="22nF" x="10.16" y="7.62" rot="R180"/>
 <element name="T1" library="t" package="TO92-CBE" value="BC547" x="15.24" y="7.62" smashed="yes">
 <attribute name="NAME" x="15.24" y="8.636" size="0.8128" layer="25" ratio="10" rot="R180" align="top-center"/>
 <attribute name="VALUE" x="11.811" y="7.62" size="0.8128" layer="27" ratio="10" rot="R90" align="bottom-center"/>
 </element>
-<element name="L2" library="l" package="L-04/7V-X" value="1uH" x="19.05" y="13.97"/>
+<element name="L1" library="l" package="L-04/7V-X" value="1uH" x="19.05" y="13.97"/>
 </elements>
 <signals>
@@
 <contactref element="R1" pad="1"/>
 <contactref element="T1" pad="E"/>
+<wire x1="20.32" y1="2.54" x2="17.78" y2="2.54" width="1.27" layer="16"/>
 <wire x1="17.78" y1="2.54" x2="15.24" y2="2.54" width="1.27" layer="16"/>
 <wire x1="15.24" y1="2.54" x2="15.24" y2="5.08" width="1.27" layer="16"/>
@@
 <contactref element="C4" pad="2"/>
 <contactref element="T1" pad="B"/>
-<wire x1="10.16" y1="7.62" x2="15.24" y2="7.62" width="1.27" layer="16"/>
-<wire x1="10.16" y1="5.08" x2="10.16" y2="7.62" width="1.27" layer="16"/>
-<wire x1="10.16" y1="7.62" x2="10.16" y2="10.16" width="1.27" layer="16"/>
-<wire x1="10.16" y1="10.16" x2="7.62" y2="10.16" width="1.27" layer="16"/>
+<wire x1="2.54" y1="15.24" x2="7.62" y2="15.24" width="1.27" layer="16"/>
+<wire x1="7.62" y1="15.24" x2="7.62" y2="10.16" width="1.27" layer="16"/>
+<wire x1="7.62" y1="10.16" x2="7.62" y2="7.62" width="1.27" layer="16"/>
+<wire x1="15.24" y1="7.62" x2="7.62" y2="7.62" width="1.27" layer="16"/>
 </signal>
 <signal name="N$6">
@@
 <contactref element="C4" pad="1"/>
 <contactref element="ECM" pad="1"/>
-<wire x1="2.54" y1="7.62" x2="5.08" y2="7.62" width="1.27" layer="16"/>
-<wire x1="5.08" y1="7.62" x2="5.08" y2="10.16" width="1.27" layer="16"/>
+<wire x1="2.54" y1="7.62" x2="2.54" y2="10.16" width="1.27" layer="16"/>
+<wire x1="2.54" y1="10.16" x2="5.08" y2="10.16" width="1.27" layer="16"/>
 </signal>
 <signal name="GND">
@@
 <contactref element="C5" pad="2"/>
 <contactref element="ECM" pad="2"/>
-<wire x1="12.7" y1="5.08" x2="12.7" y2="2.54" width="1.27" layer="16"/>
-<wire x1="12.7" y1="2.54" x2="7.62" y2="2.54" width="1.27" layer="16"/>
-<wire x1="7.62" y1="2.54" x2="5.08" y2="2.54" width="1.27" layer="16"/>
-<wire x1="5.08" y1="2.54" x2="5.08" y2="5.08" width="1.27" layer="16"/>
-<wire x1="5.08" y1="2.54" x2="2.54" y2="2.54" width="1.27" layer="16"/>
-<wire x1="5.08" y1="5.08" x2="2.54" y2="5.08" width="1.27" layer="16"/>
+<wire x1="10.16" y1="5.08" x2="10.16" y2="2.54" width="1.27" layer="16"/>
+<wire x1="10.16" y1="2.54" x2="7.62" y2="2.54" width="1.27" layer="16"/>
+<wire x1="7.62" y1="2.54" x2="2.54" y2="2.54" width="1.27" layer="16"/>
+<wire x1="2.54" y1="2.54" x2="2.54" y2="5.08" width="1.27" layer="16"/>
 <polygon width="0.254" layer="16" isolate="1.27" orphans="yes" thermals="no">
 <vertex x="0" y="0"/>
@@
 <wire x1="10.16" y1="12.7" x2="10.16" y2="17.78" width="1.27" layer="16"/>
 <wire x1="10.16" y1="17.78" x2="7.62" y2="17.78" width="1.27" layer="16"/>
-<wire x1="12.7" y1="10.16" x2="12.7" y2="12.7" width="1.27" layer="16"/>
-<wire x1="12.7" y1="12.7" x2="10.16" y2="12.7" width="1.27" layer="16"/>
+<wire x1="10.16" y1="10.16" x2="10.16" y2="12.7" width="1.27" layer="16"/>
 <wire x1="5.08" y1="17.78" x2="7.62" y2="17.78" width="1.27" layer="16"/>
-<contactref element="L2" pad="2"/>
+<contactref element="L1" pad="2"/>
 <wire x1="10.16" y1="17.78" x2="15.24" y2="17.78" width="1.27" layer="16"/>
 <wire x1="20.32" y1="17.78" x2="15.24" y2="17.78" width="1.27" layer="16"/>
@@
 </signal>
 <signal name="N$2">
-<contactref element="L2" pad="1"/>
+<contactref element="L1" pad="1"/>
 <contactref element="T1" pad="C"/>
 <contactref element="C2" pad="1"/>
 <contactref element="ANT1" pad="1"/>
 <contactref element="C1" pad="2"/>
-<wire x1="20.32" y1="7.62" x2="17.78" y2="7.62" width="1.27" layer="16"/>
-<wire x1="17.78" y1="7.62" x2="17.78" y2="10.16" width="1.27" layer="16"/>
-<wire x1="15.24" y1="10.16" x2="17.78" y2="10.16" width="1.27" layer="16"/>
-<wire x1="17.78" y1="10.16" x2="17.78" y2="7.62" width="1.27" layer="16"/>
+<wire x1="17.78" y1="10.16" x2="20.32" y2="10.16" width="1.27" layer="16"/>
+<wire x1="20.32" y1="10.16" x2="20.32" y2="7.62" width="1.27" layer="16"/>
 <wire x1="15.24" y1="10.16" x2="15.24" y2="12.7" width="1.27" layer="16"/>
 <wire x1="15.24" y1="10.16" x2="17.78" y2="10.16" width="1.27" layer="16"/>

Commit message: ...
Parts:
- renumbered +9V to 9V
Changed lines of the file:
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@@
 <element name="R1" library="r" package="0204/7" value="4.7" x="13.97" y="2.54" rot="R180"/>
 <element name="C4" library="c" package="C050-020X044" value="330nF" x="2.54" y="12.7" rot="R90"/>
-<element name="+9V" library="pad" package="SPAD" value="SPAD" x="2.54" y="17.78"/>
+<element name="9V" library="pad" package="SPAD" value="SPAD" x="2.54" y="17.78"/>
 <element name="GND" library="pad" package="SPAD" value="SPAD" x="2.54" y="2.54"/>
 <element name="ANT1" library="pad" package="SPAD" value="ANT" x="20.32" y="10.16" rot="R180"/>
@@
 <contactref element="R2" pad="1"/>
 <contactref element="C1" pad="1"/>
-<contactref element="+9V" pad="1"/>
+<contactref element="9V" pad="1"/>
 <contactref element="C5" pad="1"/>
 <contactref element="C1" pad="3"/>
