File: eagle/AstableMultivibrator-PNP-old.brd (EAGLE design)
At the start: 30.5 x 20.3 mm, 10 parts, among them T1 BC557, T2 BC557

Commit message: ...
Parts:
- C1, C2: device c:C0750-020X044 -> c:C050-020X044
- R1, R2, R3: device r:0202/7-V -> r:0202/5-V
- moved OUT 30.9 mm to (-5.08, 3.81)
- moved R4 22.7 mm to (5.08, 5.08), turned to 90 degrees
- moved R1 17.8 mm to (22.9, 5.08), turned to 180 degrees
- moved T1 13.7 mm to (22.9, 10.2), turned to 90 degrees
- moved R2 12.8 mm to (20.3, 5.08), turned to 180 degrees
- moved R3 10.2 mm to (10.2, 5.08), turned to 180 degrees
- moved T2 9.16 mm to (10.2, 10.2), turned to 270 degrees
- moved C1 2.84 mm to (15.2, 7.62), turned to 180 degrees
- moved C2 2.84 mm to (15.2, 5.08), turned to 180 degrees
Routing:
- net GND: track 40.6 -> 17.8 mm
- net VCC: track 50.8 -> 39.5 mm
- net N$3: track 17.8 -> 10.2 mm, vias 0 -> 1
- net N$1: track 25.4 -> 17.8 mm
- net N$4: track 10.2 -> 5.08 mm
- net N$6: track 2.54 -> 0.00 mm
Other:
- board size 30.5 x 20.3 mm -> 27.9 x 17.8 mm
Changed lines of the file:
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@@
 </layers>
 <board>
+<description>Forced quenching improves three-transistor FM tuner
+Lyle Williams -February 29, 2016
+http://edn.com/design/diy/4441531/Forced-quenching-improves-three-transistor-FM-tuner</description>
 <plain>
-<wire x1="0" y1="0" x2="30.48" y2="0" width="0" layer="20"/>
-<wire x1="30.48" y1="0" x2="30.48" y2="20.32" width="0" layer="20"/>
-<wire x1="30.48" y1="20.32" x2="0" y2="20.32" width="0" layer="20"/>
-<wire x1="0" y1="20.32" x2="0" y2="0" width="0" layer="20"/>
+<wire x1="27.94" y1="0" x2="0" y2="0" width="0" layer="20"/>
+<wire x1="0" y1="0" x2="0" y2="17.78" width="0" layer="20"/>
+<wire x1="0" y1="17.78" x2="27.94" y2="17.78" width="0" layer="20"/>
+<wire x1="27.94" y1="17.78" x2="27.94" y2="0" width="0" layer="20"/>
 </plain>
 <attributes>
@@
 </variantdefs>
 <classes>
-<class number="0" name="default" width="0.6096" drill="0">
+<class number="0" name="default" width="0" drill="0">
 </class>
 </classes>
@@
 </autorouter>
 <elements>
-<element name="C1" library="c" package="C0750-020X044" value="2.7nF" x="13.97" y="10.16"/>
-<element name="C2" library="c" package="C0750-020X044" value="2.7nF" x="13.97" y="7.62"/>
+<element name="C2" library="c" package="C050-020X044" value="2.7nF" x="15.24" y="5.08" rot="R180"/>
+<element name="C1" library="c" package="C050-020X044" value="2.7nF" x="15.24" y="7.62" rot="R180"/>
+<element name="R2" library="r" package="0202/5-V" value="5.1k" x="20.32" y="5.08" rot="R180"/>
+<element name="R1" library="r" package="0202/5-V" value="15k" x="22.86" y="5.08" rot="R180"/>
+<element name="R3" library="r" package="0202/5-V" value="15k" x="10.16" y="5.08" rot="R180"/>
+<element name="T1" library="t" package="TO92-CBE" value="BC557" x="22.86" y="10.16" smashed="yes" rot="R90">
+<attribute name="NAME" x="22.86" y="11.43" size="0.8128" layer="25" ratio="10" rot="R180" align="center"/>
+<attribute name="VALUE" x="22.86" y="9.3345" size="0.8128" layer="27" ratio="10" rot="R180" align="center"/>
+</element>
+<element name="T2" library="t" package="TO92-CBE" value="BC557" x="10.16" y="10.16" smashed="yes" rot="R270">
+<attribute name="NAME" x="10.16" y="8.89" size="0.8128" layer="25" ratio="10" align="center"/>
+<attribute name="VALUE" x="10.16" y="10.9855" size="0.8128" layer="27" ratio="10" align="center"/>
+</element>
+<element name="OUT" library="pad" package="SPAD-+" value="SPAD+--+" x="-5.08" y="3.81" smashed="yes">
+<attribute name="NAME" x="-5.08" y="6.604" size="0.8128" layer="21" ratio="9" rot="R180" align="top-center"/>
+</element>
 <element name="J1" library="pad" package="PWR-L" value="" x="25.4" y="3.81"/>
-<element name="OUT" library="pad" package="SPAD-+" value="SPAD+--+" x="25.4" y="8.89"/>
-<element name="R1" library="r" package="0202/7-V" value="15k" x="5.08" y="6.35"/>
-<element name="R2" library="r" package="0202/7-V" value="5.1k" x="7.62" y="6.35"/>
-<element name="R3" library="r" package="0202/7-V" value="15k" x="20.32" y="6.35"/>
-<element name="R4" library="r" package="POT-V" value="5k" x="25.4" y="15.24" rot="R180"/>
-<element name="T1" library="t" package="TO92-CBE" value="BC557" x="10.16" y="15.24" rot="R180"/>
-<element name="T2" library="t" package="TO92-CBE" value="BC557" x="17.78" y="15.24" rot="R180"/>
+<element name="R4" library="r" package="POT-V" value="5k" x="5.08" y="5.08" smashed="yes" rot="R90">
+<attribute name="NAME" x="2.54" y="1.651" size="0.8128" layer="25" ratio="10"/>
+<attribute name="VALUE" x="3.81" y="8.001" size="0.8128" layer="27" ratio="10" rot="R180"/>
+</element>
 </elements>
 <signals>
@@
 <contactref element="C1" pad="1"/>
 <contactref element="R2" pad="2"/>
-<wire x1="7.62" y1="10.16" x2="10.16" y2="10.16" width="0.6096" layer="16"/>
-<wire x1="10.16" y1="10.16" x2="10.16" y2="12.7" width="0.6096" layer="16"/>
+<wire x1="17.78" y1="7.62" x2="20.32" y2="7.62" width="0.6096" layer="16"/>
+<wire x1="20.32" y1="7.62" x2="20.32" y2="10.16" width="0.6096" layer="16"/>
+<wire x1="20.32" y1="10.16" x2="20.32" y2="7.62" width="0" layer="19" extent="1-1"/>
 </signal>
 <signal name="N$4">
@@
 <contactref element="C1" pad="2"/>
 <contactref element="R3" pad="2"/>
-<wire x1="20.32" y1="10.16" x2="17.78" y2="10.16" width="0" layer="19" extent="1-1"/>
-<wire x1="17.78" y1="10.16" x2="20.32" y2="10.16" width="0.6096" layer="16"/>
-<wire x1="20.32" y1="10.16" x2="20.32" y2="15.24" width="0.6096" layer="16"/>
-<wire x1="20.32" y1="15.24" x2="17.78" y2="15.24" width="0.6096" layer="16"/>
+<wire x1="12.7" y1="7.62" x2="10.16" y2="7.62" width="0.6096" layer="16"/>
+<wire x1="10.16" y1="7.62" x2="10.16" y2="10.16" width="0.6096" layer="16"/>
 </signal>
 <signal name="N$1">
@@
 <contactref element="C2" pad="2"/>
 <contactref element="R4" pad="E"/>
-<wire x1="17.78" y1="12.7" x2="15.24" y2="12.7" width="0.6096" layer="16"/>
-<wire x1="15.24" y1="12.7" x2="15.24" y2="7.62" width="0.6096" layer="16"/>
-<wire x1="15.24" y1="7.62" x2="17.78" y2="7.62" width="0.6096" layer="16"/>
-<wire x1="22.86" y1="17.78" x2="22.86" y2="7.62" width="0.6096" layer="16"/>
-<wire x1="22.86" y1="7.62" x2="17.78" y2="7.62" width="0.6096" layer="16"/>
+<wire x1="12.7" y1="5.08" x2="7.62" y2="5.08" width="0.6096" layer="16"/>
+<wire x1="7.62" y1="5.08" x2="7.62" y2="7.62" width="0.6096" layer="16"/>
+<wire x1="12.7" y1="10.16" x2="15.24" y2="10.16" width="0.6096" layer="16"/>
+<wire x1="15.24" y1="10.16" x2="15.24" y2="5.08" width="0.6096" layer="16"/>
+<wire x1="15.24" y1="5.08" x2="12.7" y2="5.08" width="0.6096" layer="16"/>
 </signal>
 <signal name="N$3">
@@
 <contactref element="C2" pad="1"/>
 <contactref element="R1" pad="2"/>
-<wire x1="10.16" y1="7.62" x2="5.08" y2="7.62" width="0.6096" layer="16"/>
-<wire x1="5.08" y1="7.62" x2="5.08" y2="15.24" width="0.6096" layer="16"/>
-<wire x1="5.08" y1="15.24" x2="10.16" y2="15.24" width="0.6096" layer="16"/>
-<wire x1="5.08" y1="7.62" x2="5.08" y2="10.16" width="0" layer="19" extent="16-16"/>
+<via x="22.86" y="7.62" extent="1-16" drill="0.6" shape="square"/>
+<wire x1="17.78" y1="5.08" x2="22.86" y2="5.08" width="0.6096" layer="16"/>
+<wire x1="22.86" y1="5.08" x2="22.86" y2="10.16" width="0.6096" layer="16"/>
+<wire x1="22.86" y1="10.16" x2="22.86" y2="7.62" width="0" layer="19" extent="1-1"/>
 </signal>
 <signal name="N$6">
 <contactref element="OUT" pad="2"/>
 <contactref element="R4" pad="S"/>
-<wire x1="25.4" y1="10.16" x2="25.4" y2="12.7" width="0.6096" layer="16"/>
+<wire x1="-5.08" y1="5.08" x2="2.54" y2="5.08" width="0" layer="19" extent="1-1"/>
 </signal>
 <signal name="GND">
@@
 <contactref element="R3" pad="1"/>
 <contactref element="R1" pad="1"/>
+<wire x1="10.16" y1="2.54" x2="20.32" y2="2.54" width="0.6096" layer="16"/>
 <contactref element="J1" pad="1"/>
+<contactref element="OUT" pad="1"/>
+<wire x1="20.32" y1="2.54" x2="22.86" y2="2.54" width="0.6096" layer="16"/>
+<wire x1="25.4" y1="2.54" x2="22.86" y2="2.54" width="0.6096" layer="16"/>
 <contactref element="R4" pad="A"/>
-<contactref element="OUT" pad="1"/>
-<wire x1="7.62" y1="2.54" x2="20.32" y2="2.54" width="0.6096" layer="16"/>
-<wire x1="20.32" y1="2.54" x2="25.4" y2="2.54" width="0.6096" layer="16"/>
-<wire x1="27.94" y1="17.78" x2="27.94" y2="7.62" width="0.6096" layer="16"/>
-<wire x1="27.94" y1="7.62" x2="25.4" y2="7.62" width="0.6096" layer="16"/>
-<wire x1="25.4" y1="2.54" x2="27.94" y2="2.54" width="0.6096" layer="16"/>
-<wire x1="27.94" y1="2.54" x2="27.94" y2="7.62" width="0.6096" layer="16"/>
-<wire x1="7.62" y1="2.54" x2="5.08" y2="2.54" width="0.6096" layer="16"/>
+<wire x1="10.16" y1="2.54" x2="7.62" y2="2.54" width="0.6096" layer="16"/>
+<wire x1="-5.08" y1="2.54" x2="7.62" y2="2.54" width="0" layer="19" extent="1-1"/>
 </signal>
 <signal name="VCC">
 <contactref element="T1" pad="E"/>
 <contactref element="T2" pad="E"/>
+<wire x1="1.27" y1="15.24" x2="8.89" y2="15.24" width="0.6096" layer="16"/>
 <contactref element="J1" pad="2"/>
-<wire x1="10.16" y1="17.78" x2="17.78" y2="17.78" width="0.6096" layer="16"/>
-<wire x1="25.4" y1="5.08" x2="2.54" y2="5.08" width="0.6096" layer="16"/>
-<wire x1="2.54" y1="5.08" x2="2.54" y2="17.78" width="0.6096" layer="16"/>
-<wire x1="2.54" y1="17.78" x2="10.16" y2="17.78" width="0.6096" layer="16"/>
+<wire x1="7.62" y1="10.16" x2="8.89" y2="15.24" width="0.6096" layer="16"/>
+<wire x1="8.89" y1="15.24" x2="25.4" y2="15.24" width="0.6096" layer="16"/>
+<wire x1="25.4" y1="15.24" x2="25.4" y2="10.16" width="0.6096" layer="16"/>
+<wire x1="25.4" y1="10.16" x2="25.4" y2="5.08" width="0.6096" layer="16"/>
 </signal>
 </signals>

Commit message: ...
Parts:
- moved OUT 7.62 mm to (2.54, 3.81)
- moved J1 2.54 mm to (27.9, 3.81)
- moved C1 2.54 mm to (17.8, 7.62)
- moved C2 2.54 mm to (17.8, 5.08)
- moved R4 2.54 mm to (7.62, 5.08)
- moved R1 2.54 mm to (25.4, 5.08)
- moved R2 2.54 mm to (22.9, 5.08)
- moved R3 2.54 mm to (12.7, 5.08)
- moved T1 2.54 mm to (25.4, 10.2)
- moved T2 2.54 mm to (12.7, 10.2)
Routing:
- net VCC: track 39.5 -> 27.9 mm
- net GND: track 17.8 -> 25.4 mm
- net N$6: track 0.00 -> 2.54 mm
Other:
- board size 27.9 x 17.8 mm -> 30.5 x 15.2 mm
Changed lines of the file:
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@@
 http://edn.com/design/diy/4441531/Forced-quenching-improves-three-transistor-FM-tuner</description>
 <plain>
-<wire x1="27.94" y1="0" x2="0" y2="0" width="0" layer="20"/>
-<wire x1="0" y1="0" x2="0" y2="17.78" width="0" layer="20"/>
-<wire x1="0" y1="17.78" x2="27.94" y2="17.78" width="0" layer="20"/>
-<wire x1="27.94" y1="17.78" x2="27.94" y2="0" width="0" layer="20"/>
+<wire x1="30.48" y1="0" x2="0" y2="0" width="0" layer="20"/>
+<wire x1="0" y1="0" x2="0" y2="15.24" width="0" layer="20"/>
+<wire x1="0" y1="15.24" x2="30.48" y2="15.24" width="0" layer="20"/>
+<wire x1="30.48" y1="15.24" x2="30.48" y2="0" width="0" layer="20"/>
 </plain>
 <attributes>
@@
 </variantdefs>
 <classes>
-<class number="0" name="default" width="0" drill="0">
+<class number="0" name="default" width="0.6096" drill="0">
 </class>
 </classes>
@@
 </autorouter>
 <elements>
-<element name="C2" library="c" package="C050-020X044" value="2.7nF" x="15.24" y="5.08" rot="R180"/>
-<element name="C1" library="c" package="C050-020X044" value="2.7nF" x="15.24" y="7.62" rot="R180"/>
-<element name="R2" library="r" package="0202/5-V" value="5.1k" x="20.32" y="5.08" rot="R180"/>
-<element name="R1" library="r" package="0202/5-V" value="15k" x="22.86" y="5.08" rot="R180"/>
-<element name="R3" library="r" package="0202/5-V" value="15k" x="10.16" y="5.08" rot="R180"/>
-<element name="T1" library="t" package="TO92-CBE" value="BC557" x="22.86" y="10.16" smashed="yes" rot="R90">
-<attribute name="NAME" x="22.86" y="11.43" size="0.8128" layer="25" ratio="10" rot="R180" align="center"/>
-<attribute name="VALUE" x="22.86" y="9.3345" size="0.8128" layer="27" ratio="10" rot="R180" align="center"/>
-</element>
-<element name="T2" library="t" package="TO92-CBE" value="BC557" x="10.16" y="10.16" smashed="yes" rot="R270">
-<attribute name="NAME" x="10.16" y="8.89" size="0.8128" layer="25" ratio="10" align="center"/>
-<attribute name="VALUE" x="10.16" y="10.9855" size="0.8128" layer="27" ratio="10" align="center"/>
-</element>
-<element name="OUT" library="pad" package="SPAD-+" value="SPAD+--+" x="-5.08" y="3.81" smashed="yes">
-<attribute name="NAME" x="-5.08" y="6.604" size="0.8128" layer="21" ratio="9" rot="R180" align="top-center"/>
-</element>
-<element name="J1" library="pad" package="PWR-L" value="" x="25.4" y="3.81"/>
-<element name="R4" library="r" package="POT-V" value="5k" x="5.08" y="5.08" smashed="yes" rot="R90">
-<attribute name="NAME" x="2.54" y="1.651" size="0.8128" layer="25" ratio="10"/>
-<attribute name="VALUE" x="3.81" y="8.001" size="0.8128" layer="27" ratio="10" rot="R180"/>
+<element name="C2" library="c" package="C050-020X044" value="2.7nF" x="17.78" y="5.08" rot="R180"/>
+<element name="C1" library="c" package="C050-020X044" value="2.7nF" x="17.78" y="7.62" rot="R180"/>
+<element name="R2" library="r" package="0202/5-V" value="5.1k" x="22.86" y="5.08" rot="R180"/>
+<element name="R1" library="r" package="0202/5-V" value="15k" x="25.4" y="5.08" rot="R180"/>
+<element name="R3" library="r" package="0202/5-V" value="15k" x="12.7" y="5.08" rot="R180"/>
+<element name="T1" library="t" package="TO92-CBE" value="BC557" x="25.4" y="10.16" smashed="yes" rot="R90">
+<attribute name="NAME" x="25.4" y="11.43" size="0.8128" layer="25" ratio="10" rot="R180" align="center"/>
+<attribute name="VALUE" x="25.4" y="9.3345" size="0.8128" layer="27" ratio="10" rot="R180" align="center"/>
+</element>
+<element name="T2" library="t" package="TO92-CBE" value="BC557" x="12.7" y="10.16" smashed="yes" rot="R270">
+<attribute name="NAME" x="12.7" y="8.89" size="0.8128" layer="25" ratio="10" align="center"/>
+<attribute name="VALUE" x="12.7" y="10.9855" size="0.8128" layer="27" ratio="10" align="center"/>
+</element>
+<element name="OUT" library="pad" package="SPAD-+" value="SPAD+--+" x="2.54" y="3.81" smashed="yes">
+<attribute name="NAME" x="2.54" y="6.604" size="0.8128" layer="21" ratio="9" rot="R180" align="top-center"/>
+</element>
+<element name="J1" library="pad" package="PWR-L" value="" x="27.94" y="3.81"/>
+<element name="R4" library="r" package="POT-V" value="5k" x="7.62" y="5.08" smashed="yes" rot="R90">
+<attribute name="NAME" x="5.08" y="1.651" size="0.8128" layer="25" ratio="10"/>
+<attribute name="VALUE" x="6.35" y="8.001" size="0.8128" layer="27" ratio="10" rot="R180"/>
 </element>
 </elements>
@@
 <contactref element="C1" pad="1"/>
 <contactref element="R2" pad="2"/>
-<wire x1="17.78" y1="7.62" x2="20.32" y2="7.62" width="0.6096" layer="16"/>
-<wire x1="20.32" y1="7.62" x2="20.32" y2="10.16" width="0.6096" layer="16"/>
-<wire x1="20.32" y1="10.16" x2="20.32" y2="7.62" width="0" layer="19" extent="1-1"/>
+<wire x1="20.32" y1="7.62" x2="22.86" y2="7.62" width="0.6096" layer="16"/>
+<wire x1="22.86" y1="7.62" x2="22.86" y2="10.16" width="0.6096" layer="16"/>
+<wire x1="22.86" y1="10.16" x2="22.86" y2="7.62" width="0" layer="19" extent="1-1"/>
 </signal>
 <signal name="N$4">
@@
 <contactref element="C1" pad="2"/>
 <contactref element="R3" pad="2"/>
-<wire x1="12.7" y1="7.62" x2="10.16" y2="7.62" width="0.6096" layer="16"/>
-<wire x1="10.16" y1="7.62" x2="10.16" y2="10.16" width="0.6096" layer="16"/>
+<wire x1="15.24" y1="7.62" x2="12.7" y2="7.62" width="0.6096" layer="16"/>
+<wire x1="12.7" y1="7.62" x2="12.7" y2="10.16" width="0.6096" layer="16"/>
 </signal>
 <signal name="N$1">
@@
 <contactref element="C2" pad="2"/>
 <contactref element="R4" pad="E"/>
-<wire x1="12.7" y1="5.08" x2="7.62" y2="5.08" width="0.6096" layer="16"/>
-<wire x1="7.62" y1="5.08" x2="7.62" y2="7.62" width="0.6096" layer="16"/>
-<wire x1="12.7" y1="10.16" x2="15.24" y2="10.16" width="0.6096" layer="16"/>
-<wire x1="15.24" y1="10.16" x2="15.24" y2="5.08" width="0.6096" layer="16"/>
-<wire x1="15.24" y1="5.08" x2="12.7" y2="5.08" width="0.6096" layer="16"/>
+<wire x1="15.24" y1="5.08" x2="10.16" y2="5.08" width="0.6096" layer="16"/>
+<wire x1="10.16" y1="5.08" x2="10.16" y2="7.62" width="0.6096" layer="16"/>
+<wire x1="15.24" y1="10.16" x2="17.78" y2="10.16" width="0.6096" layer="16"/>
+<wire x1="17.78" y1="10.16" x2="17.78" y2="5.08" width="0.6096" layer="16"/>
+<wire x1="17.78" y1="5.08" x2="15.24" y2="5.08" width="0.6096" layer="16"/>
 </signal>
 <signal name="N$3">
@@
 <contactref element="C2" pad="1"/>
 <contactref element="R1" pad="2"/>
-<via x="22.86" y="7.62" extent="1-16" drill="0.6" shape="square"/>
-<wire x1="17.78" y1="5.08" x2="22.86" y2="5.08" width="0.6096" layer="16"/>
-<wire x1="22.86" y1="5.08" x2="22.86" y2="10.16" width="0.6096" layer="16"/>
-<wire x1="22.86" y1="10.16" x2="22.86" y2="7.62" width="0" layer="19" extent="1-1"/>
+<via x="25.4" y="7.62" extent="1-16" drill="0.6" shape="square"/>
+<wire x1="20.32" y1="5.08" x2="25.4" y2="5.08" width="0.6096" layer="16"/>
+<wire x1="25.4" y1="5.08" x2="25.4" y2="10.16" width="0.6096" layer="16"/>
+<wire x1="25.4" y1="10.16" x2="25.4" y2="7.62" width="0" layer="19" extent="1-1"/>
 </signal>
 <signal name="N$6">
 <contactref element="OUT" pad="2"/>
 <contactref element="R4" pad="S"/>
-<wire x1="-5.08" y1="5.08" x2="2.54" y2="5.08" width="0" layer="19" extent="1-1"/>
+<wire x1="2.54" y1="5.08" x2="5.08" y2="5.08" width="0.6096" layer="16"/>
 </signal>
 <signal name="GND">
@@
 <contactref element="R3" pad="1"/>
 <contactref element="R1" pad="1"/>
-<wire x1="10.16" y1="2.54" x2="20.32" y2="2.54" width="0.6096" layer="16"/>
+<wire x1="12.7" y1="2.54" x2="22.86" y2="2.54" width="0.6096" layer="16"/>
 <contactref element="J1" pad="1"/>
 <contactref element="OUT" pad="1"/>
-<wire x1="20.32" y1="2.54" x2="22.86" y2="2.54" width="0.6096" layer="16"/>
-<wire x1="25.4" y1="2.54" x2="22.86" y2="2.54" width="0.6096" layer="16"/>
+<wire x1="22.86" y1="2.54" x2="25.4" y2="2.54" width="0.6096" layer="16"/>
+<wire x1="27.94" y1="2.54" x2="25.4" y2="2.54" width="0.6096" layer="16"/>
 <contactref element="R4" pad="A"/>
-<wire x1="10.16" y1="2.54" x2="7.62" y2="2.54" width="0.6096" layer="16"/>
-<wire x1="-5.08" y1="2.54" x2="7.62" y2="2.54" width="0" layer="19" extent="1-1"/>
+<wire x1="12.7" y1="2.54" x2="10.16" y2="2.54" width="0.6096" layer="16"/>
+<wire x1="2.54" y1="2.54" x2="10.16" y2="2.54" width="0.6096" layer="16"/>
 </signal>
 <signal name="VCC">
 <contactref element="T1" pad="E"/>
 <contactref element="T2" pad="E"/>
-<wire x1="1.27" y1="15.24" x2="8.89" y2="15.24" width="0.6096" layer="16"/>
 <contactref element="J1" pad="2"/>
-<wire x1="7.62" y1="10.16" x2="8.89" y2="15.24" width="0.6096" layer="16"/>
-<wire x1="8.89" y1="15.24" x2="25.4" y2="15.24" width="0.6096" layer="16"/>
-<wire x1="25.4" y1="15.24" x2="25.4" y2="10.16" width="0.6096" layer="16"/>
-<wire x1="25.4" y1="10.16" x2="25.4" y2="5.08" width="0.6096" layer="16"/>
+<wire x1="10.16" y1="10.16" x2="10.16" y2="12.7" width="0.6096" layer="16"/>
+<wire x1="10.16" y1="12.7" x2="27.94" y2="12.7" width="0.6096" layer="16"/>
+<wire x1="27.94" y1="12.7" x2="27.94" y2="10.16" width="0.6096" layer="16"/>
+<wire x1="27.94" y1="10.16" x2="27.94" y2="5.08" width="0.6096" layer="16"/>
 </signal>
 </signals>
