File: eagle/BatteryMonitor-12V-LMT2901.brd (EAGLE design)
At the start: 40.6 x 27.9 mm, 20 parts, among them IC1 LMT2901N

Commit message: ...
Changed lines of the file:
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@@
 <contactref element="C1" pad="-"/>
 <contactref element="R7" pad="3"/>
-<wire x1="17.78" y1="11.43" x2="17.78" y2="3.81" width="0.6096" layer="16"/>
-<wire x1="15.24" y1="3.81" x2="7.62" y2="3.81" width="0.6096" layer="16"/>
-<wire x1="25.4" y1="11.43" x2="25.4" y2="13.97" width="0.6096" layer="16"/>
-<wire x1="25.4" y1="13.97" x2="17.78" y2="13.97" width="0.6096" layer="16"/>
-<wire x1="17.78" y1="13.97" x2="17.78" y2="11.43" width="0.6096" layer="16"/>
-<wire x1="15.24" y1="3.81" x2="17.78" y2="3.81" width="0.6096" layer="16"/>
-<wire x1="33.02" y1="13.97" x2="25.4" y2="13.97" width="0.6096" layer="16"/>
+<wire x1="17.78" y1="11.43" x2="17.78" y2="3.81" width="1.27" layer="16"/>
+<wire x1="15.24" y1="3.81" x2="7.62" y2="3.81" width="1.27" layer="16"/>
+<wire x1="25.4" y1="11.43" x2="25.4" y2="13.97" width="1.27" layer="16"/>
+<wire x1="25.4" y1="13.97" x2="17.78" y2="13.97" width="1.27" layer="16"/>
+<wire x1="17.78" y1="13.97" x2="17.78" y2="11.43" width="1.27" layer="16"/>
+<wire x1="15.24" y1="3.81" x2="17.78" y2="3.81" width="1.27" layer="16"/>
+<wire x1="33.02" y1="13.97" x2="25.4" y2="13.97" width="1.27" layer="16"/>
 <wire x1="33.02" y1="13.97" x2="29.21" y2="13.97" width="0" layer="19" extent="1-1"/>
 </signal>
@@
 <contactref element="R11" pad="2"/>
 <contactref element="LED4" pad="K"/>
-<wire x1="35.56" y1="3.81" x2="35.56" y2="6.35" width="0.6096" layer="16"/>
+<wire x1="35.56" y1="3.81" x2="35.56" y2="6.35" width="1.27" layer="16"/>
 </signal>
 <signal name="N$2">
@@
 <contactref element="R9" pad="2"/>
 <contactref element="LED2" pad="K"/>
-<wire x1="35.56" y1="19.05" x2="35.56" y2="16.51" width="0.6096" layer="16"/>
+<wire x1="35.56" y1="19.05" x2="35.56" y2="16.51" width="1.27" layer="16"/>
 </signal>
 <signal name="N$4">
 <contactref element="R8" pad="2"/>
 <contactref element="LED1" pad="K"/>
-<wire x1="35.56" y1="24.13" x2="35.56" y2="21.59" width="0.6096" layer="16"/>
+<wire x1="35.56" y1="24.13" x2="35.56" y2="21.59" width="1.27" layer="16"/>
 </signal>
 <signal name="N$5">
 <contactref element="R8" pad="1"/>
 <contactref element="IC1" pad="2"/>
-<wire x1="25.4" y1="24.13" x2="20.32" y2="24.13" width="0.6096" layer="16"/>
-<wire x1="20.32" y1="24.13" x2="20.32" y2="19.05" width="0.6096" layer="16"/>
+<wire x1="25.4" y1="24.13" x2="20.32" y2="24.13" width="1.27" layer="16"/>
+<wire x1="20.32" y1="24.13" x2="20.32" y2="19.05" width="1.27" layer="16"/>
 </signal>
 <signal name="N$6">
 <contactref element="IC1" pad="1"/>
 <contactref element="R9" pad="1"/>
-<wire x1="25.4" y1="19.05" x2="22.86" y2="19.05" width="0.6096" layer="16"/>
+<wire x1="25.4" y1="19.05" x2="22.86" y2="19.05" width="1.27" layer="16"/>
 </signal>
 <signal name="N$7">
 <contactref element="IC1" pad="14"/>
 <contactref element="R10" pad="1"/>
-<wire x1="25.4" y1="8.89" x2="22.86" y2="8.89" width="0.6096" layer="16"/>
-<wire x1="22.86" y1="8.89" x2="22.86" y2="11.43" width="0.6096" layer="16"/>
+<wire x1="25.4" y1="8.89" x2="22.86" y2="8.89" width="1.27" layer="16"/>
+<wire x1="22.86" y1="8.89" x2="22.86" y2="11.43" width="1.27" layer="16"/>
 </signal>
 <signal name="N$8">
 <contactref element="IC1" pad="13"/>
 <contactref element="R11" pad="1"/>
-<wire x1="20.32" y1="11.43" x2="20.32" y2="3.81" width="0.6096" layer="16"/>
-<wire x1="20.32" y1="3.81" x2="25.4" y2="3.81" width="0.6096" layer="16"/>
+<wire x1="20.32" y1="11.43" x2="20.32" y2="3.81" width="1.27" layer="16"/>
+<wire x1="20.32" y1="3.81" x2="25.4" y2="3.81" width="1.27" layer="16"/>
 </signal>
 <signal name="N$9">
@@
 <contactref element="IC1" pad="9"/>
 <contactref element="IC1" pad="11"/>
-<wire x1="12.7" y1="19.05" x2="12.7" y2="13.97" width="0.6096" layer="16"/>
-<wire x1="15.24" y1="11.43" x2="15.24" y2="13.97" width="0.6096" layer="16"/>
-<wire x1="10.16" y1="13.97" x2="7.62" y2="13.97" width="0.6096" layer="16"/>
-<wire x1="12.7" y1="13.97" x2="10.16" y2="13.97" width="0.6096" layer="16"/>
-<wire x1="10.16" y1="13.97" x2="10.16" y2="11.43" width="0.6096" layer="16"/>
-<wire x1="7.62" y1="19.05" x2="7.62" y2="13.97" width="0.6096" layer="16"/>
-<wire x1="12.7" y1="21.59" x2="12.7" y2="19.05" width="0.6096" layer="16"/>
-<wire x1="12.7" y1="13.97" x2="15.24" y2="13.97" width="0.6096" layer="16"/>
-<wire x1="15.24" y1="11.43" x2="15.24" y2="8.89" width="0.6096" layer="16"/>
+<wire x1="12.7" y1="19.05" x2="12.7" y2="13.97" width="1.27" layer="16"/>
+<wire x1="15.24" y1="11.43" x2="15.24" y2="13.97" width="1.27" layer="16"/>
+<wire x1="10.16" y1="13.97" x2="7.62" y2="13.97" width="1.27" layer="16"/>
+<wire x1="12.7" y1="13.97" x2="10.16" y2="13.97" width="1.27" layer="16"/>
+<wire x1="10.16" y1="13.97" x2="10.16" y2="11.43" width="1.27" layer="16"/>
+<wire x1="7.62" y1="19.05" x2="7.62" y2="13.97" width="1.27" layer="16"/>
+<wire x1="12.7" y1="21.59" x2="12.7" y2="19.05" width="1.27" layer="16"/>
+<wire x1="12.7" y1="13.97" x2="15.24" y2="13.97" width="1.27" layer="16"/>
+<wire x1="15.24" y1="11.43" x2="15.24" y2="8.89" width="1.27" layer="16"/>
 </signal>
 <signal name="N$10">
@@
 <contactref element="R3" pad="2"/>
 <contactref element="IC1" pad="4"/>
-<wire x1="15.24" y1="26.67" x2="15.24" y2="24.13" width="0.6096" layer="16"/>
-<wire x1="15.24" y1="26.67" x2="15.24" y2="19.05" width="0.6096" layer="16"/>
+<wire x1="15.24" y1="26.67" x2="15.24" y2="24.13" width="1.27" layer="16"/>
+<wire x1="15.24" y1="26.67" x2="15.24" y2="19.05" width="1.27" layer="16"/>
 </signal>
 <signal name="N$11">
@@
 <contactref element="R3" pad="1"/>
 <contactref element="R4" pad="2"/>
-<wire x1="10.16" y1="19.05" x2="10.16" y2="24.13" width="0.6096" layer="16"/>
-<wire x1="5.08" y1="21.59" x2="5.08" y2="24.13" width="0.6096" layer="16"/>
-<wire x1="5.08" y1="24.13" x2="10.16" y2="24.13" width="0.6096" layer="16"/>
+<wire x1="10.16" y1="19.05" x2="10.16" y2="24.13" width="1.27" layer="16"/>
+<wire x1="5.08" y1="21.59" x2="5.08" y2="24.13" width="1.27" layer="16"/>
+<wire x1="5.08" y1="24.13" x2="10.16" y2="24.13" width="1.27" layer="16"/>
 </signal>
 <signal name="N$12">
@@
 <contactref element="R4" pad="1"/>
 <contactref element="R5" pad="2"/>
-<wire x1="7.62" y1="11.43" x2="5.08" y2="11.43" width="0.6096" layer="16"/>
-<wire x1="2.54" y1="8.89" x2="2.54" y2="11.43" width="0.6096" layer="16"/>
-<wire x1="2.54" y1="11.43" x2="5.08" y2="11.43" width="0.6096" layer="16"/>
+<wire x1="7.62" y1="11.43" x2="5.08" y2="11.43" width="1.27" layer="16"/>
+<wire x1="2.54" y1="8.89" x2="2.54" y2="11.43" width="1.27" layer="16"/>
+<wire x1="2.54" y1="11.43" x2="5.08" y2="11.43" width="1.27" layer="16"/>
 </signal>
 <signal name="N$13">
@@
 <contactref element="R5" pad="1"/>
 <contactref element="R6" pad="2"/>
-<wire x1="12.7" y1="8.89" x2="12.7" y2="11.43" width="0.6096" layer="16"/>
-<wire x1="12.7" y1="6.35" x2="12.7" y2="8.89" width="0.6096" layer="16"/>
+<wire x1="12.7" y1="8.89" x2="12.7" y2="11.43" width="1.27" layer="16"/>
+<wire x1="12.7" y1="6.35" x2="12.7" y2="8.89" width="1.27" layer="16"/>
 </signal>
 <signal name="VCC">
@@
 <contactref element="LED4" pad="A"/>
 <contactref element="IC1" pad="3"/>
-<wire x1="38.1" y1="6.35" x2="38.1" y2="16.51" width="0.6096" layer="16"/>
-<wire x1="38.1" y1="16.51" x2="38.1" y2="21.59" width="0.6096" layer="16"/>
-<wire x1="17.78" y1="19.05" x2="17.78" y2="26.67" width="0.6096" layer="16"/>
-<wire x1="17.78" y1="26.67" x2="25.4" y2="26.67" width="0.6096" layer="16"/>
-<wire x1="25.4" y1="26.67" x2="38.1" y2="26.67" width="0.6096" layer="16"/>
-<wire x1="38.1" y1="26.67" x2="38.1" y2="21.59" width="0.6096" layer="16"/>
-<wire x1="22.86" y1="21.59" x2="27.94" y2="21.59" width="0.6096" layer="16"/>
-<wire x1="27.94" y1="21.59" x2="27.94" y2="26.67" width="0.6096" layer="16"/>
-<wire x1="27.94" y1="26.67" x2="25.4" y2="26.67" width="0.6096" layer="16"/>
+<wire x1="38.1" y1="6.35" x2="38.1" y2="16.51" width="1.27" layer="16"/>
+<wire x1="38.1" y1="16.51" x2="38.1" y2="21.59" width="1.27" layer="16"/>
+<wire x1="17.78" y1="19.05" x2="17.78" y2="26.67" width="1.27" layer="16"/>
+<wire x1="17.78" y1="26.67" x2="25.4" y2="26.67" width="1.27" layer="16"/>
+<wire x1="25.4" y1="26.67" x2="38.1" y2="26.67" width="1.27" layer="16"/>
+<wire x1="38.1" y1="26.67" x2="38.1" y2="21.59" width="1.27" layer="16"/>
+<wire x1="22.86" y1="21.59" x2="27.94" y2="21.59" width="1.27" layer="16"/>
+<wire x1="27.94" y1="21.59" x2="27.94" y2="26.67" width="1.27" layer="16"/>
+<wire x1="27.94" y1="26.67" x2="25.4" y2="26.67" width="1.27" layer="16"/>
 <contactref element="PWR" pad="2"/>
 <contactref element="C2" pad="1"/>
 <contactref element="C1" pad="+"/>
-<wire x1="25.4" y1="16.51" x2="17.78" y2="16.51" width="0.6096" layer="16"/>
-<wire x1="17.78" y1="16.51" x2="17.78" y2="19.05" width="0.6096" layer="16"/>
-<wire x1="33.02" y1="16.51" x2="25.4" y2="16.51" width="0.6096" layer="16"/>
+<wire x1="25.4" y1="16.51" x2="17.78" y2="16.51" width="1.27" layer="16"/>
+<wire x1="17.78" y1="16.51" x2="17.78" y2="19.05" width="1.27" layer="16"/>
+<wire x1="33.02" y1="16.51" x2="25.4" y2="16.51" width="1.27" layer="16"/>
 <wire x1="38.1" y1="16.51" x2="38.1" y2="12.7" width="0" layer="19" extent="1-16"/>
 <wire x1="38.1" y1="12.7" x2="38.1" y2="11.43" width="0" layer="19" extent="16-16"/>
@@
 <contactref element="R7" pad="2"/>
 <contactref element="R7" pad="1"/>
-<wire x1="5.08" y1="3.81" x2="2.54" y2="3.81" width="0.6096" layer="16"/>
+<wire x1="5.08" y1="3.81" x2="2.54" y2="3.81" width="1.27" layer="16"/>
 <contactref element="R6" pad="1"/>
-<wire x1="2.54" y1="3.81" x2="2.54" y2="6.35" width="0.6096" layer="16"/>
+<wire x1="2.54" y1="3.81" x2="2.54" y2="6.35" width="1.27" layer="16"/>
 </signal>
 </signals>

Commit message: ...
Routing:
- added copper zone on layer 16, net GND
Other:
- board outline removed
Changed lines of the file:
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@@
 <?xml version="1.0" encoding="utf-8"?>
 <!DOCTYPE eagle SYSTEM "eagle.dtd">
-<eagle version="7.6.0">
+<eagle version="7.7.0">
 <drawing>
 <settings>
@@
 http://www.circuitdiagram.org/battery-monitor-using-lm339-ic.html</description>
 <plain>
-<wire x1="0" y1="1.27" x2="40.64" y2="1.27" width="0" layer="20"/>
-<wire x1="40.64" y1="1.27" x2="40.64" y2="29.21" width="0" layer="20"/>
-<wire x1="40.64" y1="29.21" x2="0" y2="29.21" width="0" layer="20"/>
-<wire x1="0" y1="29.21" x2="0" y2="1.27" width="0" layer="20"/>
+<wire x1="0" y1="1.27" x2="40.64" y2="1.27" width="0" layer="47"/>
+<wire x1="40.64" y1="1.27" x2="40.64" y2="29.21" width="0" layer="47"/>
+<wire x1="40.64" y1="29.21" x2="0" y2="29.21" width="0" layer="47"/>
+<wire x1="0" y1="29.21" x2="0" y2="1.27" width="0" layer="47"/>
 </plain>
 <attributes>
@@
 <wire x1="15.24" y1="3.81" x2="17.78" y2="3.81" width="1.27" layer="16"/>
 <wire x1="33.02" y1="13.97" x2="25.4" y2="13.97" width="1.27" layer="16"/>
-<wire x1="33.02" y1="13.97" x2="29.21" y2="13.97" width="0" layer="19" extent="1-1"/>
+<polygon width="0.254" layer="16" isolate="1.27">
+<vertex x="0" y="0"/>
+<vertex x="0" y="30.48"/>
+<vertex x="40.64" y="30.48"/>
+<vertex x="40.64" y="0"/>
+</polygon>
 </signal>
 <signal name="N$1">
@@
 <wire x1="17.78" y1="16.51" x2="17.78" y2="19.05" width="1.27" layer="16"/>
 <wire x1="33.02" y1="16.51" x2="25.4" y2="16.51" width="1.27" layer="16"/>
-<wire x1="38.1" y1="16.51" x2="38.1" y2="12.7" width="0" layer="19" extent="1-16"/>
-<wire x1="38.1" y1="12.7" x2="38.1" y2="11.43" width="0" layer="19" extent="16-16"/>
+<wire x1="38.1" y1="6.35" x2="38.1" y2="11.43" width="0" layer="19" extent="1-1"/>
 <wire x1="29.21" y1="16.51" x2="33.02" y2="16.51" width="0" layer="19" extent="1-1"/>
 </signal>

Commit message: ...
Parts:
- moved R3 8.03 mm to (2.54, 21.6), turned to 90 degrees
- moved R2 2.54 mm to (17.8, 26.7)
Routing:
- net N$10: track 10.2 -> 20.3 mm
- net N$11: track 12.7 -> 15.2 mm
- net VCC: track 78.7 -> 81.3 mm
Changed lines of the file:
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@@
 <layer number="37" name="tTest" color="7" fill="1" visible="no" active="yes"/>
 <layer number="38" name="bTest" color="7" fill="1" visible="no" active="yes"/>
-<layer number="39" name="tKeepout" color="4" fill="11" visible="yes" active="yes"/>
-<layer number="40" name="bKeepout" color="1" fill="11" visible="yes" active="yes"/>
-<layer number="41" name="tRestrict" color="4" fill="10" visible="yes" active="yes"/>
-<layer number="42" name="bRestrict" color="1" fill="10" visible="yes" active="yes"/>
+<layer number="39" name="tKeepout" color="4" fill="11" visible="no" active="yes"/>
+<layer number="40" name="bKeepout" color="1" fill="11" visible="no" active="yes"/>
+<layer number="41" name="tRestrict" color="4" fill="10" visible="no" active="yes"/>
+<layer number="42" name="bRestrict" color="1" fill="10" visible="no" active="yes"/>
 <layer number="43" name="vRestrict" color="2" fill="10" visible="yes" active="yes"/>
 <layer number="44" name="Drills" color="7" fill="1" visible="no" active="yes"/>
@@
 <layer number="46" name="Milling" color="3" fill="1" visible="no" active="yes"/>
 <layer number="47" name="Measures" color="7" fill="1" visible="no" active="yes"/>
-<layer number="48" name="Document" color="7" fill="1" visible="yes" active="yes"/>
-<layer number="49" name="Reference" color="7" fill="1" visible="yes" active="yes"/>
+<layer number="48" name="Document" color="7" fill="1" visible="no" active="yes"/>
+<layer number="49" name="Reference" color="7" fill="1" visible="no" active="yes"/>
 <layer number="51" name="tDocu" color="7" fill="1" visible="yes" active="yes"/>
 <layer number="52" name="bDocu" color="7" fill="1" visible="yes" active="yes"/>
@@
 <element name="R10" library="r" package="0204/10" value="1k" x="30.48" y="8.89"/>
 <element name="R11" library="r" package="0204/10" value="1k" x="30.48" y="3.81"/>
-<element name="R2" library="r" package="0204/10" value="12k" x="20.32" y="26.67"/>
-<element name="R3" library="r" package="0204/10" value="220" x="10.16" y="24.13"/>
+<element name="R2" library="r" package="0204/10" value="12k" x="17.78" y="26.67"/>
+<element name="R3" library="r" package="0204/10" value="220" x="2.54" y="21.59" rot="R90"/>
 <element name="R4" library="r" package="0204/10" value="220" x="5.08" y="16.51" rot="R90"/>
 <element name="R5" library="r" package="0204/10" value="220" x="7.62" y="8.89" rot="R180"/>
@@
 <contactref element="R3" pad="2"/>
 <contactref element="IC1" pad="4"/>
-<wire x1="15.24" y1="26.67" x2="15.24" y2="24.13" width="1.27" layer="16"/>
+<wire x1="12.7" y1="26.67" x2="2.54" y2="26.67" width="1.27" layer="16"/>
+<wire x1="12.7" y1="26.67" x2="15.24" y2="26.67" width="1.27" layer="16"/>
 <wire x1="15.24" y1="26.67" x2="15.24" y2="19.05" width="1.27" layer="16"/>
 </signal>
@@
 <contactref element="R3" pad="1"/>
 <contactref element="R4" pad="2"/>
-<wire x1="10.16" y1="19.05" x2="10.16" y2="24.13" width="1.27" layer="16"/>
-<wire x1="5.08" y1="21.59" x2="5.08" y2="24.13" width="1.27" layer="16"/>
-<wire x1="5.08" y1="24.13" x2="10.16" y2="24.13" width="1.27" layer="16"/>
+<wire x1="10.16" y1="19.05" x2="10.16" y2="21.59" width="1.27" layer="16"/>
+<wire x1="5.08" y1="21.59" x2="2.54" y2="21.59" width="1.27" layer="16"/>
+<wire x1="2.54" y1="16.51" x2="2.54" y2="21.59" width="1.27" layer="16"/>
+<wire x1="5.08" y1="21.59" x2="10.16" y2="21.59" width="1.27" layer="16"/>
 </signal>
 <signal name="N$12">
@@
 <wire x1="38.1" y1="16.51" x2="38.1" y2="21.59" width="1.27" layer="16"/>
 <wire x1="17.78" y1="19.05" x2="17.78" y2="26.67" width="1.27" layer="16"/>
-<wire x1="17.78" y1="26.67" x2="25.4" y2="26.67" width="1.27" layer="16"/>
-<wire x1="25.4" y1="26.67" x2="38.1" y2="26.67" width="1.27" layer="16"/>
+<wire x1="17.78" y1="26.67" x2="22.86" y2="26.67" width="1.27" layer="16"/>
+<wire x1="22.86" y1="26.67" x2="38.1" y2="26.67" width="1.27" layer="16"/>
 <wire x1="38.1" y1="26.67" x2="38.1" y2="21.59" width="1.27" layer="16"/>
 <wire x1="22.86" y1="21.59" x2="27.94" y2="21.59" width="1.27" layer="16"/>
 <wire x1="27.94" y1="21.59" x2="27.94" y2="26.67" width="1.27" layer="16"/>
-<wire x1="27.94" y1="26.67" x2="25.4" y2="26.67" width="1.27" layer="16"/>
+<wire x1="27.94" y1="26.67" x2="22.86" y2="26.67" width="1.27" layer="16"/>
 <contactref element="PWR" pad="2"/>
 <contactref element="C2" pad="1"/>
