File: eagle/AudioPreAmp-LM741.brd (EAGLE design)
At the start: 30.5 x 22.9 mm, 14 parts, among them IC1 LM741

Commit message: ...
Changed lines of the file:
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@@
 <contactref element="R2" pad="A"/>
 <contactref element="R3" pad="2"/>
-<wire x1="12.7" y1="5.08" x2="10.16" y2="5.08" width="0.6096" layer="16"/>
+<wire x1="12.7" y1="5.08" x2="10.16" y2="5.08" width="1.27" layer="16"/>
 </signal>
 <signal name="N$3">
@@
 <contactref element="R1" pad="2"/>
 <contactref element="IC1" pad="2"/>
-<wire x1="10.16" y1="15.24" x2="10.16" y2="12.7" width="0.6096" layer="16"/>
-<wire x1="10.16" y1="12.7" x2="12.7" y2="12.7" width="0.6096" layer="16"/>
-<wire x1="10.16" y1="15.24" x2="10.16" y2="17.78" width="0.6096" layer="16"/>
-<wire x1="10.16" y1="17.78" x2="12.7" y2="17.78" width="0.6096" layer="16"/>
+<wire x1="10.16" y1="15.24" x2="10.16" y2="12.7" width="1.27" layer="16"/>
+<wire x1="10.16" y1="12.7" x2="12.7" y2="12.7" width="1.27" layer="16"/>
+<wire x1="10.16" y1="15.24" x2="10.16" y2="17.78" width="1.27" layer="16"/>
+<wire x1="10.16" y1="17.78" x2="12.7" y2="17.78" width="1.27" layer="16"/>
 </signal>
 <signal name="N$2">
 <contactref element="R1" pad="1"/>
 <contactref element="C1" pad="+"/>
-<wire x1="2.54" y1="17.78" x2="2.54" y2="10.16" width="0.6096" layer="16"/>
+<wire x1="2.54" y1="17.78" x2="2.54" y2="10.16" width="1.27" layer="16"/>
 </signal>
 <signal name="VCC">
@@
 <contactref element="C5" pad="1"/>
 <contactref element="C4" pad="+"/>
-<wire x1="15.24" y1="17.78" x2="15.24" y2="20.32" width="0.6096" layer="16"/>
-<wire x1="15.24" y1="20.32" x2="17.78" y2="20.32" width="0.6096" layer="16"/>
-<wire x1="17.78" y1="20.32" x2="22.86" y2="20.32" width="0.6096" layer="16"/>
-<wire x1="22.86" y1="20.32" x2="27.94" y2="20.32" width="0.6096" layer="16"/>
-<wire x1="15.24" y1="17.78" x2="15.24" y2="15.24" width="0.6096" layer="16"/>
-<wire x1="15.24" y1="15.24" x2="15.24" y2="12.7" width="0.6096" layer="16"/>
-<wire x1="15.24" y1="12.7" x2="20.32" y2="12.7" width="0.6096" layer="16"/>
+<wire x1="15.24" y1="17.78" x2="15.24" y2="20.32" width="1.27" layer="16"/>
+<wire x1="15.24" y1="20.32" x2="17.78" y2="20.32" width="1.27" layer="16"/>
+<wire x1="17.78" y1="20.32" x2="22.86" y2="20.32" width="1.27" layer="16"/>
+<wire x1="22.86" y1="20.32" x2="27.94" y2="20.32" width="1.27" layer="16"/>
+<wire x1="15.24" y1="17.78" x2="15.24" y2="15.24" width="1.27" layer="16"/>
+<wire x1="15.24" y1="15.24" x2="15.24" y2="12.7" width="1.27" layer="16"/>
+<wire x1="15.24" y1="12.7" x2="20.32" y2="12.7" width="1.27" layer="16"/>
 </signal>
 <signal name="GND">
@@
 <contactref element="C5" pad="2"/>
 <contactref element="C4" pad="-"/>
-<wire x1="7.62" y1="2.54" x2="2.54" y2="2.54" width="0.6096" layer="16"/>
-<wire x1="5.08" y1="12.7" x2="5.08" y2="2.54" width="0.6096" layer="16"/>
-<wire x1="5.08" y1="2.54" x2="7.62" y2="2.54" width="0.6096" layer="16"/>
-<wire x1="7.62" y1="2.54" x2="15.24" y2="2.54" width="0.6096" layer="16"/>
-<wire x1="12.7" y1="7.62" x2="15.24" y2="7.62" width="0.6096" layer="16"/>
-<wire x1="15.24" y1="7.62" x2="15.24" y2="2.54" width="0.6096" layer="16"/>
-<wire x1="15.24" y1="2.54" x2="25.4" y2="2.54" width="0.6096" layer="16"/>
-<wire x1="20.32" y1="17.78" x2="22.86" y2="17.78" width="0.6096" layer="16"/>
-<wire x1="27.94" y1="3.81" x2="27.94" y2="2.54" width="0.6096" layer="16"/>
-<wire x1="27.94" y1="2.54" x2="25.4" y2="2.54" width="0.6096" layer="16"/>
+<wire x1="7.62" y1="2.54" x2="2.54" y2="2.54" width="1.27" layer="16"/>
+<wire x1="5.08" y1="12.7" x2="5.08" y2="2.54" width="1.27" layer="16"/>
+<wire x1="5.08" y1="2.54" x2="7.62" y2="2.54" width="1.27" layer="16"/>
+<wire x1="7.62" y1="2.54" x2="15.24" y2="2.54" width="1.27" layer="16"/>
+<wire x1="12.7" y1="7.62" x2="15.24" y2="7.62" width="1.27" layer="16"/>
+<wire x1="15.24" y1="7.62" x2="15.24" y2="2.54" width="1.27" layer="16"/>
+<wire x1="15.24" y1="2.54" x2="25.4" y2="2.54" width="1.27" layer="16"/>
+<wire x1="20.32" y1="17.78" x2="22.86" y2="17.78" width="1.27" layer="16"/>
+<wire x1="27.94" y1="3.81" x2="27.94" y2="2.54" width="1.27" layer="16"/>
+<wire x1="27.94" y1="2.54" x2="25.4" y2="2.54" width="1.27" layer="16"/>
 <via x="25.4" y="2.54" extent="1-16" drill="0.6" shape="square"/>
-<wire x1="25.4" y1="2.54" x2="25.4" y2="17.78" width="0.6096" layer="1"/>
+<wire x1="25.4" y1="2.54" x2="25.4" y2="17.78" width="1.27" layer="1"/>
 <via x="25.4" y="17.78" extent="1-16" drill="0.6" shape="square"/>
-<wire x1="22.86" y1="17.78" x2="25.4" y2="17.78" width="0.6096" layer="16"/>
-<wire x1="25.4" y1="17.78" x2="27.94" y2="17.78" width="0.6096" layer="16"/>
+<wire x1="22.86" y1="17.78" x2="25.4" y2="17.78" width="1.27" layer="16"/>
+<wire x1="25.4" y1="17.78" x2="27.94" y2="17.78" width="1.27" layer="16"/>
 </signal>
 <signal name="N$4">
@@
 <contactref element="R5" pad="1"/>
 <contactref element="IC1" pad="3"/>
-<wire x1="7.62" y1="12.7" x2="7.62" y2="15.24" width="0.6096" layer="16"/>
-<wire x1="7.62" y1="15.24" x2="5.08" y2="15.24" width="0.6096" layer="16"/>
-<wire x1="7.62" y1="20.32" x2="7.62" y2="12.7" width="0.6096" layer="16"/>
-<wire x1="7.62" y1="12.7" x2="7.62" y2="10.16" width="0.6096" layer="16"/>
-<wire x1="7.62" y1="10.16" x2="12.7" y2="10.16" width="0.6096" layer="16"/>
+<wire x1="7.62" y1="12.7" x2="7.62" y2="15.24" width="1.27" layer="16"/>
+<wire x1="7.62" y1="15.24" x2="5.08" y2="15.24" width="1.27" layer="16"/>
+<wire x1="7.62" y1="20.32" x2="7.62" y2="12.7" width="1.27" layer="16"/>
+<wire x1="7.62" y1="12.7" x2="7.62" y2="10.16" width="1.27" layer="16"/>
+<wire x1="7.62" y1="10.16" x2="12.7" y2="10.16" width="1.27" layer="16"/>
 </signal>
 <signal name="N$7">
 <contactref element="C1" pad="-"/>
 <contactref element="IN" pad="2"/>
-<wire x1="2.54" y1="5.08" x2="2.54" y2="7.62" width="0.6096" layer="16"/>
+<wire x1="2.54" y1="5.08" x2="2.54" y2="7.62" width="1.27" layer="16"/>
 </signal>
 <signal name="N$5">
 <contactref element="C2" pad="-"/>
 <contactref element="OUT" pad="2"/>
-<wire x1="27.94" y1="7.62" x2="27.94" y2="5.08" width="0.6096" layer="16"/>
+<wire x1="27.94" y1="7.62" x2="27.94" y2="5.08" width="1.27" layer="16"/>
 </signal>
 <signal name="N$8">
@@
 <contactref element="C2" pad="+"/>
 <contactref element="R2" pad="E"/>
-<wire x1="27.94" y1="10.16" x2="17.78" y2="10.16" width="0.6096" layer="16"/>
-<wire x1="17.78" y1="10.16" x2="17.78" y2="5.08" width="0.6096" layer="16"/>
-<wire x1="22.86" y1="5.08" x2="17.78" y2="5.08" width="0.6096" layer="16"/>
+<wire x1="27.94" y1="10.16" x2="17.78" y2="10.16" width="1.27" layer="16"/>
+<wire x1="17.78" y1="10.16" x2="17.78" y2="5.08" width="1.27" layer="16"/>
+<wire x1="22.86" y1="5.08" x2="17.78" y2="5.08" width="1.27" layer="16"/>
 <wire x1="17.78" y1="10.16" x2="20.32" y2="10.16" width="0" layer="19" extent="16-16"/>
 </signal>

Commit message: ...
Routing:
- added copper zone on layer 16, net GND
Other:
- board outline removed
Changed lines of the file:
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@@
 <?xml version="1.0" encoding="utf-8"?>
 <!DOCTYPE eagle SYSTEM "eagle.dtd">
-<eagle version="7.6.0">
+<eagle version="7.7.0">
 <drawing>
 <settings>
@@
 <board>
 <plain>
-<wire x1="0" y1="0" x2="30.48" y2="0" width="0" layer="20"/>
-<wire x1="30.48" y1="0" x2="30.48" y2="22.86" width="0" layer="20"/>
-<wire x1="30.48" y1="22.86" x2="0" y2="22.86" width="0" layer="20"/>
-<wire x1="0" y1="22.86" x2="0" y2="0" width="0" layer="20"/>
+<wire x1="0" y1="0" x2="30.48" y2="0" width="0" layer="47"/>
+<wire x1="30.48" y1="0" x2="30.48" y2="22.86" width="0" layer="47"/>
+<wire x1="30.48" y1="22.86" x2="0" y2="22.86" width="0" layer="47"/>
+<wire x1="0" y1="22.86" x2="0" y2="0" width="0" layer="47"/>
 </plain>
 <attributes>
@@
 <wire x1="22.86" y1="17.78" x2="25.4" y2="17.78" width="1.27" layer="16"/>
 <wire x1="25.4" y1="17.78" x2="27.94" y2="17.78" width="1.27" layer="16"/>
+<polygon width="0.254" layer="16" isolate="1.27">
+<vertex x="0" y="0"/>
+<vertex x="30.48" y="0"/>
+<vertex x="30.48" y="22.86"/>
+<vertex x="0" y="22.86"/>
+</polygon>
 </signal>
 <signal name="N$4">
