File: eagle/Simple-Bug-BC557.brd (EAGLE design)
At the start: 25.4 x 20.3 mm, 13 parts, among them T1 BC557

Commit message: ...
Parts:
- turned C1 to 180 degrees
- turned C2 to 90 degrees
- turned C3 to 90 degrees
- turned C4 to 0 degrees
- turned R1 to 0 degrees
- turned R2 to 90 degrees
- turned R3 to 90 degrees
- turned T1 to 180 degrees
Connections:
- net +UB: now also +.1, R1.2; no longer +.P, R1.1
- net GND: now also C1.3, R2.1, R3.1, ̶̶.1; no longer C1.2, R2.2, R3.2, ̶̶.P
- net N$1: now also ANT1.1, C1.2; no longer ANT1.P, C1.3
- net N$3: now also R1.1; no longer R1.2
- net N$5: now also R3.2; no longer R3.1
- net N$6: now also R2.2; no longer R2.1
Changed lines of the file:
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@@
 <?xml version="1.0" encoding="utf-8"?>
 <!DOCTYPE eagle SYSTEM "eagle.dtd">
-<eagle version="7.7.0">
+<eagle version="7.6.0">
 <drawing>
 <settings>
@@
 </variantdefs>
 <classes>
-<class number="0" name="default" width="0.4064" drill="0">
+<class number="0" name="default" width="0.6096" drill="0">
 </class>
 </classes>
@@
 </autorouter>
 <elements>
-<element name="C2" library="c" package="C050-020X036" value="4.7pF" x="15.24" y="12.7" smashed="yes" rot="R180">
-<attribute name="NAME" x="16.764" y="13.462" size="0.8128" layer="25" align="center-left"/>
-<attribute name="VALUE" x="16.764" y="11.938" size="0.8128" layer="27" align="center-left"/>
+<element name="C2" library="c" package="C050-020X036" value="4.7pF" x="15.24" y="12.7" smashed="yes" rot="R90">
+<attribute name="NAME" x="16.002" y="11.176" size="0.8128" layer="25" rot="R270" align="center-left"/>
+<attribute name="VALUE" x="14.478" y="11.176" size="0.8128" layer="27" rot="R270" align="center-left"/>
 </element>
-<element name="C3" library="c" package="C050-020X036" value="1nF" x="7.62" y="15.24" rot="R180"/>
+<element name="C3" library="c" package="C050-020X036" value="1nF" x="7.62" y="15.24" rot="R90"/>
 <element name="L1" library="r" package="L-04/7" value="1uH" x="19.05" y="6.35"/>
-<element name="R2" library="r" package="0202/5" value="22k" x="5.08" y="5.08" smashed="yes" rot="R180">
-<attribute name="VALUE" x="4.064" y="5.08" size="0.6096" layer="27" ratio="10" rot="R90" align="bottom-center"/>
-<attribute name="NAME" x="5.08" y="5.08" size="0.8128" layer="25" ratio="10" rot="R90" align="center"/>
-</element>
-<element name="R3" library="r" package="0202/5" value="47k" x="7.62" y="5.08" smashed="yes" rot="R180">
-<attribute name="VALUE" x="6.604" y="5.08" size="0.6096" layer="27" ratio="10" rot="R90" align="bottom-center"/>
-<attribute name="NAME" x="7.62" y="5.08" size="0.8128" layer="25" ratio="10" rot="R90" align="center"/>
-</element>
-<element name="T1" library="t" package="TO92-CBE-A" value="BC557" x="12.7" y="12.7" smashed="yes">
-<attribute name="NAME" x="11.684" y="12.7" size="0.8128" layer="25" ratio="10" rot="R90" align="center"/>
-<attribute name="VALUE" x="13.589" y="12.7" size="0.8128" layer="27" ratio="10" rot="R90" align="center"/>
+<element name="R2" library="r" package="0202/5" value="22k" x="5.08" y="5.08" rot="R90"/>
+<element name="R3" library="r" package="0202/5" value="47k" x="7.62" y="5.08" rot="R90"/>
+<element name="T1" library="t" package="TO92-CBE-A" value="BC557" x="12.7" y="12.7" smashed="yes" rot="R180">
+<attribute name="NAME" x="13.716" y="12.7" size="0.8128" layer="25" ratio="10" rot="R270" align="center"/>
+<attribute name="VALUE" x="11.811" y="12.7" size="0.8128" layer="27" ratio="10" rot="R270" align="center"/>
 </element>
 <element name="ECM" library="ECM" package="ECM-5" value="ECM-5" x="2.54" y="13.97"/>
-<element name="C1" library="cap-trim" package="TRIM808-45" value="C-TR-PH20127" x="12.7" y="5.08" smashed="yes">
-<attribute name="NAME" x="15.748" y="7.62" size="0.762" layer="25"/>
-<attribute name="VALUE" x="12.7" y="1.016" size="0.6096" layer="27" align="top-center"/>
+<element name="C1" library="cap-trim" package="TRIM808-45" value="C-TR-PH20127" x="12.7" y="5.08" smashed="yes" rot="R180">
+<attribute name="NAME" x="9.652" y="2.54" size="0.762" layer="25" rot="R180"/>
+<attribute name="VALUE" x="12.7" y="9.144" size="0.6096" layer="27" rot="R180" align="top-center"/>
 </element>
-<element name="R1" library="r" package="0202V" value="" x="17.78" y="16.51" smashed="yes" rot="R180">
-<attribute name="NAME" x="18.796" y="16.51" size="0.8128" layer="25" ratio="10" align="center-left"/>
-<attribute name="VALUE" x="17.526" y="17.018" size="0.9906" layer="27" ratio="10" rot="R180"/>
+<element name="R1" library="r" package="0202V" value="" x="17.78" y="16.51" smashed="yes">
+<attribute name="NAME" x="16.764" y="16.51" size="0.8128" layer="25" ratio="10" rot="R180" align="center-left"/>
+<attribute name="VALUE" x="18.034" y="16.002" size="0.9906" layer="27" ratio="10"/>
 </element>
-<element name="C4" library="c" package="E2,5-3" value="" x="6.35" y="10.16" rot="R180"/>
+<element name="C4" library="c" package="E2,5-3" value="" x="6.35" y="10.16"/>
 <element name="+" library="pad" package="SPAD" value="SPAD" x="22.86" y="17.78"/>
 <element name="̶̶" library="pad" package="SPAD" value="SPAD" x="22.86" y="2.54"/>
@@
 <contactref element="T1" pad="C"/>
 <contactref element="C2" pad="1"/>
-<contactref element="ANT1" pad="P"/>
-<wire x1="15.24" y1="10.16" x2="12.7" y2="10.16" width="0.4064" layer="16"/>
-<contactref element="C1" pad="3"/>
-<wire x1="12.7" y1="10.16" x2="12.7" y2="7.62" width="0.4064" layer="16"/>
-<wire x1="12.7" y1="7.62" x2="10.16" y2="7.62" width="0.4064" layer="16"/>
+<contactref element="ANT1" pad="1"/>
+<wire x1="15.24" y1="10.16" x2="12.7" y2="10.16" width="0.6096" layer="16"/>
+<contactref element="C1" pad="2"/>
+<wire x1="12.7" y1="10.16" x2="12.7" y2="7.62" width="0.6096" layer="16"/>
+<wire x1="12.7" y1="7.62" x2="15.24" y2="7.62" width="0.6096" layer="16"/>
 <contactref element="L1" pad="1"/>
-<wire x1="15.24" y1="10.16" x2="17.78" y2="10.16" width="0.4064" layer="16"/>
-<wire x1="17.78" y1="10.16" x2="22.86" y2="10.16" width="0.4064" layer="16"/>
+<wire x1="15.24" y1="10.16" x2="17.78" y2="10.16" width="0.6096" layer="16"/>
+<wire x1="17.78" y1="10.16" x2="22.86" y2="10.16" width="0.6096" layer="16"/>
 </signal>
 <signal name="N$3">
 <contactref element="C2" pad="2"/>
 <contactref element="T1" pad="E"/>
-<contactref element="R1" pad="2"/>
-<wire x1="15.24" y1="15.24" x2="17.78" y2="15.24" width="0.4064" layer="16"/>
-<wire x1="15.24" y1="15.24" x2="12.7" y2="15.24" width="0.4064" layer="16"/>
+<contactref element="R1" pad="1"/>
+<wire x1="15.24" y1="15.24" x2="17.78" y2="15.24" width="0.6096" layer="16"/>
+<wire x1="15.24" y1="15.24" x2="12.7" y2="15.24" width="0.6096" layer="16"/>
 </signal>
 <signal name="N$5">
-<contactref element="R3" pad="1"/>
+<contactref element="R3" pad="2"/>
 <contactref element="C3" pad="1"/>
 <contactref element="T1" pad="B"/>
 <contactref element="C4" pad="-"/>
-<wire x1="10.16" y1="12.7" x2="7.62" y2="12.7" width="0.4064" layer="16"/>
-<wire x1="7.62" y1="10.16" x2="7.62" y2="7.62" width="0.4064" layer="16"/>
-<wire x1="7.62" y1="10.16" x2="7.62" y2="12.7" width="0.4064" layer="16"/>
+<wire x1="10.16" y1="12.7" x2="7.62" y2="12.7" width="0.6096" layer="16"/>
+<wire x1="7.62" y1="10.16" x2="7.62" y2="7.62" width="0.6096" layer="16"/>
+<wire x1="7.62" y1="10.16" x2="7.62" y2="12.7" width="0.6096" layer="16"/>
 </signal>
 <signal name="N$6">
-<contactref element="R2" pad="1"/>
+<contactref element="R2" pad="2"/>
 <contactref element="ECM" pad="2"/>
 <contactref element="C4" pad="+"/>
-<wire x1="5.08" y1="10.16" x2="2.54" y2="10.16" width="0.4064" layer="16"/>
-<wire x1="2.54" y1="10.16" x2="2.54" y2="12.7" width="0.4064" layer="16"/>
-<wire x1="5.08" y1="10.16" x2="5.08" y2="7.62" width="0.4064" layer="16"/>
+<wire x1="5.08" y1="10.16" x2="2.54" y2="10.16" width="0.6096" layer="16"/>
+<wire x1="2.54" y1="10.16" x2="2.54" y2="12.7" width="0.6096" layer="16"/>
+<wire x1="5.08" y1="10.16" x2="5.08" y2="7.62" width="0.6096" layer="16"/>
 </signal>
 <signal name="GND">
-<contactref element="R3" pad="2"/>
-<contactref element="R2" pad="2"/>
-<contactref element="C1" pad="2"/>
-<wire x1="5.08" y1="2.54" x2="7.62" y2="2.54" width="0.4064" layer="16"/>
-<wire x1="7.62" y1="2.54" x2="10.16" y2="2.54" width="0.4064" layer="16"/>
+<contactref element="R3" pad="1"/>
+<contactref element="R2" pad="1"/>
+<contactref element="C1" pad="3"/>
+<wire x1="5.08" y1="2.54" x2="7.62" y2="2.54" width="0.6096" layer="16"/>
+<wire x1="7.62" y1="2.54" x2="15.24" y2="2.54" width="0.6096" layer="16"/>
 <contactref element="L1" pad="2"/>
-<wire x1="10.16" y1="2.54" x2="20.32" y2="2.54" width="0.4064" layer="16"/>
-<contactref element="̶̶" pad="P"/>
-<wire x1="20.32" y1="2.54" x2="22.86" y2="2.54" width="0.4064" layer="16"/>
+<wire x1="15.24" y1="2.54" x2="20.32" y2="2.54" width="0.6096" layer="16"/>
+<contactref element="̶̶" pad="1"/>
+<wire x1="20.32" y1="2.54" x2="22.86" y2="2.54" width="0.6096" layer="16"/>
 </signal>
 <signal name="+UB">
 <contactref element="C3" pad="2"/>
 <contactref element="ECM" pad="1"/>
-<contactref element="R1" pad="1"/>
-<wire x1="2.54" y1="17.78" x2="2.54" y2="15.24" width="0.4064" layer="16"/>
-<wire x1="7.62" y1="17.78" x2="2.54" y2="17.78" width="0.4064" layer="16"/>
-<wire x1="17.78" y1="17.78" x2="7.62" y2="17.78" width="0.4064" layer="16"/>
-<contactref element="+" pad="P"/>
-<wire x1="17.78" y1="17.78" x2="22.86" y2="17.78" width="0.4064" layer="16"/>
+<contactref element="R1" pad="2"/>
+<wire x1="7.62" y1="17.78" x2="2.54" y2="17.78" width="0.6096" layer="16"/>
+<wire x1="2.54" y1="17.78" x2="2.54" y2="15.24" width="0.6096" layer="16"/>
+<wire x1="17.78" y1="17.78" x2="7.62" y2="17.78" width="0.6096" layer="16"/>
+<contactref element="+" pad="1"/>
+<wire x1="17.78" y1="17.78" x2="22.86" y2="17.78" width="0.6096" layer="16"/>
 </signal>
 </signals>

Commit message: ...
Changed lines of the file:
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@@
 <contactref element="C2" pad="1"/>
 <contactref element="ANT1" pad="1"/>
-<wire x1="15.24" y1="10.16" x2="12.7" y2="10.16" width="0.6096" layer="16"/>
+<wire x1="15.24" y1="10.16" x2="12.7" y2="10.16" width="1.27" layer="16"/>
 <contactref element="C1" pad="2"/>
-<wire x1="12.7" y1="10.16" x2="12.7" y2="7.62" width="0.6096" layer="16"/>
-<wire x1="12.7" y1="7.62" x2="15.24" y2="7.62" width="0.6096" layer="16"/>
+<wire x1="12.7" y1="10.16" x2="12.7" y2="7.62" width="1.27" layer="16"/>
+<wire x1="12.7" y1="7.62" x2="15.24" y2="7.62" width="1.27" layer="16"/>
 <contactref element="L1" pad="1"/>
-<wire x1="15.24" y1="10.16" x2="17.78" y2="10.16" width="0.6096" layer="16"/>
-<wire x1="17.78" y1="10.16" x2="22.86" y2="10.16" width="0.6096" layer="16"/>
+<wire x1="15.24" y1="10.16" x2="17.78" y2="10.16" width="1.27" layer="16"/>
+<wire x1="17.78" y1="10.16" x2="22.86" y2="10.16" width="1.27" layer="16"/>
 </signal>
 <signal name="N$3">
@@
 <contactref element="T1" pad="E"/>
 <contactref element="R1" pad="1"/>
-<wire x1="15.24" y1="15.24" x2="17.78" y2="15.24" width="0.6096" layer="16"/>
-<wire x1="15.24" y1="15.24" x2="12.7" y2="15.24" width="0.6096" layer="16"/>
+<wire x1="15.24" y1="15.24" x2="17.78" y2="15.24" width="1.27" layer="16"/>
+<wire x1="15.24" y1="15.24" x2="12.7" y2="15.24" width="1.27" layer="16"/>
 </signal>
 <signal name="N$5">
@@
 <contactref element="T1" pad="B"/>
 <contactref element="C4" pad="-"/>
-<wire x1="10.16" y1="12.7" x2="7.62" y2="12.7" width="0.6096" layer="16"/>
-<wire x1="7.62" y1="10.16" x2="7.62" y2="7.62" width="0.6096" layer="16"/>
-<wire x1="7.62" y1="10.16" x2="7.62" y2="12.7" width="0.6096" layer="16"/>
+<wire x1="10.16" y1="12.7" x2="7.62" y2="12.7" width="1.27" layer="16"/>
+<wire x1="7.62" y1="10.16" x2="7.62" y2="7.62" width="1.27" layer="16"/>
+<wire x1="7.62" y1="10.16" x2="7.62" y2="12.7" width="1.27" layer="16"/>
 </signal>
 <signal name="N$6">
@@
 <contactref element="ECM" pad="2"/>
 <contactref element="C4" pad="+"/>
-<wire x1="5.08" y1="10.16" x2="2.54" y2="10.16" width="0.6096" layer="16"/>
-<wire x1="2.54" y1="10.16" x2="2.54" y2="12.7" width="0.6096" layer="16"/>
-<wire x1="5.08" y1="10.16" x2="5.08" y2="7.62" width="0.6096" layer="16"/>
+<wire x1="5.08" y1="10.16" x2="2.54" y2="10.16" width="1.27" layer="16"/>
+<wire x1="2.54" y1="10.16" x2="2.54" y2="12.7" width="1.27" layer="16"/>
+<wire x1="5.08" y1="10.16" x2="5.08" y2="7.62" width="1.27" layer="16"/>
 </signal>
 <signal name="GND">
@@
 <contactref element="R2" pad="1"/>
 <contactref element="C1" pad="3"/>
-<wire x1="5.08" y1="2.54" x2="7.62" y2="2.54" width="0.6096" layer="16"/>
-<wire x1="7.62" y1="2.54" x2="15.24" y2="2.54" width="0.6096" layer="16"/>
+<wire x1="5.08" y1="2.54" x2="7.62" y2="2.54" width="1.27" layer="16"/>
+<wire x1="7.62" y1="2.54" x2="15.24" y2="2.54" width="1.27" layer="16"/>
 <contactref element="L1" pad="2"/>
-<wire x1="15.24" y1="2.54" x2="20.32" y2="2.54" width="0.6096" layer="16"/>
+<wire x1="15.24" y1="2.54" x2="20.32" y2="2.54" width="1.27" layer="16"/>
 <contactref element="̶̶" pad="1"/>
-<wire x1="20.32" y1="2.54" x2="22.86" y2="2.54" width="0.6096" layer="16"/>
+<wire x1="20.32" y1="2.54" x2="22.86" y2="2.54" width="1.27" layer="16"/>
 </signal>
 <signal name="+UB">
@@
 <contactref element="ECM" pad="1"/>
 <contactref element="R1" pad="2"/>
-<wire x1="7.62" y1="17.78" x2="2.54" y2="17.78" width="0.6096" layer="16"/>
-<wire x1="2.54" y1="17.78" x2="2.54" y2="15.24" width="0.6096" layer="16"/>
-<wire x1="17.78" y1="17.78" x2="7.62" y2="17.78" width="0.6096" layer="16"/>
+<wire x1="7.62" y1="17.78" x2="2.54" y2="17.78" width="1.27" layer="16"/>
+<wire x1="2.54" y1="17.78" x2="2.54" y2="15.24" width="1.27" layer="16"/>
+<wire x1="17.78" y1="17.78" x2="7.62" y2="17.78" width="1.27" layer="16"/>
 <contactref element="+" pad="1"/>
-<wire x1="17.78" y1="17.78" x2="22.86" y2="17.78" width="0.6096" layer="16"/>
+<wire x1="17.78" y1="17.78" x2="22.86" y2="17.78" width="1.27" layer="16"/>
 </signal>
 </signals>

Commit message: ...
Routing:
- added copper zone on layer 16, net GND
Other:
- board outline removed
Changed lines of the file:
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@@
 <?xml version="1.0" encoding="utf-8"?>
 <!DOCTYPE eagle SYSTEM "eagle.dtd">
-<eagle version="7.6.0">
+<eagle version="7.7.0">
 <drawing>
 <settings>
@@
 <description>Simple FM Transmitter with Electret Microphone, based on PNP Transistor</description>
 <plain>
-<wire x1="25.4" y1="20.32" x2="0.02" y2="20.32" width="0" layer="20"/>
-<wire x1="0.02" y1="20.32" x2="0.02" y2="0" width="0" layer="20"/>
-<wire x1="0.02" y1="0" x2="25.4" y2="0" width="0" layer="20"/>
-<wire x1="25.4" y1="0" x2="25.4" y2="20.32" width="0" layer="20"/>
+<wire x1="25.4" y1="20.32" x2="0.02" y2="20.32" width="0" layer="47"/>
+<wire x1="0.02" y1="20.32" x2="0.02" y2="0" width="0" layer="47"/>
+<wire x1="0.02" y1="0" x2="25.4" y2="0" width="0" layer="47"/>
+<wire x1="25.4" y1="0" x2="25.4" y2="20.32" width="0" layer="47"/>
 </plain>
 <attributes>
@@
 <contactref element="̶̶" pad="1"/>
 <wire x1="20.32" y1="2.54" x2="22.86" y2="2.54" width="1.27" layer="16"/>
+<polygon width="0.254" layer="16" isolate="1.27" orphans="yes" thermals="no">
+<vertex x="0" y="0"/>
+<vertex x="0" y="20.32"/>
+<vertex x="25.4" y="20.32"/>
+<vertex x="25.4" y="0"/>
+</polygon>
 </signal>
 <signal name="+UB">

Commit message: ...
Parts:
- renumbered ̶̶ to @@@@
Changed lines of the file:
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@@
 <description language="de">&lt;b&gt;EAGLE Design Rules&lt;/b&gt;
 &lt;p&gt;
-Die Standard-Design-Rules sind so gewählt, dass sie ffür uuml;r
+Die Standard-Design-Rules sind so gew@@hlt, dass sie ff@@r uuml;r
 die meisten Anwendungen passen. Sollte ihre Platine
 besondere Anforderungen haben, treffen Sie die erforderlichen
@@
 <element name="C4" library="c" package="E2,5-3" value="" x="6.35" y="10.16"/>
 <element name="+" library="pad" package="SPAD" value="SPAD" x="22.86" y="17.78"/>
-<element name="̶̶" library="pad" package="SPAD" value="SPAD" x="22.86" y="2.54"/>
+<element name="@@@@" library="pad" package="SPAD" value="SPAD" x="22.86" y="2.54"/>
 <element name="ANT1" library="pad" package="SPAD" value="ANT" x="22.86" y="10.16"/>
 </elements>
@@
 <contactref element="L1" pad="2"/>
 <wire x1="15.24" y1="2.54" x2="20.32" y2="2.54" width="1.27" layer="16"/>
-<contactref element="̶̶" pad="1"/>
+<contactref element="@@@@" pad="1"/>
 <wire x1="20.32" y1="2.54" x2="22.86" y2="2.54" width="1.27" layer="16"/>
 <polygon width="0.254" layer="16" isolate="1.27" orphans="yes" thermals="no">
