File: eagle/EFM_VCF6c.sch (EAGLE design)
At the start: 69 parts, among them IC1 LM13700N, Q1 2N3904, Q2 2N3904, Q3 2N3906, Q4 2N3904, Q5 2N3906, U1 POWER

Commit message: ...
Parts:
- C1, C11, C12, C2, C5: value 10uF -> 10μF
- C10: value 220uF -> 220μF
- C3, C4, C6, C7, C8, C9: value 0.1uF -> 0.1μF
- CUTOFF, CUTOFF_INIT, CV1_LEVEL, CV2_LEVEL, IN1_LEVEL, IN2_LEVEL, R10, R11, R26, R30, R6, R7, R8, R9, RESONANCE: value 100k -> 100kΩ
- R12, R15, R17, R18, R19: value 1k -> 1kΩ
- R16: value 560k -> 560kΩ
- R20, R23, R28, R29: value 10k -> 10kΩ
- R22: value 470k -> 470kΩ
- R24, R25: value 220k -> 220kΩ
- R27: value 1M -> 1MΩ
- R31: value 220 -> 220Ω
- SCALE_TRIM: value 2k -> 2kΩ
