File: eagle/One-Transistor-FM-Super-Regen.sch (EAGLE design)
At the start: 19 parts, among them J1 SPAD+-+-, SW1 SW-SPST-SL-1P2T-H, T1 2N3904

Commit message: ...
Parts:
- R1: value 2.2kΩ -> 2.2kΩ
- VR1: value 10kΩ -> 10kΩ
- VR2: value 100kΩ -> 100kΩ
Changed lines of the file:
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@@
 <part name="C1" library="c" deviceset="C" device="025-015X024" value="5pF"/>
 <part name="L1" library="l" deviceset="L" device="04/7-V" value="4t"/>
-<part name="R1" library="r" deviceset="R" device="0204/10-V" value="2.2kΩ"/>
+<part name="R1" library="r" deviceset="R" device="0204/10-V" value="2.2kΩ"/>
 <part name="C2" library="c" deviceset="C" device="050-020X036/V" value="0.001"/>
-<part name="VR1" library="r" deviceset="POT" device="-TRIM" value="10kΩ"/>
+<part name="VR1" library="r" deviceset="POT" device="-TRIM" value="10kΩ"/>
 <part name="SW1" library="sw" deviceset="SW-SPST" device="-SL-1P2T-H"/>
 <part name="C3" library="c" deviceset="C-H" device="050-020X036" value="0.001"/>
@@
 <part name="S4" library="pad" deviceset="GND" device=""/>
 <part name="S5" library="pad" deviceset="GND" device=""/>
-<part name="VR2" library="r" deviceset="TRIM-2" device="-TR-3TO2" value="100kΩ"/>
+<part name="VR2" library="r" deviceset="TRIM-2" device="-TR-3TO2" value="100kΩ"/>
 <part name="S6" library="pad" deviceset="VCC_GND" device="PWR-R"/>
 <part name="J1" library="pad" deviceset="SPAD+-" device="+-"/>
