File: eagle/Simple-Bug-BC557.sch (EAGLE design)
At the start: 13 parts, among them T1 BC557

Commit message: ...
Parts:
- renumbered ̶̶ to @@@@
Changed lines of the file:
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@@
 <part name="C4" library="c" deviceset="CPOL" device="E2,5-3"/>
 <part name="+" library="pad" deviceset="SPAD" device=""/>
-<part name="̶̶" library="pad" deviceset="SPAD" device=""/>
+<part name="@@@@" library="pad" deviceset="SPAD" device=""/>
 <part name="ANT1" library="pad" deviceset="ANT" device=""/>
 </parts>
@@
 <instance part="C4" gate="1" x="13.97" y="38.1" rot="MR270"/>
 <instance part="+" gate="1" x="60.96" y="63.5" rot="MR180"/>
-<instance part="̶̶" gate="1" x="60.96" y="58.42" rot="MR180"/>
+<instance part="@@@@" gate="1" x="60.96" y="58.42" rot="MR180"/>
 <instance part="ANT1" gate="ANT" x="68.58" y="35.56" rot="MR0"/>
 </instances>
@@
 <segment>
 <pinref part="GND3" gate="1" pin="GND"/>
-<pinref part="̶̶" gate="1" pin="P$1"/>
+<pinref part="@@@@" gate="1" pin="P$1"/>
 <wire x1="68.58" y1="57.15" x2="68.58" y2="55.88" width="0.1524" layer="91"/>
 <wire x1="60.96" y1="58.42" x2="68.58" y2="58.42" width="0.1524" layer="91"/>

Commit message: ...
Parts:
- L1: value 1uH -> 1μH
- R2: value 22k -> 22kΩ
- R3: value 47k -> 47kΩ
Changed lines of the file:
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@@
 <parts>
 <part name="T1" library="t" deviceset="BC547" device="CBE-A" value="BC557"/>
-<part name="L1" library="r" deviceset="L" device="04/7" value="1uH"/>
+<part name="L1" library="r" deviceset="L" device="04/7" value="1μH"/>
 <part name="C2" library="c" deviceset="C" device="050-020X036" value="4.7pF"/>
 <part name="C3" library="c" deviceset="C" device="050-020X036" value="1nF"/>
-<part name="R2" library="r" deviceset="R" device="0202/5" value="22k"/>
-<part name="R3" library="r" deviceset="R" device="0202/5" value="47k"/>
+<part name="R2" library="r" deviceset="R" device="0202/5" value="22kΩ"/>
+<part name="R3" library="r" deviceset="R" device="0202/5" value="47kΩ"/>
 <part name="GND1" library="supply1" deviceset="GND" device=""/>
 <part name="SUPPLY1" library="supply2" deviceset="+UB" device=""/>
