File: eagle/Simple-NPN-Regen-Receiver.sch (EAGLE design)
At the start: 9 parts, among them T1 2N2222, T2 2N3904

Commit message: ...
Parts:
- added AF: HPORT, pad:HPORT
- C1: value 1 - 20p -> 1 - 20pF
- C2: value 1n -> 1nF
- L1: value (none) -> 0.2μH
- R1: value 47 -> 47Ω
- R2: value 100K -> 100kΩ
- R3: value 10k -> 10kΩ
Connections:
- net N$5: now also AF.P$1
Other:
- moved on the sheet: C2, R1, R2, R3, T2
