File: eagle/AM-Crystal-RX-LM324.sch (EAGLE design)
At the start: 24 parts, among them IC2 LM324, SW1 SL-SW-1P-2T-H

Commit message: ...
Parts:
- renumbered +9V to 9V
Changed lines of the file:
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@@
 <part name="SP-" library="pad" deviceset="SPAD" device="" value="SPKR-"/>
 <part name="GND7" library="supply1" deviceset="GND" device=""/>
-<part name="+9V" library="pad" deviceset="SPAD" device="" value="BAT+"/>
+<part name="9V" library="pad" deviceset="SPAD" device="" value="BAT+"/>
 <part name="GND8" library="supply1" deviceset="GND" device=""/>
 <part name="GND" library="pad" deviceset="SPAD" device="" value="BAT-"/>
@@
 <instance part="SP-" gate="1" x="132.08" y="22.86" rot="R180"/>
 <instance part="GND7" gate="1" x="129.54" y="15.24"/>
-<instance part="+9V" gate="1" x="88.9" y="50.8" rot="R180"/>
+<instance part="9V" gate="1" x="88.9" y="50.8" rot="R180"/>
 <instance part="GND8" gate="1" x="81.28" y="40.64"/>
 <instance part="GND" gate="1" x="88.9" y="45.72" rot="R180"/>
@@
 <segment>
 <wire x1="86.36" y1="60.96" x2="86.36" y2="50.8" width="0.1524" layer="91"/>
-<pinref part="+9V" gate="1" pin="P$1"/>
+<pinref part="9V" gate="1" pin="P$1"/>
 <wire x1="86.36" y1="50.8" x2="88.9" y2="50.8" width="0.1524" layer="91"/>
 <wire x1="86.36" y1="60.96" x2="81.28" y2="60.96" width="0.1524" layer="91"/>

Commit message: ...
Parts:
- C5, C6: value 1uF -> 1μF
- C7, C8: value 100uF -> 100μF
- L1: value 0.15uH -> 0.15μH
- R1, R7: value 1M -> 1MΩ
- R2, R5: value 100k -> 100kΩ
- R3, R4: value 3.3k -> 3.3kΩ
- R6: value 100 -> 100Ω
Changed lines of the file:
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@@
 <parts>
 <part name="C1" library="cap-trim" deviceset="C-TR-PH20127" device="2222-808-2PIN" value="5-18pF"/>
-<part name="L1" library="r" deviceset="L-SHORT" device="04-5/5" value="0.15uH"/>
-<part name="R1" library="r" deviceset="R" device="0202/7-V" value="1M"/>
+<part name="L1" library="r" deviceset="L-SHORT" device="04-5/5" value="0.15μH"/>
+<part name="R1" library="r" deviceset="R" device="0202/7-V" value="1MΩ"/>
 <part name="C2" library="c" deviceset="C" device="050-025X075/V" value="10nF"/>
 <part name="GND1" library="supply1" deviceset="GND" device=""/>
@@
 <part name="C4" library="c" deviceset="C" device="050-024X044/V" value="330pF"/>
 <part name="GND2" library="supply1" deviceset="GND" device=""/>
-<part name="R2" library="r" deviceset="TRIM" device="" value="100k"/>
-<part name="R3" library="r" deviceset="R" device="0202/7" value="3.3k"/>
-<part name="R4" library="r" deviceset="R" device="0202/7-V" value="3.3k"/>
-<part name="R5" library="r" deviceset="R" device="0202/7-V" value="100k"/>
-<part name="R6" library="r" deviceset="R" device="0202/7-V" value="100"/>
-<part name="C5" library="c" deviceset="CPOL" device="E2,5-4/V" value="1uF"/>
-<part name="C6" library="c" deviceset="CPOL" device="E2,5-3/V" value="1uF"/>
-<part name="C7" library="c" deviceset="CPOL" device="E5-5/V" value="100uF"/>
+<part name="R2" library="r" deviceset="TRIM" device="" value="100kΩ"/>
+<part name="R3" library="r" deviceset="R" device="0202/7" value="3.3kΩ"/>
+<part name="R4" library="r" deviceset="R" device="0202/7-V" value="3.3kΩ"/>
+<part name="R5" library="r" deviceset="R" device="0202/7-V" value="100kΩ"/>
+<part name="R6" library="r" deviceset="R" device="0202/7-V" value="100Ω"/>
+<part name="C5" library="c" deviceset="CPOL" device="E2,5-4/V" value="1μF"/>
+<part name="C6" library="c" deviceset="CPOL" device="E2,5-3/V" value="1μF"/>
+<part name="C7" library="c" deviceset="CPOL" device="E5-5/V" value="100μF"/>
 <part name="SW1" library="sw" deviceset="SL-SW-1P-2T" device="-H"/>
 <part name="GND3" library="supply1" deviceset="GND" device=""/>
 <part name="GND4" library="supply1" deviceset="GND" device=""/>
 <part name="GND5" library="supply1" deviceset="GND" device=""/>
-<part name="R7" library="r" deviceset="R" device="0202/7-V" value="1M"/>
+<part name="R7" library="r" deviceset="R" device="0202/7-V" value="1MΩ"/>
 <part name="GND6" library="supply1" deviceset="GND" device=""/>
-<part name="C8" library="c" deviceset="CPOL" device="E2,5-5/V" value="100uF"/>
+<part name="C8" library="c" deviceset="CPOL" device="E2,5-5/V" value="100μF"/>
 <part name="SP+" library="pad" deviceset="SPAD" device="" value="SPKR+"/>
 <part name="SP-" library="pad" deviceset="SPAD" device="" value="SPKR-"/>

Commit message: ...
Parts:
- C1: device cap-trim:C-TR-PH201272222-808-2PIN -> cap-trim:C-TR-PH201272222-808-2PINB
Changed lines of the file:
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@@
 <grid distance="0.05" unitdist="inch" unit="inch" style="lines" multiple="2" display="yes" altdistance="4" altunitdist="inch" altunit="inch"/>
 <layers>
-<layer number="1" name="Top" color="4" fill="1" visible="no" active="no"/>
-<layer number="2" name="Route2" color="1" fill="3" visible="no" active="no"/>
-<layer number="3" name="Route3" color="4" fill="3" visible="no" active="no"/>
-<layer number="4" name="Route4" color="1" fill="4" visible="no" active="no"/>
-<layer number="5" name="Route5" color="4" fill="4" visible="no" active="no"/>
-<layer number="6" name="Route6" color="1" fill="8" visible="no" active="no"/>
-<layer number="7" name="Route7" color="4" fill="8" visible="no" active="no"/>
-<layer number="8" name="Route8" color="1" fill="2" visible="no" active="no"/>
-<layer number="9" name="Route9" color="4" fill="2" visible="no" active="no"/>
-<layer number="10" name="Route10" color="1" fill="7" visible="no" active="no"/>
-<layer number="11" name="Route11" color="4" fill="7" visible="no" active="no"/>
-<layer number="12" name="Route12" color="1" fill="5" visible="no" active="no"/>
-<layer number="13" name="Route13" color="4" fill="5" visible="no" active="no"/>
-<layer number="14" name="Route14" color="1" fill="6" visible="no" active="no"/>
-<layer number="15" name="Route15" color="4" fill="6" visible="no" active="no"/>
-<layer number="16" name="Bottom" color="1" fill="1" visible="no" active="no"/>
-<layer number="17" name="Pads" color="2" fill="1" visible="no" active="no"/>
-<layer number="18" name="Vias" color="2" fill="1" visible="no" active="no"/>
-<layer number="19" name="Unrouted" color="6" fill="1" visible="no" active="no"/>
-<layer number="20" name="Dimension" color="15" fill="1" visible="no" active="no"/>
-<layer number="21" name="tPlace" color="7" fill="1" visible="no" active="no"/>
-<layer number="22" name="bPlace" color="7" fill="1" visible="no" active="no"/>
-<layer number="23" name="tOrigins" color="15" fill="1" visible="no" active="no"/>
-<layer number="24" name="bOrigins" color="15" fill="1" visible="no" active="no"/>
-<layer number="25" name="tNames" color="7" fill="1" visible="no" active="no"/>
-<layer number="26" name="bNames" color="7" fill="1" visible="no" active="no"/>
-<layer number="27" name="tValues" color="7" fill="1" visible="no" active="no"/>
-<layer number="28" name="bValues" color="7" fill="1" visible="no" active="no"/>
+<layer number="1" name="Top" color="4" fill="1" visible="yes" active="no"/>
+<layer number="2" name="Route2" color="1" fill="3" visible="yes" active="no"/>
+<layer number="3" name="Route3" color="4" fill="3" visible="yes" active="no"/>
+<layer number="4" name="Route4" color="1" fill="4" visible="yes" active="no"/>
+<layer number="5" name="Route5" color="4" fill="4" visible="yes" active="no"/>
+<layer number="6" name="Route6" color="1" fill="8" visible="yes" active="no"/>
+<layer number="7" name="Route7" color="4" fill="8" visible="yes" active="no"/>
+<layer number="8" name="Route8" color="1" fill="2" visible="yes" active="no"/>
+<layer number="9" name="Route9" color="4" fill="2" visible="yes" active="no"/>
+<layer number="10" name="Route10" color="1" fill="7" visible="yes" active="no"/>
+<layer number="11" name="Route11" color="4" fill="7" visible="yes" active="no"/>
+<layer number="12" name="Route12" color="1" fill="5" visible="yes" active="no"/>
+<layer number="13" name="Route13" color="4" fill="5" visible="yes" active="no"/>
+<layer number="14" name="Route14" color="1" fill="6" visible="yes" active="no"/>
+<layer number="15" name="Route15" color="4" fill="6" visible="yes" active="no"/>
+<layer number="16" name="Bottom" color="1" fill="1" visible="yes" active="no"/>
+<layer number="17" name="Pads" color="2" fill="1" visible="yes" active="no"/>
+<layer number="18" name="Vias" color="2" fill="1" visible="yes" active="no"/>
+<layer number="19" name="Unrouted" color="6" fill="1" visible="yes" active="no"/>
+<layer number="20" name="Dimension" color="15" fill="1" visible="yes" active="no"/>
+<layer number="21" name="tPlace" color="7" fill="1" visible="yes" active="no"/>
+<layer number="22" name="bPlace" color="7" fill="1" visible="yes" active="no"/>
+<layer number="23" name="tOrigins" color="15" fill="1" visible="yes" active="no"/>
+<layer number="24" name="bOrigins" color="15" fill="1" visible="yes" active="no"/>
+<layer number="25" name="tNames" color="7" fill="1" visible="yes" active="no"/>
+<layer number="26" name="bNames" color="7" fill="1" visible="yes" active="no"/>
+<layer number="27" name="tValues" color="7" fill="1" visible="yes" active="no"/>
+<layer number="28" name="bValues" color="7" fill="1" visible="yes" active="no"/>
 <layer number="29" name="tStop" color="7" fill="3" visible="no" active="no"/>
 <layer number="30" name="bStop" color="7" fill="6" visible="no" active="no"/>
@@
 <layer number="35" name="tGlue" color="7" fill="4" visible="no" active="no"/>
 <layer number="36" name="bGlue" color="7" fill="5" visible="no" active="no"/>
-<layer number="37" name="tTest" color="7" fill="1" visible="no" active="no"/>
-<layer number="38" name="bTest" color="7" fill="1" visible="no" active="no"/>
+<layer number="37" name="tTest" color="7" fill="1" visible="yes" active="no"/>
+<layer number="38" name="bTest" color="7" fill="1" visible="yes" active="no"/>
 <layer number="39" name="tKeepout" color="4" fill="11" visible="no" active="no"/>
 <layer number="40" name="bKeepout" color="1" fill="11" visible="no" active="no"/>
@@
 <layer number="44" name="Drills" color="7" fill="1" visible="no" active="no"/>
 <layer number="45" name="Holes" color="7" fill="1" visible="no" active="no"/>
-<layer number="46" name="Milling" color="3" fill="1" visible="no" active="no"/>
-<layer number="47" name="Measures" color="7" fill="1" visible="no" active="no"/>
-<layer number="48" name="Document" color="7" fill="1" visible="no" active="no"/>
-<layer number="49" name="Reference" color="7" fill="1" visible="no" active="no"/>
-<layer number="51" name="tDocu" color="7" fill="1" visible="no" active="no"/>
-<layer number="52" name="bDocu" color="7" fill="1" visible="no" active="no"/>
+<layer number="46" name="Milling" color="3" fill="1" visible="yes" active="no"/>
+<layer number="47" name="Measures" color="7" fill="1" visible="yes" active="no"/>
+<layer number="48" name="Document" color="7" fill="1" visible="yes" active="no"/>
+<layer number="49" name="Reference" color="7" fill="1" visible="yes" active="no"/>
+<layer number="51" name="tDocu" color="7" fill="1" visible="yes" active="no"/>
+<layer number="52" name="bDocu" color="7" fill="1" visible="yes" active="no"/>
 <layer number="90" name="Modules" color="5" fill="1" visible="yes" active="yes"/>
 <layer number="91" name="Nets" color="2" fill="1" visible="yes" active="yes"/>
@@
 </classes>
 <parts>
-<part name="C1" library="cap-trim" deviceset="C-TR-PH20127" device="2222-808-2PIN" value="5-18pF"/>
+<part name="C1" library="cap-trim" deviceset="C-TR-PH20127" device="2222-808-2PINB" value="5-18pF"/>
 <part name="L1" library="r" deviceset="L-SHORT" device="04-5/5" value="0.15μH"/>
 <part name="R1" library="r" deviceset="R" device="0202/7-V" value="1MΩ"/>
