File: eagle/Headphone-Amplifier-ClassAB-alt2.brd (EAGLE design)
At the start: 17 parts, among them T1 BC547, T2 BC327, T3 BC337

Commit message: ...
Parts:
- BAT: value (none) -> SPAD+-+-
- C1, C2: device c:E2,5-4 -> c:E2,5-3
- C3: value 100-1000uF -> 470uF; device c:E2,5-6/V -> c:E5-5
- C4: value 220uF -> 100uF
- D1: value (none) -> 1N4148; device d:DO34-5V -> d:DO34-5-V
- D2: value (none) -> 1N4148
- IN: value (none) -> SPAD+--+
- R1: device r:0202/5 -> r:0204/10
- R4: value 22 -> 27; device r:0204/2.54 -> r:0204/10
- T1: value BC547 -> 2N3904; device t:TO92-CBE -> t:TO92
- T2: value BC327 -> 2N3904
- T3: value BC337 -> 2N3906; device t:TO92-CBE -> t:TO92
- moved C4 10.5 mm to (31.8, 5.08)
- moved IN 10.2 mm to (2.54, 3.81)
- moved T2 8.03 mm to (20.3, 12.7)
- moved T3 8.03 mm to (20.3, 5.08)
- moved R4 4.58 mm to (30.5, 10.2), turned to 0 degrees
- moved HDPH 3.59 mm to (38.1, 14.0), turned to 0 degrees
- moved C3 2.84 mm to (25.4, 5.08), turned to 270 degrees
- moved R2 2.54 mm to (27.9, 12.7)
- moved R3 2.54 mm to (27.9, 15.2)
- moved BAT 2.54 mm to (38.1, 3.81)
- turned C1 to 180 degrees
- turned C2 to 180 degrees
- turned D1 to 0 degrees
- turned T1 to 90 degrees
Connections:
- net GND: now also T1.1, T3.3; no longer T1.E, T2.1
- net N$1: now also T2.2; no longer T3.B
- net N$2: now also T1.3, T3.2; no longer T1.C, T2.2
- net N$4: now also T2.1, T3.1; no longer T2.3, T3.E
- net N$7: now also T1.2; no longer T1.B
- net N$8: now also T2.3; no longer T3.C
Routing:
- net N$8: track 33.0 -> 2.54 mm
- net GND: track 53.3 -> 43.2 mm
- net N$4: track 7.62 -> 17.8 mm
- net N$10: track 5.08 -> 15.2 mm
- net N$6: track 7.62 -> 2.54 mm
- net V+: track 2.54 -> 0.00 mm
- net N$7: track 5.08 -> 7.62 mm
- net N$2: track 10.2 -> 12.7 mm
- net N$1: track 7.62 -> 10.2 mm
- net N$9: vias 2 -> 0
Other:
- board outline added: 40.6 x 17.8 mm

Commit message: ...
Parts:
- moved C4 6.75 mm to (25.4, 7.37)
- moved C3 2.96 mm to (27.9, 3.56)
- moved BAT 2.84 mm to (35.6, 2.54)
- moved R3 2.55 mm to (25.4, 15.0)
- moved R2 2.54 mm to (25.4, 12.7)
- moved R4 2.54 mm to (33.0, 10.2)
- moved C1 0.36 mm to (8.64, 15.0)
- moved C2 0.25 mm to (8.64, 10.2)
- moved R1 0.25 mm to (12.7, 7.37)
- moved IN 0.25 mm to (2.54, 3.56)
- moved D1 0.25 mm to (15.0, 12.7)
Routing:
- net N$4: track 17.8 -> 10.2 mm
- net N$9: track 20.3 -> 23.9 mm
- net N$1: track 10.2 -> 7.63 mm
- net GND: track 43.2 -> 40.8 mm
- net N$8: track 2.54 -> 0.25 mm
Changed lines of the file:
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@@
 </autorouter>
 <elements>
-<element name="BAT" library="pad" package="SPAD+-" value="SPAD+-+-" x="38.1" y="3.81"/>
-<element name="C1" library="c" package="E2,5-3" value="4.7uF" x="8.89" y="15.24" rot="R180"/>
-<element name="C2" library="c" package="E2,5-3" value="4.7uF" x="8.89" y="10.16" rot="R180"/>
-<element name="C3" library="c" package="E5-5" value="470uF" x="25.4" y="5.08" rot="R270"/>
-<element name="C4" library="c" package="E2,5-5" value="100uF" x="31.75" y="5.08"/>
-<element name="D1" library="d" package="DO34-5-V" value="1N4148" x="15.24" y="12.7"/>
+<element name="BAT" library="pad" package="SPAD+-" value="SPAD+-+-" x="35.56" y="2.54"/>
+<element name="C1" library="c" package="E2,5-3" value="4.7uF" x="8.636" y="14.986" rot="R180"/>
+<element name="C2" library="c" package="E2,5-3" value="4.7uF" x="8.636" y="10.16" rot="R180"/>
+<element name="C3" library="c" package="E5-5" value="470uF" x="27.94" y="3.556" rot="R270"/>
+<element name="C4" library="c" package="E2,5-5" value="100uF" x="25.4" y="7.366"/>
+<element name="D1" library="d" package="DO34-5-V" value="1N4148" x="14.986" y="12.7"/>
 <element name="D2" library="d" package="DO34-5V" value="1N4148" x="12.7" y="12.7"/>
 <element name="HDPH" library="pad" package="SPAD-+" value="SPAD+--+" x="38.1" y="13.97"/>
-<element name="IN" library="pad" package="SPAD-+" value="SPAD+--+" x="2.54" y="3.81"/>
-<element name="R1" library="r" package="0204/10" value="100k" x="12.7" y="7.62"/>
-<element name="R2" library="r" package="0204/10" value="330" x="27.94" y="12.7"/>
-<element name="R3" library="r" package="0204/10" value="100" x="27.94" y="15.24"/>
-<element name="R4" library="r" package="0204/10" value="27" x="30.48" y="10.16"/>
+<element name="IN" library="pad" package="SPAD-+" value="SPAD+--+" x="2.54" y="3.556"/>
+<element name="R1" library="r" package="0204/10" value="100k" x="12.7" y="7.366"/>
+<element name="R2" library="r" package="0204/10" value="330" x="25.4" y="12.7"/>
+<element name="R3" library="r" package="0204/10" value="100" x="25.4" y="14.986"/>
+<element name="R4" library="r" package="0204/10" value="27" x="33.02" y="10.16"/>
 <element name="R5" library="r" package="CONN-3P" value="100k" x="5.08" y="10.16"/>
 <element name="T1" library="t" package="TO92" value="2N3904" x="10.16" y="5.08" rot="R90"/>
@@
 <contactref element="R2" pad="1"/>
 <contactref element="T2" pad="2"/>
-<wire x1="15.24" y1="10.16" x2="15.24" y2="12.7" width="1.27" layer="16"/>
+<wire x1="14.986" y1="10.16" x2="15.24" y2="12.7" width="1.27" layer="16"/>
 <wire x1="15.24" y1="12.7" x2="20.32" y2="12.7" width="1.27" layer="16"/>
-<wire x1="20.32" y1="12.7" x2="22.86" y2="12.7" width="1.27" layer="16"/>
 </signal>
 <signal name="N$2">
@@
 <contactref element="D2" pad="A"/>
 <contactref element="D1" pad="C"/>
-<wire x1="12.7" y1="15.24" x2="15.24" y2="15.24" width="1.27" layer="16"/>
+<wire x1="12.7" y1="15.24" x2="14.986" y2="15.24" width="1.27" layer="16"/>
 </signal>
 <signal name="N$4">
@@
 <contactref element="T2" pad="1"/>
 <contactref element="T3" pad="1"/>
-<wire x1="17.78" y1="7.62" x2="20.32" y2="7.62" width="1.27" layer="16"/>
+<wire x1="17.78" y1="7.366" x2="20.32" y2="7.62" width="1.27" layer="16"/>
 <wire x1="20.32" y1="7.62" x2="20.32" y2="10.16" width="1.27" layer="16"/>
-<wire x1="20.32" y1="7.62" x2="22.86" y2="7.62" width="1.27" layer="16"/>
-<wire x1="22.86" y1="7.62" x2="22.86" y2="5.08" width="1.27" layer="16"/>
-<wire x1="22.86" y1="5.08" x2="30.48" y2="5.08" width="1.27" layer="16"/>
+<wire x1="20.32" y1="7.62" x2="21.59" y2="7.62" width="1.27" layer="16"/>
+<wire x1="22.86" y1="7.62" x2="21.59" y2="7.62" width="1.27" layer="16"/>
+<wire x1="21.59" y1="7.62" x2="24.13" y2="7.366" width="1.27" layer="16"/>
 </signal>
 <signal name="N$5">
 <contactref element="C1" pad="+"/>
 <contactref element="R5" pad="3"/>
-<wire x1="10.16" y1="15.24" x2="10.16" y2="12.7" width="1.27" layer="16"/>
+<wire x1="9.906" y1="14.986" x2="10.16" y2="12.7" width="1.27" layer="16"/>
 <wire x1="10.16" y1="12.7" x2="5.08" y2="12.7" width="1.27" layer="16"/>
 </signal>
@@
 <contactref element="R5" pad="2"/>
 <contactref element="C2" pad="-"/>
-<wire x1="5.08" y1="10.16" x2="7.62" y2="10.16" width="1.27" layer="16"/>
+<wire x1="5.08" y1="10.16" x2="7.366" y2="10.16" width="1.27" layer="16"/>
 </signal>
 <signal name="N$7">
@@
 <contactref element="R1" pad="1"/>
 <wire x1="10.16" y1="5.08" x2="10.16" y2="7.62" width="1.27" layer="16"/>
-<wire x1="7.62" y1="7.62" x2="10.16" y2="7.62" width="1.27" layer="16"/>
-<wire x1="10.16" y1="7.62" x2="10.16" y2="10.16" width="1.27" layer="16"/>
+<wire x1="7.62" y1="7.366" x2="10.16" y2="7.62" width="1.27" layer="16"/>
+<wire x1="10.16" y1="7.62" x2="9.906" y2="10.16" width="1.27" layer="16"/>
 </signal>
 <signal name="GND">
@@
 <contactref element="IN" pad="1"/>
 <contactref element="T3" pad="3"/>
-<wire x1="2.54" y1="2.54" x2="5.08" y2="2.54" width="1.27" layer="16"/>
+<wire x1="2.54" y1="2.286" x2="5.08" y2="2.54" width="1.27" layer="16"/>
 <wire x1="5.08" y1="7.62" x2="5.08" y2="2.54" width="1.27" layer="16"/>
 <wire x1="5.08" y1="2.54" x2="7.62" y2="2.54" width="1.27" layer="16"/>
 <wire x1="7.62" y1="5.08" x2="7.62" y2="2.54" width="1.27" layer="16"/>
 <wire x1="7.62" y1="2.54" x2="20.32" y2="2.54" width="1.27" layer="16"/>
-<wire x1="25.4" y1="2.54" x2="20.32" y2="2.54" width="1.27" layer="16"/>
-<wire x1="25.4" y1="2.54" x2="38.1" y2="2.54" width="1.27" layer="16"/>
+<wire x1="27.94" y1="1.016" x2="20.32" y2="2.54" width="1.27" layer="16"/>
+<wire x1="27.94" y1="1.016" x2="35.56" y2="1.27" width="1.27" layer="16"/>
 </signal>
 <signal name="N$9">
@@
 <contactref element="HDPH" pad="1"/>
 <contactref element="R3" pad="2"/>
-<wire x1="38.1" y1="12.7" x2="33.02" y2="12.7" width="1.27" layer="16"/>
-<wire x1="33.02" y1="12.7" x2="33.02" y2="15.24" width="1.27" layer="16"/>
-<wire x1="33.02" y1="12.7" x2="30.48" y2="12.7" width="1.27" layer="16"/>
+<wire x1="38.1" y1="12.7" x2="30.48" y2="12.7" width="1.27" layer="16"/>
+<wire x1="30.48" y1="12.7" x2="30.48" y2="14.986" width="1.27" layer="16"/>
 <wire x1="30.48" y1="12.7" x2="30.48" y2="7.62" width="1.27" layer="16"/>
 <wire x1="30.48" y1="7.62" x2="33.02" y2="7.62" width="1.27" layer="16"/>
-<wire x1="33.02" y1="7.62" x2="33.02" y2="5.08" width="1.27" layer="16"/>
+<wire x1="33.02" y1="7.62" x2="26.67" y2="7.366" width="1.27" layer="16"/>
 </signal>
 <signal name="N$8">
@@
 <contactref element="R3" pad="1"/>
 <contactref element="T2" pad="3"/>
-<wire x1="20.32" y1="15.24" x2="22.86" y2="15.24" width="1.27" layer="16"/>
-<wire x1="25.4" y1="10.16" x2="38.1" y2="15.24" width="0" layer="19" extent="1-1"/>
-<wire x1="25.4" y1="7.62" x2="25.4" y2="10.16" width="0" layer="19" extent="1-1"/>
-<wire x1="22.86" y1="15.24" x2="25.4" y2="10.16" width="0" layer="19" extent="1-1"/>
+<wire x1="20.32" y1="15.24" x2="20.32" y2="14.986" width="1.27" layer="16"/>
+<wire x1="27.94" y1="10.16" x2="38.1" y2="15.24" width="0" layer="19" extent="1-1"/>
+<wire x1="27.94" y1="6.096" x2="27.94" y2="10.16" width="0" layer="19" extent="1-1"/>
+<wire x1="20.32" y1="14.986" x2="27.94" y2="10.16" width="0" layer="19" extent="1-1"/>
 </signal>
 <signal name="V+">
 <contactref element="R4" pad="2"/>
 <contactref element="BAT" pad="2"/>
-<wire x1="38.1" y1="5.08" x2="35.56" y2="10.16" width="0" layer="19" extent="1-1"/>
+<wire x1="35.56" y1="3.81" x2="38.1" y2="10.16" width="0" layer="19" extent="1-1"/>
 </signal>
 <signal name="N$10">
 <contactref element="IN" pad="2"/>
 <contactref element="C1" pad="-"/>
-<wire x1="7.62" y1="15.24" x2="2.54" y2="15.24" width="1.27" layer="16"/>
-<wire x1="2.54" y1="15.24" x2="2.54" y2="5.08" width="1.27" layer="16"/>
+<wire x1="7.366" y1="14.986" x2="2.54" y2="15.24" width="1.27" layer="16"/>
+<wire x1="2.54" y1="15.24" x2="2.54" y2="4.826" width="1.27" layer="16"/>
 </signal>
 </signals>

Commit message: ...
Parts:
- moved BAT 2.84 mm to (38.1, 3.81)
- moved C3 1.27 mm to (29.2, 3.56)
Routing:
- net GND: track 40.8 -> 43.5 mm
Changed lines of the file:
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@@
 </autorouter>
 <elements>
-<element name="BAT" library="pad" package="SPAD+-" value="SPAD+-+-" x="35.56" y="2.54"/>
+<element name="BAT" library="pad" package="SPAD+-" value="SPAD+-+-" x="38.1" y="3.81"/>
 <element name="C1" library="c" package="E2,5-3" value="4.7uF" x="8.636" y="14.986" rot="R180"/>
 <element name="C2" library="c" package="E2,5-3" value="4.7uF" x="8.636" y="10.16" rot="R180"/>
-<element name="C3" library="c" package="E5-5" value="470uF" x="27.94" y="3.556" rot="R270"/>
+<element name="C3" library="c" package="E5-5" value="470uF" x="29.21" y="3.556" rot="R270"/>
 <element name="C4" library="c" package="E2,5-5" value="100uF" x="25.4" y="7.366"/>
 <element name="D1" library="d" package="DO34-5-V" value="1N4148" x="14.986" y="12.7"/>
@@
 <wire x1="7.62" y1="5.08" x2="7.62" y2="2.54" width="1.27" layer="16"/>
 <wire x1="7.62" y1="2.54" x2="20.32" y2="2.54" width="1.27" layer="16"/>
-<wire x1="27.94" y1="1.016" x2="20.32" y2="2.54" width="1.27" layer="16"/>
-<wire x1="27.94" y1="1.016" x2="35.56" y2="1.27" width="1.27" layer="16"/>
+<wire x1="29.21" y1="1.016" x2="20.32" y2="2.54" width="1.27" layer="16"/>
+<wire x1="29.21" y1="1.016" x2="38.1" y2="2.54" width="1.27" layer="16"/>
 </signal>
 <signal name="N$9">
@@
 <wire x1="20.32" y1="15.24" x2="20.32" y2="14.986" width="1.27" layer="16"/>
 <wire x1="27.94" y1="10.16" x2="38.1" y2="15.24" width="0" layer="19" extent="1-1"/>
-<wire x1="27.94" y1="6.096" x2="27.94" y2="10.16" width="0" layer="19" extent="1-1"/>
+<wire x1="29.21" y1="6.096" x2="27.94" y2="10.16" width="0" layer="19" extent="1-1"/>
 <wire x1="20.32" y1="14.986" x2="27.94" y2="10.16" width="0" layer="19" extent="1-1"/>
 </signal>
@@
 <contactref element="R4" pad="2"/>
 <contactref element="BAT" pad="2"/>
-<wire x1="35.56" y1="3.81" x2="38.1" y2="10.16" width="0" layer="19" extent="1-1"/>
+<wire x1="38.1" y1="5.08" x2="38.1" y2="10.16" width="0" layer="19" extent="1-1"/>
 </signal>
 <signal name="N$10">

Commit message: ...
Parts:
- R4: device r:0204/10 -> r:0204/2.54
- moved R4 4.58 mm to (36.8, 7.62), turned to 180 degrees
- moved R3 2.55 mm to (27.9, 15.2)
- moved R2 2.54 mm to (27.9, 12.7)
- moved C3 1.80 mm to (30.5, 4.83)
- moved C4 1.05 mm to (25.1, 6.35), turned to 270 degrees
- moved C1 0.36 mm to (8.89, 15.2)
Routing:
- net N$1: track 7.63 -> 10.2 mm
- net N$8: track 0.25 -> 2.54 mm
- net N$9: track 23.9 -> 23.1 mm
Changed lines of the file:
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@@
 <layer number="44" name="Drills" color="7" fill="1" visible="no" active="yes"/>
 <layer number="45" name="Holes" color="7" fill="1" visible="yes" active="yes"/>
-<layer number="46" name="Milling" color="3" fill="1" visible="no" active="yes"/>
-<layer number="47" name="Measures" color="7" fill="1" visible="no" active="yes"/>
-<layer number="48" name="Document" color="7" fill="1" visible="no" active="yes"/>
-<layer number="49" name="Reference" color="7" fill="1" visible="no" active="yes"/>
+<layer number="46" name="Milling" color="3" fill="1" visible="yes" active="yes"/>
+<layer number="47" name="Measures" color="7" fill="1" visible="yes" active="yes"/>
+<layer number="48" name="Document" color="7" fill="1" visible="yes" active="yes"/>
+<layer number="49" name="Reference" color="7" fill="1" visible="yes" active="yes"/>
 <layer number="51" name="tDocu" color="6" fill="1" visible="yes" active="yes"/>
 <layer number="52" name="bDocu" color="7" fill="1" visible="no" active="yes"/>
@@
 <elements>
 <element name="BAT" library="pad" package="SPAD+-" value="SPAD+-+-" x="38.1" y="3.81"/>
-<element name="C1" library="c" package="E2,5-3" value="4.7uF" x="8.636" y="14.986" rot="R180"/>
+<element name="C1" library="c" package="E2,5-3" value="4.7uF" x="8.89" y="15.24" rot="R180"/>
 <element name="C2" library="c" package="E2,5-3" value="4.7uF" x="8.636" y="10.16" rot="R180"/>
-<element name="C3" library="c" package="E5-5" value="470uF" x="29.21" y="3.556" rot="R270"/>
-<element name="C4" library="c" package="E2,5-5" value="100uF" x="25.4" y="7.366"/>
+<element name="C3" library="c" package="E5-5" value="470uF" x="30.48" y="4.826" rot="R270"/>
+<element name="C4" library="c" package="E2,5-5" value="100uF" x="25.146" y="6.35" rot="R270"/>
 <element name="D1" library="d" package="DO34-5-V" value="1N4148" x="14.986" y="12.7"/>
 <element name="D2" library="d" package="DO34-5V" value="1N4148" x="12.7" y="12.7"/>
@@
 <element name="IN" library="pad" package="SPAD-+" value="SPAD+--+" x="2.54" y="3.556"/>
 <element name="R1" library="r" package="0204/10" value="100k" x="12.7" y="7.366"/>
-<element name="R2" library="r" package="0204/10" value="330" x="25.4" y="12.7"/>
-<element name="R3" library="r" package="0204/10" value="100" x="25.4" y="14.986"/>
-<element name="R4" library="r" package="0204/10" value="27" x="33.02" y="10.16"/>
+<element name="R2" library="r" package="0204/10" value="330" x="27.94" y="12.7"/>
+<element name="R3" library="r" package="0204/10" value="100" x="27.94" y="15.24"/>
+<element name="R4" library="r" package="0204/2.54" value="27" x="36.83" y="7.62" rot="R180"/>
 <element name="R5" library="r" package="CONN-3P" value="100k" x="5.08" y="10.16"/>
 <element name="T1" library="t" package="TO92" value="2N3904" x="10.16" y="5.08" rot="R90"/>
@@
 <contactref element="T2" pad="2"/>
 <wire x1="14.986" y1="10.16" x2="15.24" y2="12.7" width="1.27" layer="16"/>
-<wire x1="15.24" y1="12.7" x2="20.32" y2="12.7" width="1.27" layer="16"/>
+<wire x1="15.24" y1="12.7" x2="22.86" y2="12.7" width="1.27" layer="16"/>
 </signal>
 <signal name="N$2">
@@
 <wire x1="20.32" y1="7.62" x2="21.59" y2="7.62" width="1.27" layer="16"/>
 <wire x1="22.86" y1="7.62" x2="21.59" y2="7.62" width="1.27" layer="16"/>
-<wire x1="21.59" y1="7.62" x2="24.13" y2="7.366" width="1.27" layer="16"/>
+<wire x1="22.86" y1="7.62" x2="25.146" y2="7.62" width="1.27" layer="16"/>
 </signal>
 <signal name="N$5">
 <contactref element="C1" pad="+"/>
 <contactref element="R5" pad="3"/>
-<wire x1="9.906" y1="14.986" x2="10.16" y2="12.7" width="1.27" layer="16"/>
+<wire x1="10.16" y1="15.24" x2="10.16" y2="12.7" width="1.27" layer="16"/>
 <wire x1="10.16" y1="12.7" x2="5.08" y2="12.7" width="1.27" layer="16"/>
 </signal>
@@
 <wire x1="7.62" y1="5.08" x2="7.62" y2="2.54" width="1.27" layer="16"/>
 <wire x1="7.62" y1="2.54" x2="20.32" y2="2.54" width="1.27" layer="16"/>
-<wire x1="29.21" y1="1.016" x2="20.32" y2="2.54" width="1.27" layer="16"/>
-<wire x1="29.21" y1="1.016" x2="38.1" y2="2.54" width="1.27" layer="16"/>
+<wire x1="30.48" y1="2.286" x2="20.32" y2="2.54" width="1.27" layer="16"/>
+<wire x1="30.48" y1="2.286" x2="38.1" y2="2.54" width="1.27" layer="16"/>
 </signal>
 <signal name="N$9">
@@
 <contactref element="HDPH" pad="1"/>
 <contactref element="R3" pad="2"/>
-<wire x1="38.1" y1="12.7" x2="30.48" y2="12.7" width="1.27" layer="16"/>
-<wire x1="30.48" y1="12.7" x2="30.48" y2="14.986" width="1.27" layer="16"/>
-<wire x1="30.48" y1="12.7" x2="30.48" y2="7.62" width="1.27" layer="16"/>
-<wire x1="30.48" y1="7.62" x2="33.02" y2="7.62" width="1.27" layer="16"/>
-<wire x1="33.02" y1="7.62" x2="26.67" y2="7.366" width="1.27" layer="16"/>
+<wire x1="38.1" y1="12.7" x2="33.02" y2="12.7" width="1.27" layer="16"/>
+<wire x1="33.02" y1="12.7" x2="33.02" y2="15.24" width="1.27" layer="16"/>
+<wire x1="33.02" y1="12.7" x2="33.02" y2="5.08" width="1.27" layer="16"/>
+<wire x1="33.02" y1="5.08" x2="25.146" y2="5.08" width="1.27" layer="16"/>
 </signal>
 <signal name="N$8">
@@
 <contactref element="R3" pad="1"/>
 <contactref element="T2" pad="3"/>
-<wire x1="20.32" y1="15.24" x2="20.32" y2="14.986" width="1.27" layer="16"/>
-<wire x1="27.94" y1="10.16" x2="38.1" y2="15.24" width="0" layer="19" extent="1-1"/>
-<wire x1="29.21" y1="6.096" x2="27.94" y2="10.16" width="0" layer="19" extent="1-1"/>
-<wire x1="20.32" y1="14.986" x2="27.94" y2="10.16" width="0" layer="19" extent="1-1"/>
+<wire x1="20.32" y1="15.24" x2="22.86" y2="15.24" width="1.27" layer="16"/>
+<wire x1="35.56" y1="7.62" x2="38.1" y2="15.24" width="0" layer="19" extent="1-1"/>
+<wire x1="30.48" y1="7.366" x2="35.56" y2="7.62" width="0" layer="19" extent="1-1"/>
+<wire x1="22.86" y1="15.24" x2="30.48" y2="7.366" width="0" layer="19" extent="1-1"/>
 </signal>
 <signal name="V+">
 <contactref element="R4" pad="2"/>
 <contactref element="BAT" pad="2"/>
-<wire x1="38.1" y1="5.08" x2="38.1" y2="10.16" width="0" layer="19" extent="1-1"/>
+<wire x1="38.1" y1="5.08" x2="38.1" y2="7.62" width="0" layer="19" extent="1-1"/>
 </signal>
 <signal name="N$10">
 <contactref element="IN" pad="2"/>
 <contactref element="C1" pad="-"/>
-<wire x1="7.366" y1="14.986" x2="2.54" y2="15.24" width="1.27" layer="16"/>
+<wire x1="7.62" y1="15.24" x2="2.54" y2="15.24" width="1.27" layer="16"/>
 <wire x1="2.54" y1="15.24" x2="2.54" y2="4.826" width="1.27" layer="16"/>
 </signal>
