File: eagle/Headphone-Amplifier-ClassAB-alt2.brd (EAGLE design)
At the start: 40.6 x 17.8 mm, 17 parts, among them T1 2N3904, T2 2N3904, T3 2N3906

Commit message: ...
Parts:
- moved C2 0.25 mm to (8.89, 10.2)
- moved C3 0.25 mm to (30.5, 5.08)
- moved R1 0.25 mm to (12.7, 7.62)
- moved IN 0.25 mm to (2.54, 3.81)
- moved D1 0.25 mm to (15.2, 12.7)
- moved C4 0.25 mm to (25.4, 6.35)
Changed lines of the file:
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@@
 <wire x1="40.64" y1="17.78" x2="0" y2="17.78" width="0" layer="20"/>
 <wire x1="0" y1="17.78" x2="0" y2="0" width="0" layer="20"/>
+<wire x1="0" y1="1.27" x2="40.64" y2="1.27" width="0" layer="47"/>
+<wire x1="40.64" y1="1.27" x2="40.64" y2="16.51" width="0" layer="47"/>
+<wire x1="40.64" y1="16.51" x2="0" y2="16.51" width="0" layer="47"/>
+<wire x1="0" y1="16.51" x2="0" y2="1.27" width="0" layer="47"/>
 </plain>
 <attributes>
@@
 <element name="BAT" library="pad" package="SPAD+-" value="SPAD+-+-" x="38.1" y="3.81"/>
 <element name="C1" library="c" package="E2,5-3" value="4.7uF" x="8.89" y="15.24" rot="R180"/>
-<element name="C2" library="c" package="E2,5-3" value="4.7uF" x="8.636" y="10.16" rot="R180"/>
-<element name="C3" library="c" package="E5-5" value="470uF" x="30.48" y="4.826" rot="R270"/>
-<element name="C4" library="c" package="E2,5-5" value="100uF" x="25.146" y="6.35" rot="R270"/>
-<element name="D1" library="d" package="DO34-5-V" value="1N4148" x="14.986" y="12.7"/>
+<element name="C2" library="c" package="E2,5-3" value="4.7uF" x="8.89" y="10.16" rot="R180"/>
+<element name="C3" library="c" package="E5-5" value="470uF" x="30.48" y="5.08" rot="R270"/>
+<element name="C4" library="c" package="E2,5-5" value="100uF" x="25.4" y="6.35" rot="R270"/>
+<element name="D1" library="d" package="DO34-5-V" value="1N4148" x="15.24" y="12.7"/>
 <element name="D2" library="d" package="DO34-5V" value="1N4148" x="12.7" y="12.7"/>
 <element name="HDPH" library="pad" package="SPAD-+" value="SPAD+--+" x="38.1" y="13.97"/>
-<element name="IN" library="pad" package="SPAD-+" value="SPAD+--+" x="2.54" y="3.556"/>
-<element name="R1" library="r" package="0204/10" value="100k" x="12.7" y="7.366"/>
+<element name="IN" library="pad" package="SPAD-+" value="SPAD+--+" x="2.54" y="3.81"/>
+<element name="R1" library="r" package="0204/10" value="100k" x="12.7" y="7.62"/>
 <element name="R2" library="r" package="0204/10" value="330" x="27.94" y="12.7"/>
 <element name="R3" library="r" package="0204/10" value="100" x="27.94" y="15.24"/>
@@
 <contactref element="R2" pad="1"/>
 <contactref element="T2" pad="2"/>
-<wire x1="14.986" y1="10.16" x2="15.24" y2="12.7" width="1.27" layer="16"/>
+<wire x1="15.24" y1="10.16" x2="15.24" y2="12.7" width="1.27" layer="16"/>
 <wire x1="15.24" y1="12.7" x2="22.86" y2="12.7" width="1.27" layer="16"/>
+<wire x1="22.86" y1="12.7" x2="20.32" y2="12.7" width="0" layer="19" extent="1-1"/>
 </signal>
 <signal name="N$2">
@@
 <contactref element="D2" pad="A"/>
 <contactref element="D1" pad="C"/>
-<wire x1="12.7" y1="15.24" x2="14.986" y2="15.24" width="1.27" layer="16"/>
+<wire x1="12.7" y1="15.24" x2="15.24" y2="15.24" width="1.27" layer="16"/>
 </signal>
 <signal name="N$4">
@@
 <contactref element="T2" pad="1"/>
 <contactref element="T3" pad="1"/>
-<wire x1="17.78" y1="7.366" x2="20.32" y2="7.62" width="1.27" layer="16"/>
+<wire x1="17.78" y1="7.62" x2="20.32" y2="7.62" width="1.27" layer="16"/>
 <wire x1="20.32" y1="7.62" x2="20.32" y2="10.16" width="1.27" layer="16"/>
 <wire x1="20.32" y1="7.62" x2="21.59" y2="7.62" width="1.27" layer="16"/>
 <wire x1="22.86" y1="7.62" x2="21.59" y2="7.62" width="1.27" layer="16"/>
-<wire x1="22.86" y1="7.62" x2="25.146" y2="7.62" width="1.27" layer="16"/>
+<wire x1="22.86" y1="7.62" x2="25.4" y2="7.62" width="1.27" layer="16"/>
 </signal>
 <signal name="N$5">
@@
 <contactref element="R5" pad="2"/>
 <contactref element="C2" pad="-"/>
-<wire x1="5.08" y1="10.16" x2="7.366" y2="10.16" width="1.27" layer="16"/>
+<wire x1="5.08" y1="10.16" x2="7.62" y2="10.16" width="1.27" layer="16"/>
 </signal>
 <signal name="N$7">
@@
 <contactref element="R1" pad="1"/>
 <wire x1="10.16" y1="5.08" x2="10.16" y2="7.62" width="1.27" layer="16"/>
-<wire x1="7.62" y1="7.366" x2="10.16" y2="7.62" width="1.27" layer="16"/>
-<wire x1="10.16" y1="7.62" x2="9.906" y2="10.16" width="1.27" layer="16"/>
+<wire x1="7.62" y1="7.62" x2="10.16" y2="7.62" width="1.27" layer="16"/>
+<wire x1="10.16" y1="7.62" x2="10.16" y2="10.16" width="1.27" layer="16"/>
 </signal>
 <signal name="GND">
@@
 <contactref element="IN" pad="1"/>
 <contactref element="T3" pad="3"/>
-<wire x1="2.54" y1="2.286" x2="5.08" y2="2.54" width="1.27" layer="16"/>
+<wire x1="2.54" y1="2.54" x2="5.08" y2="2.54" width="1.27" layer="16"/>
 <wire x1="5.08" y1="7.62" x2="5.08" y2="2.54" width="1.27" layer="16"/>
 <wire x1="5.08" y1="2.54" x2="7.62" y2="2.54" width="1.27" layer="16"/>
 <wire x1="7.62" y1="5.08" x2="7.62" y2="2.54" width="1.27" layer="16"/>
 <wire x1="7.62" y1="2.54" x2="20.32" y2="2.54" width="1.27" layer="16"/>
-<wire x1="30.48" y1="2.286" x2="20.32" y2="2.54" width="1.27" layer="16"/>
-<wire x1="30.48" y1="2.286" x2="38.1" y2="2.54" width="1.27" layer="16"/>
+<wire x1="30.48" y1="2.54" x2="20.32" y2="2.54" width="1.27" layer="16"/>
+<wire x1="30.48" y1="2.54" x2="38.1" y2="2.54" width="1.27" layer="16"/>
 </signal>
 <signal name="N$9">
@@
 <wire x1="33.02" y1="12.7" x2="33.02" y2="15.24" width="1.27" layer="16"/>
 <wire x1="33.02" y1="12.7" x2="33.02" y2="5.08" width="1.27" layer="16"/>
-<wire x1="33.02" y1="5.08" x2="25.146" y2="5.08" width="1.27" layer="16"/>
+<wire x1="33.02" y1="5.08" x2="25.4" y2="5.08" width="1.27" layer="16"/>
 </signal>
 <signal name="N$8">
@@
 <wire x1="20.32" y1="15.24" x2="22.86" y2="15.24" width="1.27" layer="16"/>
 <wire x1="35.56" y1="7.62" x2="38.1" y2="15.24" width="0" layer="19" extent="1-1"/>
-<wire x1="30.48" y1="7.366" x2="35.56" y2="7.62" width="0" layer="19" extent="1-1"/>
-<wire x1="22.86" y1="15.24" x2="30.48" y2="7.366" width="0" layer="19" extent="1-1"/>
+<wire x1="30.48" y1="7.62" x2="35.56" y2="7.62" width="0" layer="19" extent="1-1"/>
+<wire x1="22.86" y1="15.24" x2="30.48" y2="7.62" width="0" layer="19" extent="1-1"/>
 </signal>
 <signal name="V+">
@@
 <contactref element="C1" pad="-"/>
 <wire x1="7.62" y1="15.24" x2="2.54" y2="15.24" width="1.27" layer="16"/>
-<wire x1="2.54" y1="15.24" x2="2.54" y2="4.826" width="1.27" layer="16"/>
+<wire x1="2.54" y1="15.24" x2="2.54" y2="5.08" width="1.27" layer="16"/>
 </signal>
 </signals>

Commit message: ...
Parts:
- C1, C2: value 4.7uF -> 4.7μF
- C3: value 470uF -> 470μF
- C4: value 100uF -> 100μF
- R1, R5: value 100k -> 100kΩ
- R2: value 330 -> 330Ω
- R3: value 100 -> 100Ω
- R4: value 27 -> 27Ω
Changed lines of the file:
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@@
 <elements>
 <element name="BAT" library="pad" package="SPAD+-" value="SPAD+-+-" x="38.1" y="3.81"/>
-<element name="C1" library="c" package="E2,5-3" value="4.7uF" x="8.89" y="15.24" rot="R180"/>
-<element name="C2" library="c" package="E2,5-3" value="4.7uF" x="8.89" y="10.16" rot="R180"/>
-<element name="C3" library="c" package="E5-5" value="470uF" x="30.48" y="5.08" rot="R270"/>
-<element name="C4" library="c" package="E2,5-5" value="100uF" x="25.4" y="6.35" rot="R270"/>
+<element name="C1" library="c" package="E2,5-3" value="4.7μF" x="8.89" y="15.24" rot="R180"/>
+<element name="C2" library="c" package="E2,5-3" value="4.7μF" x="8.89" y="10.16" rot="R180"/>
+<element name="C3" library="c" package="E5-5" value="470μF" x="30.48" y="5.08" rot="R270"/>
+<element name="C4" library="c" package="E2,5-5" value="100μF" x="25.4" y="6.35" rot="R270"/>
 <element name="D1" library="d" package="DO34-5-V" value="1N4148" x="15.24" y="12.7"/>
 <element name="D2" library="d" package="DO34-5V" value="1N4148" x="12.7" y="12.7"/>
 <element name="HDPH" library="pad" package="SPAD-+" value="SPAD+--+" x="38.1" y="13.97"/>
 <element name="IN" library="pad" package="SPAD-+" value="SPAD+--+" x="2.54" y="3.81"/>
-<element name="R1" library="r" package="0204/10" value="100k" x="12.7" y="7.62"/>
-<element name="R2" library="r" package="0204/10" value="330" x="27.94" y="12.7"/>
-<element name="R3" library="r" package="0204/10" value="100" x="27.94" y="15.24"/>
-<element name="R4" library="r" package="0204/2.54" value="27" x="36.83" y="7.62" rot="R180"/>
-<element name="R5" library="r" package="CONN-3P" value="100k" x="5.08" y="10.16"/>
+<element name="R1" library="r" package="0204/10" value="100kΩ" x="12.7" y="7.62"/>
+<element name="R2" library="r" package="0204/10" value="330Ω" x="27.94" y="12.7"/>
+<element name="R3" library="r" package="0204/10" value="100Ω" x="27.94" y="15.24"/>
+<element name="R4" library="r" package="0204/2.54" value="27Ω" x="36.83" y="7.62" rot="R180"/>
+<element name="R5" library="r" package="CONN-3P" value="100kΩ" x="5.08" y="10.16"/>
 <element name="T1" library="t" package="TO92" value="2N3904" x="10.16" y="5.08" rot="R90"/>
 <element name="T2" library="t" package="TO92" value="2N3904" x="20.32" y="12.7" rot="R180"/>

Commit message: ...
Routing:
- net V+: track 0.00 -> 2.54 mm
Changed lines of the file:
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@@
 <contactref element="R4" pad="2"/>
 <contactref element="BAT" pad="2"/>
-<wire x1="38.1" y1="5.08" x2="38.1" y2="7.62" width="0" layer="19" extent="1-1"/>
+<wire x1="38.1" y1="5.08" x2="38.1" y2="7.62" width="1.27" layer="16"/>
 </signal>
 <signal name="N$10">
