File: eagle/555-Oscillator.brd (EAGLE design)
At the start: 27.9 x 30.5 mm, 8 parts, among them J1 SPAD+--+

Commit message: ...
Parts:
- removed J1: SPAD+--+, pad:SPAD-+
- removed U$1: 555_ALT, ic:DIL08
- added IC1: 555, ic:DIL08
- added OUT: SPAD+--+, pad:SPAD-+
- moved R3 10.2 mm to (7.62, 25.4)
- moved C1 10.2 mm to (12.7, 5.08)
- moved C2 10.2 mm to (17.8, 5.08)
- moved R1 10.2 mm to (17.8, 27.9)
- moved R2 10.2 mm to (22.9, 10.2)
- moved S1 10.2 mm to (25.4, 3.81)
Connections:
- net GND: now also IC1.1, OUT.1; no longer J1.1, U$1.1
- net N$1: now also IC1.7; no longer U$1.7
- net N$3: now also IC1.2, IC1.6; no longer U$1.2, U$1.6
- net N$6: now also IC1.5; no longer U$1.5
- net N$8: now also IC1.3, OUT.2; no longer J1.2, U$1.3
- net VCC: now also IC1.4, IC1.8; no longer U$1.4, U$1.8
Changed lines of the file:
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@@
 <layer number="23" name="tOrigins" color="15" fill="1" visible="yes" active="yes"/>
 <layer number="24" name="bOrigins" color="15" fill="1" visible="yes" active="yes"/>
-<layer number="25" name="tNames" color="7" fill="1" visible="no" active="yes"/>
+<layer number="25" name="tNames" color="7" fill="1" visible="yes" active="yes"/>
 <layer number="26" name="bNames" color="7" fill="1" visible="no" active="yes"/>
-<layer number="27" name="tValues" color="7" fill="1" visible="no" active="yes"/>
+<layer number="27" name="tValues" color="7" fill="1" visible="yes" active="yes"/>
 <layer number="28" name="bValues" color="7" fill="1" visible="no" active="yes"/>
 <layer number="29" name="tStop" color="7" fill="3" visible="no" active="yes"/>
@@
 <layer number="46" name="Milling" color="3" fill="1" visible="no" active="yes"/>
 <layer number="47" name="Measures" color="7" fill="1" visible="no" active="yes"/>
-<layer number="48" name="Document" color="7" fill="1" visible="no" active="yes"/>
+<layer number="48" name="Document" color="7" fill="1" visible="yes" active="yes"/>
 <layer number="49" name="Reference" color="7" fill="1" visible="no" active="yes"/>
 <layer number="50" name="dxf" color="7" fill="1" visible="no" active="yes"/>
@@
 <board>
 <plain>
-<wire x1="0" y1="10.16" x2="27.94" y2="10.16" width="0" layer="20"/>
-<wire x1="27.94" y1="10.16" x2="27.94" y2="40.64" width="0" layer="20"/>
-<wire x1="27.94" y1="40.64" x2="0" y2="40.64" width="0" layer="20"/>
-<wire x1="0" y1="40.64" x2="0" y2="10.16" width="0" layer="20"/>
+<wire x1="0" y1="0" x2="27.94" y2="0" width="0" layer="20"/>
+<wire x1="27.94" y1="0" x2="27.94" y2="30.48" width="0" layer="20"/>
+<wire x1="27.94" y1="30.48" x2="0" y2="30.48" width="0" layer="20"/>
+<wire x1="0" y1="30.48" x2="0" y2="0" width="0" layer="20"/>
 </plain>
 <attributes>
@@
 </autorouter>
 <elements>
-<element name="C1" library="c" package="C050-020X036/V" value="470n" x="12.7" y="15.24" rot="R180"/>
-<element name="C2" library="c" package="C050-020X036/V" value="10n" x="17.78" y="15.24" rot="R180"/>
-<element name="J1" library="pad" package="SPAD-+" value="SPAD+--+" x="5.08" y="13.97" rot="R180"/>
-<element name="R1" library="r" package="0207/10" value="1k" x="17.78" y="38.1" rot="R180"/>
-<element name="R2" library="r" package="0207/10" value="10k" x="22.86" y="20.32" rot="R90"/>
-<element name="R3" library="r" package="POT-V" value="220k" x="7.62" y="35.56" rot="R90"/>
-<element name="S1" library="pad" package="PWR-R" value="VCC_GNDPWR-R" x="25.4" y="13.97"/>
-<element name="U$1" library="ic" package="DIL08" value="555_ALT" x="13.97" y="24.13"/>
+<element name="C1" library="c" package="C050-020X036/V" value="470n" x="12.7" y="5.08" rot="R180"/>
+<element name="C2" library="c" package="C050-020X036/V" value="10n" x="17.78" y="5.08" rot="R180"/>
+<element name="OUT" library="pad" package="SPAD-+" value="SPAD+--+" x="5.08" y="3.81" rot="R180"/>
+<element name="R1" library="r" package="0207/10" value="1k" x="17.78" y="27.94" rot="R180"/>
+<element name="R2" library="r" package="0207/10" value="10k" x="22.86" y="10.16" rot="R90"/>
+<element name="R3" library="r" package="POT-V" value="220k" x="7.62" y="25.4" rot="R90"/>
+<element name="S1" library="pad" package="PWR-R" value="VCC_GNDPWR-R" x="25.4" y="3.81"/>
+<element name="IC1" library="ic" package="DIL08" value="555" x="13.97" y="13.97"/>
 </elements>
 <signals>
@@
 <contactref element="R2" pad="2"/>
 <contactref element="R1" pad="1"/>
-<contactref element="U$1" pad="7"/>
-<wire x1="17.78" y1="25.4" x2="22.86" y2="25.4" width="1.27" layer="16"/>
-<wire x1="22.86" y1="38.1" x2="22.86" y2="25.4" width="1.27" layer="16"/>
+<contactref element="IC1" pad="7"/>
+<wire x1="17.78" y1="15.24" x2="22.86" y2="15.24" width="1.27" layer="16"/>
+<wire x1="22.86" y1="27.94" x2="22.86" y2="15.24" width="1.27" layer="16"/>
 </signal>
 <signal name="N$2">
 <contactref element="R1" pad="2"/>
 <contactref element="R3" pad="E"/>
-<wire x1="12.7" y1="38.1" x2="10.16" y2="38.1" width="1.27" layer="16"/>
+<wire x1="12.7" y1="27.94" x2="10.16" y2="27.94" width="1.27" layer="16"/>
 </signal>
 <signal name="N$3">
@@
 <contactref element="C1" pad="1"/>
 <contactref element="R3" pad="S"/>
-<contactref element="U$1" pad="6"/>
-<contactref element="U$1" pad="2"/>
-<wire x1="10.16" y1="33.02" x2="12.7" y2="33.02" width="1.27" layer="16"/>
-<wire x1="12.7" y1="33.02" x2="12.7" y2="25.4" width="1.27" layer="16"/>
-<wire x1="10.16" y1="25.4" x2="12.7" y2="25.4" width="1.27" layer="16"/>
-<wire x1="12.7" y1="25.4" x2="12.7" y2="22.86" width="1.27" layer="16"/>
-<wire x1="12.7" y1="22.86" x2="17.78" y2="22.86" width="1.27" layer="16"/>
-<wire x1="10.16" y1="33.02" x2="5.08" y2="33.02" width="1.27" layer="16"/>
-<wire x1="5.08" y1="33.02" x2="5.08" y2="35.56" width="1.27" layer="16"/>
-<wire x1="12.7" y1="17.78" x2="12.7" y2="22.86" width="1.27" layer="16"/>
+<contactref element="IC1" pad="6"/>
+<contactref element="IC1" pad="2"/>
+<wire x1="10.16" y1="22.86" x2="12.7" y2="22.86" width="1.27" layer="16"/>
+<wire x1="12.7" y1="22.86" x2="12.7" y2="15.24" width="1.27" layer="16"/>
+<wire x1="10.16" y1="15.24" x2="12.7" y2="15.24" width="1.27" layer="16"/>
+<wire x1="12.7" y1="15.24" x2="12.7" y2="12.7" width="1.27" layer="16"/>
+<wire x1="12.7" y1="12.7" x2="17.78" y2="12.7" width="1.27" layer="16"/>
+<wire x1="10.16" y1="22.86" x2="5.08" y2="22.86" width="1.27" layer="16"/>
+<wire x1="5.08" y1="22.86" x2="5.08" y2="25.4" width="1.27" layer="16"/>
+<wire x1="12.7" y1="7.62" x2="12.7" y2="12.7" width="1.27" layer="16"/>
 </signal>
 <signal name="GND">
-<contactref element="U$1" pad="1"/>
+<contactref element="IC1" pad="1"/>
 <contactref element="S1" pad="1"/>
 <contactref element="C1" pad="2"/>
 <contactref element="C2" pad="2"/>
-<contactref element="J1" pad="1"/>
-<wire x1="10.16" y1="27.94" x2="2.54" y2="27.94" width="1.27" layer="16"/>
-<wire x1="2.54" y1="27.94" x2="2.54" y2="12.7" width="1.27" layer="16"/>
-<wire x1="2.54" y1="12.7" x2="5.08" y2="12.7" width="1.27" layer="16"/>
-<wire x1="5.08" y1="12.7" x2="12.7" y2="12.7" width="1.27" layer="16"/>
-<wire x1="12.7" y1="12.7" x2="17.78" y2="12.7" width="1.27" layer="16"/>
-<wire x1="25.4" y1="12.7" x2="17.78" y2="12.7" width="1.27" layer="16"/>
+<contactref element="OUT" pad="1"/>
+<wire x1="10.16" y1="17.78" x2="2.54" y2="17.78" width="1.27" layer="16"/>
+<wire x1="2.54" y1="17.78" x2="2.54" y2="2.54" width="1.27" layer="16"/>
+<wire x1="2.54" y1="2.54" x2="5.08" y2="2.54" width="1.27" layer="16"/>
+<wire x1="5.08" y1="2.54" x2="12.7" y2="2.54" width="1.27" layer="16"/>
+<wire x1="12.7" y1="2.54" x2="17.78" y2="2.54" width="1.27" layer="16"/>
+<wire x1="25.4" y1="2.54" x2="17.78" y2="2.54" width="1.27" layer="16"/>
 </signal>
 <signal name="N$6">
-<contactref element="U$1" pad="5"/>
+<contactref element="IC1" pad="5"/>
 <contactref element="C2" pad="1"/>
-<wire x1="17.78" y1="20.32" x2="17.78" y2="17.78" width="1.27" layer="16"/>
+<wire x1="17.78" y1="10.16" x2="17.78" y2="7.62" width="1.27" layer="16"/>
 </signal>
 <signal name="VCC">
 <contactref element="S1" pad="2"/>
-<contactref element="U$1" pad="8"/>
-<contactref element="U$1" pad="4"/>
+<contactref element="IC1" pad="8"/>
+<contactref element="IC1" pad="4"/>
 <contactref element="R2" pad="1"/>
-<wire x1="10.16" y1="20.32" x2="10.16" y2="15.24" width="1.27" layer="16"/>
-<wire x1="10.16" y1="15.24" x2="20.32" y2="15.24" width="1.27" layer="16"/>
-<wire x1="20.32" y1="15.24" x2="22.86" y2="15.24" width="1.27" layer="16"/>
-<wire x1="25.4" y1="15.24" x2="22.86" y2="15.24" width="1.27" layer="16"/>
-<wire x1="17.78" y1="27.94" x2="20.32" y2="27.94" width="1.27" layer="16"/>
-<wire x1="20.32" y1="27.94" x2="20.32" y2="15.24" width="1.27" layer="1"/>
-<via x="20.32" y="15.24" extent="1-16" drill="0.79375" diameter="1.6764"/>
-<via x="20.32" y="27.94" extent="1-16" drill="0.79375" diameter="1.6764"/>
+<wire x1="10.16" y1="10.16" x2="10.16" y2="5.08" width="1.27" layer="16"/>
+<wire x1="10.16" y1="5.08" x2="20.32" y2="5.08" width="1.27" layer="16"/>
+<wire x1="20.32" y1="5.08" x2="22.86" y2="5.08" width="1.27" layer="16"/>
+<wire x1="25.4" y1="5.08" x2="22.86" y2="5.08" width="1.27" layer="16"/>
+<wire x1="17.78" y1="17.78" x2="20.32" y2="17.78" width="1.27" layer="16"/>
+<wire x1="20.32" y1="17.78" x2="20.32" y2="5.08" width="1.27" layer="1"/>
+<via x="20.32" y="5.08" extent="1-16" drill="0.79375" diameter="1.6764"/>
+<via x="20.32" y="17.78" extent="1-16" drill="0.79375" diameter="1.6764"/>
 </signal>
 <signal name="N$8">
-<contactref element="J1" pad="2"/>
-<contactref element="U$1" pad="3"/>
-<wire x1="5.08" y1="15.24" x2="5.08" y2="22.86" width="1.27" layer="16"/>
-<wire x1="5.08" y1="22.86" x2="10.16" y2="22.86" width="1.27" layer="16"/>
+<contactref element="OUT" pad="2"/>
+<contactref element="IC1" pad="3"/>
+<wire x1="5.08" y1="5.08" x2="5.08" y2="12.7" width="1.27" layer="16"/>
+<wire x1="5.08" y1="12.7" x2="10.16" y2="12.7" width="1.27" layer="16"/>
 </signal>
 </signals>

Commit message: ...
Parts:
- moved OUT 7.62 mm to (5.08, 11.4)
- moved R1 5.08 mm to (17.8, 22.9)
- moved C1 5.08 mm to (7.62, 5.08), turned to 90 degrees
- turned R3 to 0 degrees
Routing:
- net N$3: track 33.0 -> 41.2 mm, vias 0 -> 4
- net N$8: track 12.7 -> 5.08 mm
- net GND: track 45.7 -> 40.6 mm, vias 0 -> 2
- net N$1: track 17.8 -> 12.7 mm
Changed lines of the file:
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@@
 <layer number="24" name="bOrigins" color="15" fill="1" visible="yes" active="yes"/>
 <layer number="25" name="tNames" color="7" fill="1" visible="yes" active="yes"/>
-<layer number="26" name="bNames" color="7" fill="1" visible="no" active="yes"/>
+<layer number="26" name="bNames" color="7" fill="1" visible="yes" active="yes"/>
 <layer number="27" name="tValues" color="7" fill="1" visible="yes" active="yes"/>
-<layer number="28" name="bValues" color="7" fill="1" visible="no" active="yes"/>
+<layer number="28" name="bValues" color="7" fill="1" visible="yes" active="yes"/>
 <layer number="29" name="tStop" color="7" fill="3" visible="no" active="yes"/>
 <layer number="30" name="bStop" color="7" fill="6" visible="no" active="yes"/>
@@
 <layer number="46" name="Milling" color="3" fill="1" visible="no" active="yes"/>
 <layer number="47" name="Measures" color="7" fill="1" visible="no" active="yes"/>
-<layer number="48" name="Document" color="7" fill="1" visible="yes" active="yes"/>
+<layer number="48" name="Document" color="7" fill="1" visible="no" active="yes"/>
 <layer number="49" name="Reference" color="7" fill="1" visible="no" active="yes"/>
 <layer number="50" name="dxf" color="7" fill="1" visible="no" active="yes"/>
@@
 </autorouter>
 <elements>
-<element name="C1" library="c" package="C050-020X036/V" value="470n" x="12.7" y="5.08" rot="R180"/>
+<element name="C1" library="c" package="C050-020X036/V" value="470n" x="7.62" y="5.08" rot="R90"/>
 <element name="C2" library="c" package="C050-020X036/V" value="10n" x="17.78" y="5.08" rot="R180"/>
-<element name="OUT" library="pad" package="SPAD-+" value="SPAD+--+" x="5.08" y="3.81" rot="R180"/>
-<element name="R1" library="r" package="0207/10" value="1k" x="17.78" y="27.94" rot="R180"/>
+<element name="OUT" library="pad" package="SPAD-+" value="SPAD+--+" x="5.08" y="11.43" rot="R180"/>
+<element name="R1" library="r" package="0207/10" value="1k" x="17.78" y="22.86" rot="R180"/>
 <element name="R2" library="r" package="0207/10" value="10k" x="22.86" y="10.16" rot="R90"/>
-<element name="R3" library="r" package="POT-V" value="220k" x="7.62" y="25.4" rot="R90"/>
+<element name="R3" library="r" package="POT-V" value="220k" x="7.62" y="25.4"/>
 <element name="S1" library="pad" package="PWR-R" value="VCC_GNDPWR-R" x="25.4" y="3.81"/>
 <element name="IC1" library="ic" package="DIL08" value="555" x="13.97" y="13.97"/>
@@
 <contactref element="IC1" pad="7"/>
 <wire x1="17.78" y1="15.24" x2="22.86" y2="15.24" width="1.27" layer="16"/>
-<wire x1="22.86" y1="27.94" x2="22.86" y2="15.24" width="1.27" layer="16"/>
+<wire x1="22.86" y1="22.86" x2="22.86" y2="15.24" width="1.27" layer="16"/>
 </signal>
 <signal name="N$2">
 <contactref element="R1" pad="2"/>
 <contactref element="R3" pad="E"/>
-<wire x1="12.7" y1="27.94" x2="10.16" y2="27.94" width="1.27" layer="16"/>
+<wire x1="12.7" y1="22.86" x2="10.16" y2="22.86" width="1.27" layer="16"/>
 </signal>
 <signal name="N$3">
@@
 <contactref element="IC1" pad="6"/>
 <contactref element="IC1" pad="2"/>
-<wire x1="10.16" y1="22.86" x2="12.7" y2="22.86" width="1.27" layer="16"/>
-<wire x1="12.7" y1="22.86" x2="12.7" y2="15.24" width="1.27" layer="16"/>
-<wire x1="10.16" y1="15.24" x2="12.7" y2="15.24" width="1.27" layer="16"/>
-<wire x1="12.7" y1="15.24" x2="12.7" y2="12.7" width="1.27" layer="16"/>
-<wire x1="12.7" y1="12.7" x2="17.78" y2="12.7" width="1.27" layer="16"/>
-<wire x1="10.16" y1="22.86" x2="5.08" y2="22.86" width="1.27" layer="16"/>
-<wire x1="5.08" y1="22.86" x2="5.08" y2="25.4" width="1.27" layer="16"/>
-<wire x1="12.7" y1="7.62" x2="12.7" y2="12.7" width="1.27" layer="16"/>
+<wire x1="10.16" y1="15.24" x2="15.24" y2="15.24" width="1.27" layer="16"/>
+<wire x1="15.24" y1="15.24" x2="15.24" y2="12.7" width="1.27" layer="16"/>
+<wire x1="15.24" y1="12.7" x2="17.78" y2="12.7" width="1.27" layer="16"/>
+<wire x1="5.08" y1="22.86" x2="7.62" y2="27.94" width="1.27" layer="16"/>
+<wire x1="10.16" y1="15.24" x2="5.08" y2="15.24" width="1.27" layer="16"/>
+<via x="5.08" y="15.24" extent="1-16" drill="0.381"/>
+<wire x1="5.08" y1="15.24" x2="5.08" y2="20.32" width="1.27" layer="1"/>
+<via x="5.08" y="20.32" extent="1-16" drill="0.381"/>
+<wire x1="5.08" y1="20.32" x2="5.08" y2="22.86" width="1.27" layer="16"/>
+<wire x1="10.16" y1="5.08" x2="10.16" y2="7.62" width="1.27" layer="16"/>
+<via x="10.16" y="7.62" extent="1-16" drill="0.381"/>
+<wire x1="10.16" y1="7.62" x2="15.24" y2="7.62" width="1.27" layer="1"/>
+<via x="15.24" y="7.62" extent="1-16" drill="0.381"/>
+<wire x1="15.24" y1="7.62" x2="15.24" y2="12.7" width="1.27" layer="16"/>
 </signal>
 <signal name="GND">
@@
 <contactref element="C2" pad="2"/>
 <contactref element="OUT" pad="1"/>
-<wire x1="10.16" y1="17.78" x2="2.54" y2="17.78" width="1.27" layer="16"/>
-<wire x1="2.54" y1="17.78" x2="2.54" y2="2.54" width="1.27" layer="16"/>
-<wire x1="2.54" y1="2.54" x2="5.08" y2="2.54" width="1.27" layer="16"/>
-<wire x1="5.08" y1="2.54" x2="12.7" y2="2.54" width="1.27" layer="16"/>
-<wire x1="12.7" y1="2.54" x2="17.78" y2="2.54" width="1.27" layer="16"/>
+<wire x1="10.16" y1="17.78" x2="7.62" y2="17.78" width="1.27" layer="16"/>
+<wire x1="7.62" y1="17.78" x2="7.62" y2="10.16" width="1.27" layer="1"/>
+<wire x1="7.62" y1="10.16" x2="5.08" y2="10.16" width="1.27" layer="16"/>
+<wire x1="5.08" y1="10.16" x2="5.08" y2="5.08" width="1.27" layer="16"/>
+<wire x1="5.08" y1="5.08" x2="5.08" y2="2.54" width="1.27" layer="16"/>
+<wire x1="5.08" y1="2.54" x2="17.78" y2="2.54" width="1.27" layer="16"/>
 <wire x1="25.4" y1="2.54" x2="17.78" y2="2.54" width="1.27" layer="16"/>
+<via x="7.62" y="17.78" extent="1-16" drill="0.381"/>
+<via x="7.62" y="10.16" extent="1-16" drill="0.381"/>
 </signal>
 <signal name="N$6">
@@
 <contactref element="IC1" pad="4"/>
 <contactref element="R2" pad="1"/>
-<wire x1="10.16" y1="10.16" x2="10.16" y2="5.08" width="1.27" layer="16"/>
-<wire x1="10.16" y1="5.08" x2="20.32" y2="5.08" width="1.27" layer="16"/>
+<wire x1="10.16" y1="10.16" x2="12.7" y2="10.16" width="1.27" layer="16"/>
+<wire x1="12.7" y1="10.16" x2="12.7" y2="5.08" width="1.27" layer="16"/>
+<wire x1="12.7" y1="5.08" x2="20.32" y2="5.08" width="1.27" layer="16"/>
 <wire x1="20.32" y1="5.08" x2="22.86" y2="5.08" width="1.27" layer="16"/>
 <wire x1="25.4" y1="5.08" x2="22.86" y2="5.08" width="1.27" layer="16"/>
@@
 <contactref element="OUT" pad="2"/>
 <contactref element="IC1" pad="3"/>
-<wire x1="5.08" y1="5.08" x2="5.08" y2="12.7" width="1.27" layer="16"/>
 <wire x1="5.08" y1="12.7" x2="10.16" y2="12.7" width="1.27" layer="16"/>
 </signal>

Commit message: ...
Parts:
- R1: value 1k -> 1kΩ
- R2: value 10k -> 10kΩ
- R3: value 220k -> 220kΩ
Changed lines of the file:
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@@
 <element name="C2" library="c" package="C050-020X036/V" value="10n" x="17.78" y="5.08" rot="R180"/>
 <element name="OUT" library="pad" package="SPAD-+" value="SPAD+--+" x="5.08" y="11.43" rot="R180"/>
-<element name="R1" library="r" package="0207/10" value="1k" x="17.78" y="22.86" rot="R180"/>
-<element name="R2" library="r" package="0207/10" value="10k" x="22.86" y="10.16" rot="R90"/>
-<element name="R3" library="r" package="POT-V" value="220k" x="7.62" y="25.4"/>
+<element name="R1" library="r" package="0207/10" value="1kΩ" x="17.78" y="22.86" rot="R180"/>
+<element name="R2" library="r" package="0207/10" value="10kΩ" x="22.86" y="10.16" rot="R90"/>
+<element name="R3" library="r" package="POT-V" value="220kΩ" x="7.62" y="25.4"/>
 <element name="S1" library="pad" package="PWR-R" value="VCC_GNDPWR-R" x="25.4" y="3.81"/>
 <element name="IC1" library="ic" package="DIL08" value="555" x="13.97" y="13.97"/>
