File: eagle/FM-Radio-Simple-Receiver.sch (EAGLE design)
At the start: 14 parts, among them T1 2N2222, T2 2N2222

Commit message: ...
Parts:
- C1: value (none) -> 100µF
- C3: device cap-trim:C-TR-PH20127 -> cap-trim:C-TR-PH201272222-808-2PIND
- L1: value 200nH -> 0.2µH; device l:L04/7-V -> l:L10/10X
- renumbered 100µF to C1, VR1 to R3
Other:
- moved on the sheet: AF+, AF-
Changed lines of the file:
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@@
 <setting verticaltext="up"/>
 </settings>
-<grid distance="0.1" unitdist="inch" unit="inch" style="lines" multiple="1" display="yes" altdistance="2" altunitdist="inch" altunit="inch"/>
+<grid distance="0.05" unitdist="inch" unit="inch" style="lines" multiple="2" display="yes" altdistance="4" altunitdist="inch" altunit="inch"/>
 <layers>
 <layer number="1" name="Top" color="4" fill="1" visible="yes" active="no"/>
@@
 </classes>
 <parts>
-<part name="T1" library="t" deviceset="2N2222" device=""/>
-<part name="C3" library="cap-trim" deviceset="C-TR-PH20127" device="" value="2 - 20pF"/>
-<part name="L1" library="l" deviceset="L" device="04/7-V" value="200nH"/>
+<part name="C3" library="cap-trim" deviceset="C-TR-PH20127" device="2222-808-2PIND" value="2 - 20pF"/>
+<part name="L1" library="l" deviceset="L" device="10/10X" value="0.2µH"/>
 <part name="T2" library="t" deviceset="2N2222" device=""/>
 <part name="C4" library="c" deviceset="C-H" device="050-020X044" value="220nF"/>
-<part name="VR1" library="r" deviceset="POT" device="" value="10kΩ"/>
+<part name="R3" library="r" deviceset="POT" device="" value="10kΩ"/>
 <part name="R2" library="r" deviceset="R-H" device="0204/10" value="10kΩ"/>
-<part name="AF" library="pad" deviceset="SPAD+-" device="+-" value=""/>
-<part name="BAT" library="pad" deviceset="VCC_GND" device="L" value=""/>
+<part name="AF" library="pad" deviceset="SPAD+-" device="+-" value="SPAD+-+-"/>
+<part name="BAT" library="pad" deviceset="VCC_GND" device="L" value="VCC_GNDL"/>
 <part name="ANT" library="pad" deviceset="ANT" device=""/>
 <part name="C5" library="c" deviceset="C" device="050-020X036/V" value="2.2nF"/>
 <part name="C2" library="c" deviceset="C" device="050-020X036/V" value="100nF"/>
-<part name="100µF" library="c" deviceset="CPOL" device="E2,5-5/V"/>
+<part name="C1" library="c" deviceset="CPOL" device="E2,5-5/V" value="100µF"/>
 <part name="R1" library="r" deviceset="R-H" device="0204/10" value="1kΩ"/>
+<part name="T1" library="t" deviceset="2N2222" device=""/>
+<part name="S1" library="pad" deviceset="GND" device=""/>
 </parts>
 <sheets>
@@
 </plain>
 <instances>
-<instance part="T1" gate="G$1" x="38.1" y="58.42"/>
 <instance part="C3" gate="1" x="27.94" y="53.34"/>
 <instance part="L1" gate="1" x="40.64" y="78.74"/>
 <instance part="T2" gate="G$1" x="50.8" y="68.58"/>
 <instance part="C4" gate="1" x="60.96" y="88.9"/>
-<instance part="VR1" gate="1" x="81.28" y="68.58" rot="MR180"/>
+<instance part="R3" gate="1" x="81.28" y="68.58" rot="MR180"/>
 <instance part="R2" gate="1" x="20.32" y="88.9"/>
-<instance part="AF" gate="-" x="88.9" y="48.26" rot="R180"/>
-<instance part="AF" gate="+" x="88.9" y="68.58" rot="R180"/>
+<instance part="AF" gate="-" x="96.52" y="63.5" rot="R180"/>
+<instance part="AF" gate="+" x="96.52" y="68.58" rot="R180"/>
 <instance part="BAT" gate="1" x="-10.16" y="93.98"/>
 <instance part="BAT" gate="2" x="40.64" y="45.72"/>
@@
 <instance part="C5" gate="1" x="68.58" y="68.58"/>
 <instance part="C2" gate="1" x="12.7" y="68.58"/>
-<instance part="100µF" gate="1" x="5.08" y="68.58"/>
+<instance part="C1" gate="1" x="5.08" y="68.58"/>
 <instance part="R1" gate="1" x="-2.54" y="88.9"/>
+<instance part="T1" gate="G$1" x="38.1" y="58.42"/>
+<instance part="S1" gate="1" x="91.44" y="58.42"/>
 </instances>
 <busses>
@@
 <segment>
 <pinref part="C4" gate="1" pin="2"/>
-<pinref part="VR1" gate="1" pin="A"/>
+<pinref part="R3" gate="1" pin="A"/>
 <wire x1="63.5" y1="88.9" x2="68.58" y2="88.9" width="0.1524" layer="91"/>
 <wire x1="68.58" y1="88.9" x2="81.28" y2="88.9" width="0.1524" layer="91"/>
@@
 <net name="N$6" class="0">
 <segment>
-<pinref part="VR1" gate="1" pin="S"/>
+<pinref part="R3" gate="1" pin="S"/>
 <pinref part="AF" gate="+" pin="P$1"/>
-<wire x1="88.9" y1="68.58" x2="83.82" y2="68.58" width="0.1524" layer="91"/>
+<wire x1="96.52" y1="68.58" x2="83.82" y2="68.58" width="0.1524" layer="91"/>
 </segment>
 </net>
@@
 <segment>
 <pinref part="C3" gate="1" pin="E"/>
-<pinref part="T1" gate="G$1" pin="B"/>
 <wire x1="35.56" y1="58.42" x2="27.94" y2="58.42" width="0.1524" layer="91"/>
 <wire x1="27.94" y1="58.42" x2="27.94" y2="55.88" width="0.1524" layer="91"/>
@@
 <junction x="53.34" y="88.9"/>
 <pinref part="R2" gate="1" pin="2"/>
+<pinref part="T1" gate="G$1" pin="B"/>
 </segment>
 </net>
 <net name="N$5" class="0">
 <segment>
-<pinref part="T1" gate="G$1" pin="C"/>
 <pinref part="L1" gate="1" pin="2"/>
 <wire x1="40.64" y1="71.12" x2="40.64" y2="68.58" width="0.1524" layer="91"/>
@@
 <wire x1="48.26" y1="68.58" x2="40.64" y2="68.58" width="0.1524" layer="91"/>
 <junction x="40.64" y="68.58"/>
+<pinref part="T1" gate="G$1" pin="C"/>
 </segment>
 </net>
@@
 <pinref part="BAT" gate="2" pin="GND"/>
 <wire x1="40.64" y1="48.26" x2="40.64" y2="45.72" width="0.1524" layer="91"/>
-<pinref part="VR1" gate="1" pin="E"/>
-<wire x1="81.28" y1="48.26" x2="81.28" y2="63.5" width="0.1524" layer="91"/>
-<pinref part="AF" gate="-" pin="P$1"/>
-<wire x1="88.9" y1="48.26" x2="81.28" y2="48.26" width="0.1524" layer="91"/>
-<pinref part="T1" gate="G$1" pin="E"/>
+<pinref part="R3" gate="1" pin="E"/>
 <wire x1="40.64" y1="53.34" x2="40.64" y2="48.26" width="0.1524" layer="91"/>
 <wire x1="40.64" y1="48.26" x2="53.34" y2="48.26" width="0.1524" layer="91"/>
-<junction x="81.28" y="48.26"/>
 <pinref part="T2" gate="G$1" pin="E"/>
 <wire x1="53.34" y1="48.26" x2="68.58" y2="48.26" width="0.1524" layer="91"/>
 <wire x1="68.58" y1="48.26" x2="81.28" y2="48.26" width="0.1524" layer="91"/>
+<wire x1="81.28" y1="48.26" x2="81.28" y2="63.5" width="0.1524" layer="91"/>
 <wire x1="53.34" y1="63.5" x2="53.34" y2="48.26" width="0.1524" layer="91"/>
 <junction x="53.34" y="48.26"/>
@@
 <pinref part="C2" gate="1" pin="2"/>
 <wire x1="12.7" y1="48.26" x2="12.7" y2="66.04" width="0.1524" layer="91"/>
-<pinref part="100µF" gate="1" pin="-"/>
+<pinref part="C1" gate="1" pin="-"/>
 <wire x1="5.08" y1="66.04" x2="5.08" y2="48.26" width="0.1524" layer="91"/>
 <wire x1="5.08" y1="48.26" x2="12.7" y2="48.26" width="0.1524" layer="91"/>
 <junction x="12.7" y="48.26"/>
+<pinref part="T1" gate="G$1" pin="E"/>
+</segment>
+<segment>
+<pinref part="AF" gate="-" pin="P$1"/>
+<wire x1="96.52" y1="63.5" x2="91.44" y2="63.5" width="0.1524" layer="91"/>
+<wire x1="91.44" y1="63.5" x2="91.44" y2="58.42" width="0.1524" layer="91"/>
+<pinref part="S1" gate="1" pin="GND"/>
 </segment>
 </net>
@@
 <wire x1="12.7" y1="71.12" x2="12.7" y2="88.9" width="0.1524" layer="91"/>
 <wire x1="12.7" y1="88.9" x2="15.24" y2="88.9" width="0.1524" layer="91"/>
-<pinref part="100µF" gate="1" pin="+"/>
+<pinref part="C1" gate="1" pin="+"/>
 <wire x1="5.08" y1="71.12" x2="5.08" y2="88.9" width="0.1524" layer="91"/>
 <wire x1="5.08" y1="88.9" x2="12.7" y2="88.9" width="0.1524" layer="91"/>
