File: eagle/MotorControllerOpto-BA6229.brd (EAGLE design)
At the start: 35.6 x 20.3 mm, 11 parts, among them IC1 BA6229, J1 CONN-3P-3P

Commit message: ...
Changed lines of the file:
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@@
 <contactref element="C4" pad="-"/>
 <contactref element="J1" pad="1"/>
-<wire x1="2.54" y1="5.08" x2="7.62" y2="5.08" width="0.6096" layer="16"/>
-<wire x1="12.7" y1="5.08" x2="27.94" y2="5.08" width="0.6096" layer="16"/>
-<wire x1="27.94" y1="5.08" x2="30.48" y2="5.08" width="0.6096" layer="16"/>
-<wire x1="15.24" y1="5.08" x2="30.48" y2="5.08" width="0.6096" layer="16"/>
-<wire x1="15.24" y1="5.08" x2="12.7" y2="5.08" width="0.6096" layer="16"/>
-<wire x1="2.54" y1="17.78" x2="7.62" y2="17.78" width="0.6096" layer="16"/>
-<wire x1="12.7" y1="5.08" x2="7.62" y2="5.08" width="0.6096" layer="16"/>
-<wire x1="7.62" y1="5.08" x2="7.62" y2="17.78" width="0.6096" layer="16"/>
+<wire x1="2.54" y1="5.08" x2="7.62" y2="5.08" width="1.27" layer="16"/>
+<wire x1="12.7" y1="5.08" x2="27.94" y2="5.08" width="1.27" layer="16"/>
+<wire x1="27.94" y1="5.08" x2="30.48" y2="5.08" width="1.27" layer="16"/>
+<wire x1="15.24" y1="5.08" x2="30.48" y2="5.08" width="1.27" layer="16"/>
+<wire x1="15.24" y1="5.08" x2="12.7" y2="5.08" width="1.27" layer="16"/>
+<wire x1="2.54" y1="17.78" x2="7.62" y2="17.78" width="1.27" layer="16"/>
+<wire x1="12.7" y1="5.08" x2="7.62" y2="5.08" width="1.27" layer="16"/>
+<wire x1="7.62" y1="5.08" x2="7.62" y2="17.78" width="1.27" layer="16"/>
 </signal>
 <signal name="N$2">
 <contactref element="C2" pad="1"/>
 <contactref element="IC1" pad="9"/>
-<wire x1="27.94" y1="10.16" x2="27.94" y2="17.78" width="0.6096" layer="16"/>
+<wire x1="27.94" y1="10.16" x2="27.94" y2="17.78" width="1.27" layer="16"/>
 </signal>
 <signal name="N$3">
 <contactref element="C1" pad="1"/>
 <contactref element="IC1" pad="3"/>
-<wire x1="12.7" y1="10.16" x2="12.7" y2="17.78" width="0.6096" layer="16"/>
+<wire x1="12.7" y1="10.16" x2="12.7" y2="17.78" width="1.27" layer="16"/>
 </signal>
 <signal name="N$4">
 <contactref element="IC1" pad="4"/>
 <contactref element="D1" pad="C"/>
-<wire x1="15.24" y1="17.78" x2="15.24" y2="10.16" width="0.6096" layer="16"/>
+<wire x1="15.24" y1="17.78" x2="15.24" y2="10.16" width="1.27" layer="16"/>
 </signal>
 <signal name="N$1">
@@
 <contactref element="MOTOR" pad="2"/>
 <contactref element="C3" pad="1"/>
-<wire x1="33.02" y1="7.62" x2="30.48" y2="7.62" width="0.6096" layer="16"/>
-<wire x1="30.48" y1="7.62" x2="10.16" y2="7.62" width="0.6096" layer="16"/>
-<wire x1="10.16" y1="7.62" x2="10.16" y2="17.78" width="0.6096" layer="16"/>
-<wire x1="10.16" y1="19.05" x2="10.16" y2="17.78" width="0.6096" layer="16"/>
+<wire x1="33.02" y1="7.62" x2="30.48" y2="7.62" width="1.27" layer="16"/>
+<wire x1="30.48" y1="7.62" x2="10.16" y2="7.62" width="1.27" layer="16"/>
+<wire x1="10.16" y1="7.62" x2="10.16" y2="17.78" width="1.27" layer="16"/>
+<wire x1="10.16" y1="19.05" x2="10.16" y2="17.78" width="1.27" layer="16"/>
 </signal>
 <signal name="N$6">
@@
 <contactref element="IC1" pad="10"/>
 <contactref element="C3" pad="2"/>
-<wire x1="33.02" y1="10.16" x2="33.02" y2="12.7" width="0.6096" layer="16"/>
-<wire x1="30.48" y1="17.78" x2="33.02" y2="17.78" width="0.6096" layer="16"/>
-<wire x1="33.02" y1="17.78" x2="33.02" y2="12.7" width="0.6096" layer="16"/>
-<wire x1="33.02" y1="12.7" x2="30.48" y2="12.7" width="0.6096" layer="16"/>
+<wire x1="33.02" y1="10.16" x2="33.02" y2="12.7" width="1.27" layer="16"/>
+<wire x1="30.48" y1="17.78" x2="33.02" y2="17.78" width="1.27" layer="16"/>
+<wire x1="33.02" y1="17.78" x2="33.02" y2="12.7" width="1.27" layer="16"/>
+<wire x1="33.02" y1="12.7" x2="30.48" y2="12.7" width="1.27" layer="16"/>
 </signal>
 <signal name="N$8">
 <contactref element="IC1" pad="8"/>
 <contactref element="R1" pad="1"/>
-<wire x1="25.4" y1="10.16" x2="25.4" y2="17.78" width="0.6096" layer="16"/>
+<wire x1="25.4" y1="10.16" x2="25.4" y2="17.78" width="1.27" layer="16"/>
 </signal>
 <signal name="VCC">
@@
 <contactref element="PWR" pad="2"/>
 <contactref element="C4" pad="+"/>
-<wire x1="22.86" y1="17.78" x2="22.86" y2="12.7" width="0.6096" layer="16"/>
-<wire x1="22.86" y1="12.7" x2="22.86" y2="2.54" width="0.6096" layer="1"/>
-<wire x1="22.86" y1="2.54" x2="2.54" y2="2.54" width="0.6096" layer="16"/>
+<wire x1="22.86" y1="17.78" x2="22.86" y2="12.7" width="1.27" layer="16"/>
+<wire x1="22.86" y1="12.7" x2="22.86" y2="2.54" width="1.27" layer="1"/>
+<wire x1="22.86" y1="2.54" x2="2.54" y2="2.54" width="1.27" layer="16"/>
 <via x="22.86" y="12.7" extent="1-16" drill="0.6" shape="square"/>
 <via x="22.86" y="2.54" extent="1-16" drill="0.6" shape="square"/>
-<wire x1="22.86" y1="2.54" x2="25.4" y2="2.54" width="0.6096" layer="16"/>
-<wire x1="22.86" y1="2.54" x2="30.48" y2="2.54" width="0.6096" layer="16"/>
+<wire x1="22.86" y1="2.54" x2="25.4" y2="2.54" width="1.27" layer="16"/>
+<wire x1="22.86" y1="2.54" x2="30.48" y2="2.54" width="1.27" layer="16"/>
 </signal>
 <signal name="N$5">
 <contactref element="IC1" pad="5"/>
 <contactref element="J1" pad="2"/>
-<wire x1="2.54" y1="15.24" x2="5.08" y2="15.24" width="0.6096" layer="16"/>
+<wire x1="2.54" y1="15.24" x2="5.08" y2="15.24" width="1.27" layer="16"/>
 <via x="5.08" y="15.24" extent="1-16" drill="0.6" shape="square"/>
-<wire x1="5.08" y1="15.24" x2="17.78" y2="15.24" width="0.6096" layer="1"/>
+<wire x1="5.08" y1="15.24" x2="17.78" y2="15.24" width="1.27" layer="1"/>
 <via x="17.78" y="15.24" extent="1-16" drill="0.6" shape="square"/>
-<wire x1="17.78" y1="15.24" x2="17.78" y2="17.78" width="0.6096" layer="16"/>
+<wire x1="17.78" y1="15.24" x2="17.78" y2="17.78" width="1.27" layer="16"/>
 </signal>
 <signal name="N$7">
 <contactref element="J1" pad="3"/>
 <contactref element="IC1" pad="6"/>
-<wire x1="2.54" y1="12.7" x2="5.08" y2="12.7" width="0.6096" layer="16"/>
+<wire x1="2.54" y1="12.7" x2="5.08" y2="12.7" width="1.27" layer="16"/>
 <via x="5.08" y="12.7" extent="1-16" drill="0.6" shape="square"/>
-<wire x1="5.08" y1="12.7" x2="20.32" y2="12.7" width="0.6096" layer="1"/>
+<wire x1="5.08" y1="12.7" x2="20.32" y2="12.7" width="1.27" layer="1"/>
 <via x="20.32" y="12.7" extent="1-16" drill="0.6" shape="square"/>
-<wire x1="20.32" y1="12.7" x2="20.32" y2="17.78" width="0.6096" layer="16"/>
+<wire x1="20.32" y1="12.7" x2="20.32" y2="17.78" width="1.27" layer="16"/>
 </signal>
 </signals>

Commit message: ...
Other:
- board outline removed
Changed lines of the file:
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@@
 http://beatsdownloadg5.hatenablog.com/entry/reversible-motor-driver-circuit</description>
 <plain>
-<wire x1="0" y1="0" x2="35.56" y2="0" width="0" layer="20"/>
-<wire x1="35.56" y1="0" x2="35.56" y2="20.32" width="0" layer="20"/>
-<wire x1="35.56" y1="20.32" x2="0" y2="20.32" width="0" layer="20"/>
-<wire x1="0" y1="20.32" x2="0" y2="0" width="0" layer="20"/>
+<wire x1="0" y1="0" x2="35.56" y2="0" width="0" layer="47"/>
+<wire x1="35.56" y1="0" x2="35.56" y2="20.32" width="0" layer="47"/>
+<wire x1="35.56" y1="20.32" x2="0" y2="20.32" width="0" layer="47"/>
+<wire x1="0" y1="20.32" x2="0" y2="0" width="0" layer="47"/>
 </plain>
 <attributes>

Commit message: ...
Parts:
- C1, C2: value 0.1uF -> 0.1μF
- C3: value 0.33uF -> 0.33μF
- C4: value 100uF -> 100μF
- R1: value 10 -> 10Ω
Changed lines of the file:
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@@
 </autorouter>
 <elements>
-<element name="C1" library="c" package="C050-020X044" value="0.1uF" x="12.7" y="7.62" rot="R90"/>
-<element name="C2" library="c" package="C050-020X044" value="0.1uF" x="27.94" y="7.62" rot="R90"/>
-<element name="C3" library="c" package="C050-020X044" value="0.33uF" x="30.48" y="10.16" rot="R270"/>
-<element name="C4" library="c" package="E2,5-4" value="100uF" x="30.48" y="3.81" rot="R180"/>
+<element name="C1" library="c" package="C050-020X044" value="0.1μF" x="12.7" y="7.62" rot="R90"/>
+<element name="C2" library="c" package="C050-020X044" value="0.1μF" x="27.94" y="7.62" rot="R90"/>
+<element name="C3" library="c" package="C050-020X044" value="0.33μF" x="30.48" y="10.16" rot="R270"/>
+<element name="C4" library="c" package="E2,5-4" value="100μF" x="30.48" y="3.81" rot="R180"/>
 <element name="D1" library="d" package="DO34Z5V" value="Z=4.7V" x="15.24" y="7.62" rot="R180"/>
 <element name="IC1" library="ic" package="SIL10" value="BA6229" x="19.05" y="17.78" rot="R90"/>
@@
 <element name="MOTOR" library="pad" package="SPAD+-" value="SPAD+-" x="33.02" y="8.89" rot="R180"/>
 <element name="PWR" library="pad" package="SPAD+-" value="SPAD+-" x="2.54" y="3.81" rot="R180"/>
-<element name="R1" library="r" package="0204/7-V" value="10" x="25.4" y="6.35"/>
+<element name="R1" library="r" package="0204/7-V" value="10Ω" x="25.4" y="6.35"/>
 <element name="OK1" library="optocoupler" package="DIL08" value="HCPL2730" x="-7.62" y="7.62">
 <attribute name="MPN" value="HCPL-2730-000E" x="-7.62" y="7.62" size="1.778" layer="27" display="off"/>

Commit message: ...
Other:
- board outline added: 35.6 x 20.3 mm
Changed lines of the file:
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@@
 http://beatsdownloadg5.hatenablog.com/entry/reversible-motor-driver-circuit</description>
 <plain>
-<wire x1="0" y1="0" x2="35.56" y2="0" width="0" layer="47"/>
-<wire x1="35.56" y1="0" x2="35.56" y2="20.32" width="0" layer="47"/>
-<wire x1="35.56" y1="20.32" x2="0" y2="20.32" width="0" layer="47"/>
-<wire x1="0" y1="20.32" x2="0" y2="0" width="0" layer="47"/>
+<wire x1="0" y1="0" x2="35.56" y2="0" width="0" layer="20"/>
+<wire x1="35.56" y1="0" x2="35.56" y2="20.32" width="0" layer="20"/>
+<wire x1="35.56" y1="20.32" x2="0" y2="20.32" width="0" layer="20"/>
+<wire x1="0" y1="20.32" x2="0" y2="0" width="0" layer="20"/>
 </plain>
 <attributes>
