File: eagle/Cellphone-Detector-LM358.brd (EAGLE design)
At the start: 38.1 x 76.2 mm, 10 parts, among them IC1 LM358N

Commit message: ...
Parts:
- C1: device c:C050-025X075/V -> c:C025-024X044
- R1: device r:0204/10-V -> r:0202/7-V
- R2: device r:POT -> r:POT-V
- S1: value VCC_GNDPWR-L -> VCC_GNDPWR-R; device pad:PWR-L -> pad:PWR-R
- moved R2 28.5 mm to (6.35, 17.8), turned to 180 degrees
- moved R4 27.4 mm to (33.0, 7.62), turned to 180 degrees
- moved ANT1 20.5 mm to (5.08, 10.2)
- moved R3 17.0 mm to (17.8, 7.62), turned to 180 degrees
- moved T1 17.0 mm to (35.6, 10.2)
- moved U$1 13.0 mm to (40.6, 6.35)
- moved S1 10.9 mm to (5.08, 3.81), turned to 180 degrees
- moved IC1 9.16 mm to (24.1, 11.4)
- moved C1 8.52 mm to (15.2, 11.4), turned to 90 degrees
- moved R1 8.52 mm to (10.2, 8.89)
Routing:
- net N$5: track 20.3 -> 72.4 mm, vias 0 -> 2
- net VCC: track 2.54 -> 43.2 mm, vias 1 -> 4
- net GND: track 0.00 -> 38.1 mm
- net N$2: track 53.3 -> 26.7 mm, vias 2 -> 3
- net N$3: track 0.00 -> 10.2 mm
- net N$7: track 0.00 -> 5.08 mm
- net N$6: track 0.00 -> 2.54 mm
Other:
- board size 38.1 x 76.2 mm -> 43.2 x 22.9 mm
Changed lines of the file:
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@@
 <board>
 <plain>
-<wire x1="0" y1="0" x2="38.1" y2="0" width="0" layer="20"/>
-<wire x1="38.1" y1="0" x2="38.1" y2="76.2" width="0" layer="20"/>
-<wire x1="38.1" y1="76.2" x2="0" y2="76.2" width="0" layer="20"/>
-<wire x1="0" y1="76.2" x2="0" y2="0" width="0" layer="20"/>
+<wire x1="0" y1="0" x2="43.18" y2="0" width="0" layer="20"/>
+<wire x1="43.18" y1="0" x2="43.18" y2="22.86" width="0" layer="20"/>
+<wire x1="43.18" y1="22.86" x2="0" y2="22.86" width="0" layer="20"/>
+<wire x1="0" y1="22.86" x2="0" y2="0" width="0" layer="20"/>
 </plain>
 <attributes>
@@
 </autorouter>
 <elements>
-<element name="ANT1" library="pad" package="SPAD" value="ANT" x="2.54" y="30.48"/>
-<element name="C1" library="c" package="C050-025X075/V" value="1µF" x="7.62" y="15.24" rot="R180"/>
-<element name="IC1" library="ic" package="DIL08" value="LM358N" x="16.51" y="16.51"/>
-<element name="R1" library="r" package="0204/10-V" value="100kΩ" x="2.54" y="12.7"/>
-<element name="R2" library="r" package="POT" value="1MΩ" x="33.02" y="27.94" rot="R90"/>
-<element name="R3" library="r" package="0204/10-V" value="220kΩ" x="10.16" y="22.86"/>
-<element name="R4" library="r" package="0204/10-V" value="1kΩ" x="22.86" y="33.02" rot="R90"/>
-<element name="S1" library="pad" package="PWR-L" value="VCC_GNDPWR-L" x="-5.08" y="7.62"/>
-<element name="T1" library="t" package="TO92" value="" x="27.94" y="25.4"/>
-<element name="U$1" library="d" package="LED_3MM/V" value="LED-3MM/V" x="27.94" y="8.89"/>
+<element name="ANT1" library="pad" package="SPAD" value="ANT" x="5.08" y="10.16"/>
+<element name="C1" library="c" package="C025-024X044" value="1µF" x="15.24" y="11.43" rot="R90"/>
+<element name="IC1" library="ic" package="DIL08" value="LM358N" x="24.13" y="11.43"/>
+<element name="R1" library="r" package="0202/7-V" value="100kΩ" x="10.16" y="8.89"/>
+<element name="R2" library="r" package="POT-V" value="1MΩ" x="6.35" y="17.78" rot="R180"/>
+<element name="R3" library="r" package="0204/10-V" value="220kΩ" x="17.78" y="7.62" rot="R180"/>
+<element name="R4" library="r" package="0204/10-V" value="1kΩ" x="33.02" y="7.62" rot="R180"/>
+<element name="S1" library="pad" package="PWR-R" value="VCC_GNDPWR-R" x="5.08" y="3.81" rot="R180"/>
+<element name="T1" library="t" package="TO92" value="" x="35.56" y="10.16"/>
+<element name="U$1" library="d" package="LED_3MM/V" value="LED-3MM/V" x="40.64" y="6.35"/>
 </elements>
 <signals>
@@
 <contactref element="R1" pad="2"/>
 <contactref element="IC1" pad="4"/>
-<wire x1="12.7" y1="12.7" x2="27.94" y2="7.62" width="0" layer="19" extent="1-1"/>
-<wire x1="2.54" y1="7.62" x2="12.7" y2="12.7" width="0" layer="19" extent="1-1"/>
-<wire x1="-5.08" y1="7.62" x2="2.54" y2="7.62" width="0" layer="19" extent="1-1"/>
+<wire x1="40.64" y1="5.08" x2="20.32" y2="5.08" width="0.8128" layer="16"/>
+<wire x1="20.32" y1="7.62" x2="20.32" y2="5.08" width="0.8128" layer="16"/>
+<wire x1="20.32" y1="5.08" x2="10.16" y2="5.08" width="0.8128" layer="16"/>
+<wire x1="10.16" y1="5.08" x2="10.16" y2="5.08" width="0" layer="19" extent="1-16"/>
+<wire x1="5.08" y1="5.08" x2="10.16" y2="5.08" width="0.8128" layer="16"/>
 </signal>
 <signal name="N$2">
@@
 <contactref element="IC1" pad="3"/>
 <contactref element="R2" pad="S"/>
-<wire x1="33.02" y1="27.94" x2="33.02" y2="30.48" width="0.8128" layer="16"/>
-<wire x1="33.02" y1="30.48" x2="5.08" y2="30.48" width="0.8128" layer="16"/>
-<via x="5.08" y="30.48" extent="1-16" drill="0.6" shape="square"/>
-<wire x1="5.08" y1="30.48" x2="5.08" y2="15.24" width="0.8128" layer="1"/>
-<via x="5.08" y="15.24" extent="1-16" drill="0.6" shape="square"/>
-<wire x1="12.7" y1="15.24" x2="5.08" y2="15.24" width="0.8128" layer="16"/>
-<wire x1="5.08" y1="30.48" x2="2.54" y2="30.48" width="0" layer="19" extent="16-16"/>
-<wire x1="7.62" y1="12.7" x2="5.08" y2="15.24" width="0" layer="19" extent="1-1"/>
+<via x="12.7" y="10.16" extent="1-16" drill="0.6" shape="square"/>
+<via x="12.7" y="10.16" extent="1-16" drill="0.6" shape="square"/>
+<wire x1="6.35" y1="15.24" x2="12.7" y2="15.24" width="0.8128" layer="16"/>
+<wire x1="12.7" y1="15.24" x2="12.7" y2="10.16" width="0.8128" layer="1"/>
+<wire x1="20.32" y1="10.16" x2="12.7" y2="10.16" width="0.8128" layer="16"/>
+<wire x1="15.24" y1="10.16" x2="12.7" y2="10.16" width="0" layer="19" extent="1-1"/>
+<wire x1="12.7" y1="10.16" x2="5.08" y2="10.16" width="0.8128" layer="16"/>
+<via x="12.7" y="15.24" extent="1-16" drill="0.6" shape="square"/>
 </signal>
 <signal name="N$3">
@@
 <contactref element="R1" pad="1"/>
 <contactref element="R3" pad="2"/>
-<wire x1="10.16" y1="17.78" x2="12.7" y2="17.78" width="0" layer="19" extent="1-1"/>
-<wire x1="7.62" y1="17.78" x2="10.16" y2="17.78" width="0" layer="19" extent="1-1"/>
-<wire x1="2.54" y1="17.78" x2="7.62" y2="17.78" width="0" layer="19" extent="1-1"/>
+<wire x1="20.32" y1="12.7" x2="17.78" y2="12.7" width="0.8128" layer="16"/>
+<wire x1="17.78" y1="12.7" x2="15.24" y2="12.7" width="0.8128" layer="16"/>
+<wire x1="15.24" y1="12.7" x2="10.16" y2="12.7" width="0.8128" layer="16"/>
 </signal>
 <signal name="VCC">
@@
 <contactref element="R3" pad="1"/>
 <contactref element="R4" pad="1"/>
-<wire x1="10.16" y1="27.94" x2="17.78" y2="33.02" width="0" layer="19" extent="1-1"/>
-<wire x1="-5.08" y1="10.16" x2="10.16" y2="27.94" width="0" layer="19" extent="1-1"/>
-<wire x1="20.32" y1="20.32" x2="22.86" y2="20.32" width="0.8128" layer="16"/>
-<via x="22.86" y="20.32" extent="1-16" drill="0.6" shape="square"/>
-<wire x1="22.86" y1="20.32" x2="17.78" y2="33.02" width="0" layer="19" extent="1-16"/>
+<wire x1="27.94" y1="15.24" x2="30.48" y2="15.24" width="0.8128" layer="16"/>
+<via x="30.48" y="15.24" extent="1-16" drill="0.6" shape="square"/>
+<wire x1="17.78" y1="2.54" x2="30.48" y2="2.54" width="0.8128" layer="16"/>
+<wire x1="30.48" y1="2.54" x2="30.48" y2="15.24" width="0.8128" layer="1"/>
+<via x="30.48" y="2.54" extent="1-16" drill="0.6" shape="square"/>
+<wire x1="33.02" y1="2.54" x2="30.48" y2="2.54" width="0.8128" layer="16"/>
+<wire x1="17.78" y1="2.54" x2="8.89" y2="2.54" width="0.8128" layer="16"/>
+<wire x1="8.89" y1="2.54" x2="5.08" y2="2.54" width="0.8128" layer="16"/>
+<via x="8.89" y="2.54" extent="1-16" drill="0.6" shape="square"/>
+<via x="8.89" y="2.54" extent="1-16" drill="0.6" shape="square"/>
 </signal>
 <signal name="N$5">
@@
 <contactref element="T1" pad="2"/>
 <contactref element="R2" pad="A"/>
-<wire x1="12.7" y1="20.32" x2="12.7" y2="25.4" width="0.8128" layer="16"/>
-<wire x1="12.7" y1="25.4" x2="27.94" y2="25.4" width="0.8128" layer="16"/>
-<wire x1="27.94" y1="25.4" x2="33.02" y2="25.4" width="0" layer="19" extent="1-1"/>
+<wire x1="20.32" y1="15.24" x2="20.32" y2="20.32" width="0.8128" layer="16"/>
+<wire x1="20.32" y1="20.32" x2="40.64" y2="20.32" width="0.8128" layer="16"/>
+<wire x1="8.89" y1="20.32" x2="40.64" y2="20.32" width="0.8128" layer="16"/>
+<via x="40.64" y="20.32" extent="1-16" drill="0.6" shape="square"/>
+<wire x1="40.64" y1="20.32" x2="40.64" y2="10.16" width="0.8128" layer="1"/>
+<via x="40.64" y="10.16" extent="1-16" drill="0.6" shape="square"/>
+<wire x1="40.64" y1="10.16" x2="35.56" y2="10.16" width="0.8128" layer="16"/>
 </signal>
 <signal name="N$6">
 <contactref element="R4" pad="2"/>
 <contactref element="T1" pad="1"/>
-<wire x1="27.94" y1="27.94" x2="27.94" y2="33.02" width="0" layer="19" extent="1-1"/>
+<wire x1="35.56" y1="12.7" x2="33.02" y2="12.7" width="0.8128" layer="16"/>
 </signal>
 <signal name="N$7">
 <contactref element="T1" pad="3"/>
 <contactref element="U$1" pad="A"/>
-<wire x1="27.94" y1="10.16" x2="27.94" y2="22.86" width="0" layer="19" extent="1-1"/>
+<wire x1="40.64" y1="7.62" x2="35.56" y2="7.62" width="0.8128" layer="16"/>
 </signal>
 </signals>
