File: eagle/Super-Regenerative-FM.sch (EAGLE design)
At the start: 15 parts, among them Q1 BF245B

Commit message: ...
Parts:
- removed Q1: BF245B, t:BF245B
- added T1: BF256B, t:BF256B
Connections:
- net GND: now also T1.G; no longer Q1.G
- net N$2: now also T1.D; no longer Q1.D
- net N$5: now also T1.S; no longer Q1.S
Changed lines of the file:
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@@
 </classes>
 <parts>
-<part name="Q1" library="t" deviceset="BF245B" device=""/>
 <part name="C3" library="cap-trim" deviceset="C-TR-PH20127" device="2222-808-2PIN" value="15p"/>
 <part name="C1" library="c" deviceset="C" device="050-020X036/V" value="1n"/>
@@
 <part name="U$5" library="pad" deviceset="GND" device=""/>
 <part name="L1" library="l" deviceset="L-TAP1" device="L-08/12-X-TAP1" value="0.22μH"/>
+<part name="T1" library="t" deviceset="BF256B" device=""/>
 </parts>
 <sheets>
@@
 </plain>
 <instances>
-<instance part="Q1" gate="1" x="55.88" y="60.96"/>
 <instance part="C3" gate="1" x="48.26" y="50.8" rot="MR180"/>
 <instance part="C1" gate="1" x="22.86" y="50.8" rot="MR0"/>
@@
 <instance part="U$5" gate="1" x="7.62" y="35.56" rot="MR0"/>
 <instance part="L1" gate="1" x="35.56" y="60.96"/>
+<instance part="T1" gate="1" x="55.88" y="60.96" rot="R90"/>
 </instances>
 <busses>
@@
 <net name="GND" class="0">
 <segment>
-<pinref part="Q1" gate="1" pin="G"/>
 <pinref part="U$2" gate="1" pin="GND"/>
 <wire x1="55.88" y1="53.34" x2="55.88" y2="40.64" width="0.1524" layer="91"/>
@@
 <pinref part="C3" gate="1" pin="E"/>
 <wire x1="48.26" y1="48.26" x2="48.26" y2="40.64" width="0.1524" layer="91"/>
+<pinref part="T1" gate="1" pin="G"/>
 </segment>
 <segment>
@@
 <net name="N$2" class="0">
 <segment>
-<pinref part="Q1" gate="1" pin="D"/>
 <wire x1="48.26" y1="60.96" x2="50.8" y2="60.96" width="0.1524" layer="91"/>
 <wire x1="43.18" y1="60.96" x2="48.26" y2="60.96" width="0.1524" layer="91"/>
@@
 <wire x1="48.26" y1="60.96" x2="48.26" y2="53.34" width="0.1524" layer="91"/>
 <pinref part="L1" gate="1" pin="2"/>
+<pinref part="T1" gate="1" pin="D"/>
 </segment>
 </net>
@@
 <wire x1="58.42" y1="71.12" x2="63.5" y2="71.12" width="0.1524" layer="91"/>
 <wire x1="63.5" y1="71.12" x2="63.5" y2="60.96" width="0.1524" layer="91"/>
-<pinref part="Q1" gate="1" pin="S"/>
 <wire x1="63.5" y1="60.96" x2="60.96" y2="60.96" width="0.1524" layer="91"/>
 <pinref part="L2" gate="1" pin="2"/>
 <wire x1="63.5" y1="60.96" x2="66.04" y2="60.96" width="0.1524" layer="91"/>
 <junction x="63.5" y="60.96"/>
+<pinref part="T1" gate="1" pin="S"/>
 </segment>
 </net>
