File: eagle/Mind-Synchronizing-Generator-PinHdrPot.sch (EAGLE design)
At the start: 30 parts, among them IC1 555, IC2 555, IC3 555, J1 MONO-JACK, J2 AUDIO_JACK, J3 MONO-JACK

Commit message: ...
Parts:
- J1: value MONO-JACK -> SPAD+--+; device pad:MONO-JACK -> pad:SPAD+--+
- J3: value MONO-JACK -> SPAD-2; device pad:MONO-JACK -> pad:SPAD-2
Connections:
- net N$18: now also J1-.P$1; no longer J1.SLEEVE
- net N$4: now also J1+.P$1; no longer J1.LEFT
- net N$6: now also J3-2.P$1; no longer J3.LEFT
- net Q1: now also J3-1.P$1; no longer J3.SLEEVE
Other:
- moved on the sheet: R12
Changed lines of the file:
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@@
 <part name="S13" library="pad" deviceset="GND" device=""/>
 <part name="J2" library="pad" deviceset="AUDIO_JACK" device=""/>
-<part name="J1" library="pad" deviceset="MONO-JACK" device=""/>
-<part name="J3" library="pad" deviceset="MONO-JACK" device=""/>
+<part name="J1" library="pad" deviceset="SPAD+-" device="-+" value="SPAD+--+"/>
+<part name="J3" library="pad" deviceset="SPAD-2" device=""/>
 </parts>
 <sheets>
@@
 <instance part="BATT" gate="+" x="-48.26" y="40.64"/>
 <instance part="S" gate="1" x="-43.18" y="24.13" rot="MR270"/>
-<instance part="R12" gate="1" x="60.96" y="-5.08"/>
+<instance part="R12" gate="1" x="63.5" y="-5.08"/>
 <instance part="S11" gate="1" x="50.8" y="-7.62"/>
 <instance part="S12" gate="1" x="132.08" y="20.32"/>
 <instance part="S13" gate="1" x="96.52" y="20.32"/>
 <instance part="J2" gate="G$1" x="157.48" y="33.02" rot="R180"/>
-<instance part="J1" gate="G$1" x="83.82" y="-2.54" rot="R180"/>
-<instance part="J3" gate="G$1" x="-53.34" y="88.9"/>
+<instance part="J1" gate="-" x="78.74" y="-5.08" rot="R180"/>
+<instance part="J1" gate="+" x="78.74" y="0" rot="R180"/>
+<instance part="J3" gate="-1" x="-48.26" y="91.44"/>
+<instance part="J3" gate="-2" x="-48.26" y="86.36"/>
 </instances>
 <busses>
@@
 <pinref part="R12" gate="1" pin="1"/>
 <pinref part="S11" gate="1" pin="GND"/>
-<wire x1="55.88" y1="-5.08" x2="50.8" y2="-5.08" width="0.1524" layer="91"/>
+<wire x1="58.42" y1="-5.08" x2="50.8" y2="-5.08" width="0.1524" layer="91"/>
 <wire x1="50.8" y1="-5.08" x2="50.8" y2="-7.62" width="0.1524" layer="91"/>
 </segment>
@@
 <wire x1="7.62" y1="78.74" x2="10.16" y2="78.74" width="0.1524" layer="91"/>
 <junction x="7.62" y="78.74"/>
-<pinref part="J3" gate="G$1" pin="SLEEVE"/>
 <wire x1="-48.26" y1="91.44" x2="10.16" y2="91.44" width="0.1524" layer="91"/>
+<pinref part="J3" gate="-1" pin="P$1"/>
 </segment>
 </net>
@@
 <wire x1="-20.32" y1="30.48" x2="-20.32" y2="40.64" width="0.1524" layer="91"/>
 <junction x="-20.32" y="40.64"/>
-<pinref part="J3" gate="G$1" pin="LEFT"/>
 <wire x1="-48.26" y1="86.36" x2="-20.32" y2="86.36" width="0.1524" layer="91"/>
+<pinref part="J3" gate="-2" pin="P$1"/>
 </segment>
 </net>
@@
 <segment>
 <pinref part="R12" gate="1" pin="2"/>
-<wire x1="78.74" y1="-5.08" x2="66.04" y2="-5.08" width="0.1524" layer="91"/>
-<pinref part="J1" gate="G$1" pin="SLEEVE"/>
+<wire x1="78.74" y1="-5.08" x2="68.58" y2="-5.08" width="0.1524" layer="91"/>
+<pinref part="J1" gate="-" pin="P$1"/>
 </segment>
 </net>
@@
 <pinref part="R7" gate="1" pin="E"/>
 <wire x1="68.58" y1="7.62" x2="68.58" y2="0" width="0.1524" layer="91"/>
-<pinref part="J1" gate="G$1" pin="LEFT"/>
-</segment>
-</net>
+<pinref part="J1" gate="+" pin="P$1"/>
+</segment>
+</net>

Commit message: ...
Parts:
- C1: device c:CPOLE2.5-6 -> c:CPOLE5-8.5
Connections:
- net GND: now also J2.LEFT; no longer J2.SLEEVE
- net N$16: now also J2.SLEEVE; no longer J2.LEFT
Other:
- moved on the sheet: J2
