File: eagle/Aurel-super-regen-receiver-ASR2.brd (EAGLE design)
At the start: 43.2 x 25.4 mm, 18 parts, among them T1 2N2222

Commit message: ...
Parts:
- R1, R3: value 10kΩ -> 10kΩ
- R2, R4, R5, R6: value 1kΩ -> 1kΩ
Changed lines of the file:
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@@
 <element name="AF" library="pad" package="SPAD+-" value="" x="40.64" y="3.81"/>
 <element name="L1" library="l" package="L-04/7-V" value="200nH" x="12.7" y="6.35"/>
-<element name="R1" library="r" package="POT" value="10kΩ" x="38.1" y="20.32" rot="R90"/>
-<element name="R2" library="r" package="0204/10-V" value="1kΩ" x="33.02" y="7.62"/>
-<element name="R3" library="r" package="0204/10" value="10kΩ" x="30.48" y="22.86" rot="R180"/>
-<element name="R4" library="r" package="0204/10-V" value="1kΩ" x="20.32" y="17.78"/>
-<element name="R5" library="r" package="0204/10-V" value="1kΩ" x="22.86" y="15.24"/>
-<element name="R6" library="r" package="0204/10" value="1kΩ" x="30.48" y="15.24"/>
+<element name="R1" library="r" package="POT" value="10kΩ" x="38.1" y="20.32" rot="R90"/>
+<element name="R2" library="r" package="0204/10-V" value="1kΩ" x="33.02" y="7.62"/>
+<element name="R3" library="r" package="0204/10" value="10kΩ" x="30.48" y="22.86" rot="R180"/>
+<element name="R4" library="r" package="0204/10-V" value="1kΩ" x="20.32" y="17.78"/>
+<element name="R5" library="r" package="0204/10-V" value="1kΩ" x="22.86" y="15.24"/>
+<element name="R6" library="r" package="0204/10" value="1kΩ" x="30.48" y="15.24"/>
 <element name="S2" library="pad" package="PWR-L" value="" x="2.54" y="21.59" rot="R180"/>
 <element name="T1" library="t" package="TO92-EBC" value="2N2222" x="25.4" y="10.16" rot="R180"/>
