File: eagle/RX-FM-Radio-Circuit.sch (EAGLE design)
At the start: 10 parts, among them T1 2N2222, T2 2N2222

Commit message: ...
Parts:
- added U$1: (no value), l:L-ALT-TEST
Changed lines of the file:
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@@
 <part name="BAT" library="pad" deviceset="VCC_GND" device="L" value=""/>
 <part name="ANT" library="pad" deviceset="ANT" device=""/>
+<part name="U$1" library="l" deviceset="L-ALT" device="-TEST"/>
 </parts>
 <sheets>
@@
 <instance part="T1" gate="G$1" x="27.94" y="68.58" rot="MR0"/>
 <instance part="C1" gate="1" x="38.1" y="78.74"/>
-<instance part="L1" gate="1" x="50.8" y="78.74"/>
+<instance part="L1" gate="G$1" x="50.8" y="78.74"/>
 <instance part="T2" gate="G$1" x="53.34" y="60.96" rot="MR0"/>
 <instance part="C2" gate="1" x="68.58" y="60.96"/>
@@
 <instance part="BAT" gate="2" x="38.1" y="40.64"/>
 <instance part="ANT" gate="ANT" x="38.1" y="93.98"/>
+<instance part="U$1" gate="G$1" x="83.82" y="78.74"/>
 </instances>
 <busses>
@@
 <net name="N$1" class="0">
 <segment>
-<pinref part="L1" gate="1" pin="2"/>
+<pinref part="L1" gate="G$1" pin="2"/>
 <pinref part="T2" gate="G$1" pin="C"/>
 <wire x1="50.8" y1="66.04" x2="50.8" y2="68.58" width="0.1524" layer="91"/>
@@
 <wire x1="66.04" y1="60.96" x2="60.96" y2="60.96" width="0.1524" layer="91"/>
 <pinref part="R2" gate="1" pin="1"/>
-<pinref part="L1" gate="1" pin="1"/>
+<pinref part="L1" gate="G$1" pin="1"/>
 <wire x1="60.96" y1="60.96" x2="55.88" y2="60.96" width="0.1524" layer="91"/>
 <wire x1="63.5" y1="88.9" x2="60.96" y2="88.9" width="0.1524" layer="91"/>
