File: eagle/OpAmp-Inverting-3Transistor-alt3.sch (EAGLE design)
At the start: 15 parts, among them J1 VCC_GNDPWR-R, T1 BC547, T2 BC547, T3 BC557

Commit message: ...
Parts:
- C3: value 3.3uF -> 3.3μF
- R1: value 100k -> 100kΩ
- R2: value 1M -> 1MΩ
- R3: value 75k -> 75kΩ
- R4: value 7.5k -> 7.5kΩ
- R5: value 4.7k -> 4.7kΩ
- R6: value 1k -> 1kΩ
Changed lines of the file:
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@@
 <part name="T2" library="t" deviceset="BC547" device="CBE" value="BC547"/>
 <part name="T3" library="t" deviceset="BC557" device="CBE" value="BC557"/>
-<part name="R1" library="r" deviceset="R-H" device="0202/10-V" value="100k"/>
-<part name="R2" library="r" deviceset="R-H" device="0202/10" value="1M"/>
-<part name="R3" library="r" deviceset="R-H" device="0202/7" value="75k"/>
-<part name="R4" library="r" deviceset="R" device="0202/7" value="7.5k"/>
-<part name="R5" library="r" deviceset="R" device="0202/7" value="4.7k"/>
-<part name="R6" library="r" deviceset="R" device="0202/10-V" value="1k"/>
+<part name="R1" library="r" deviceset="R-H" device="0202/10-V" value="100kΩ"/>
+<part name="R2" library="r" deviceset="R-H" device="0202/10" value="1MΩ"/>
+<part name="R3" library="r" deviceset="R-H" device="0202/7" value="75kΩ"/>
+<part name="R4" library="r" deviceset="R" device="0202/7" value="7.5kΩ"/>
+<part name="R5" library="r" deviceset="R" device="0202/7" value="4.7kΩ"/>
+<part name="R6" library="r" deviceset="R" device="0202/10-V" value="1kΩ"/>
 <part name="D1" library="d" deviceset="Z-DIODE" device="34Z2,5" value="Z=3.3V"/>
 <part name="C2" library="c" deviceset="C" device="050-020X044" value="33nF"/>
 <part name="IN" library="pad" deviceset="SPAD+-" device="-+" value="SPAD+--+"/>
 <part name="OUT" library="pad" deviceset="SPAD+-" device="+-"/>
-<part name="C3" library="c" deviceset="CPOL" device="E2,5-4/V" value="3.3uF"/>
+<part name="C3" library="c" deviceset="CPOL" device="E2,5-4/V" value="3.3μF"/>
 <part name="S2" library="pad" deviceset="GND" device=""/>
 <part name="S3" library="pad" deviceset="GND" device=""/>

Commit message: ...
Parts:
- R1: device r:R-H0202/10-V -> r:R-H0204/10-V
- R2: device r:R-H0202/10 -> r:R-H0204/10
- R3: device r:R-H0202/7 -> r:R-H0204/10
- R4, R5: device r:R0202/7 -> r:R0204/10
- R6: device r:R0202/10-V -> r:R0204/10-V
Changed lines of the file:
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@@
 <?xml version="1.0" encoding="utf-8"?>
 <!DOCTYPE eagle SYSTEM "eagle.dtd">
-<eagle version="7.6.0">
+<eagle version="7.2.0">
 <drawing>
 <settings>
@@
 <part name="T2" library="t" deviceset="BC547" device="CBE" value="BC547"/>
 <part name="T3" library="t" deviceset="BC557" device="CBE" value="BC557"/>
-<part name="R1" library="r" deviceset="R-H" device="0202/10-V" value="100kΩ"/>
-<part name="R2" library="r" deviceset="R-H" device="0202/10" value="1MΩ"/>
-<part name="R3" library="r" deviceset="R-H" device="0202/7" value="75kΩ"/>
-<part name="R4" library="r" deviceset="R" device="0202/7" value="7.5kΩ"/>
-<part name="R5" library="r" deviceset="R" device="0202/7" value="4.7kΩ"/>
-<part name="R6" library="r" deviceset="R" device="0202/10-V" value="1kΩ"/>
+<part name="R1" library="r" deviceset="R-H" device="0204/10-V" value="100kΩ"/>
+<part name="R2" library="r" deviceset="R-H" device="0204/10" value="1MΩ"/>
+<part name="R3" library="r" deviceset="R-H" device="0204/10" value="75kΩ"/>
+<part name="R4" library="r" deviceset="R" device="0204/10" value="7.5kΩ"/>
+<part name="R5" library="r" deviceset="R" device="0204/10" value="4.7kΩ"/>
+<part name="R6" library="r" deviceset="R" device="0204/10-V" value="1kΩ"/>
 <part name="D1" library="d" deviceset="Z-DIODE" device="34Z2,5" value="Z=3.3V"/>
 <part name="C2" library="c" deviceset="C" device="050-020X044" value="33nF"/>
