File: eagle/TBA820-Module-KOSMOS.brd (EAGLE design)
At the start: 17.8 x 27.9 mm, 10 parts, among them IC1 TBA820

Commit message: ...
Parts:
- C3: device c:C075-035X050 -> c:C050-020X044
- moved C3 1.31 mm to (10.2, 17.5)
Routing:
- net GND: track 35.6 -> 26.0 mm
- net VCC: track 25.4 -> 23.8 mm
- net N$3: track 24.1 -> 22.8 mm
- net N$7: track 14.0 -> 12.9 mm
- net N$5: track 14.0 -> 13.0 mm
- net N$2: track 11.2 -> 10.3 mm
Changed lines of the file:
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@@
 <setting verticaltext="up"/>
 </settings>
-<grid distance="0.025" unitdist="inch" unit="inch" style="lines" multiple="4" display="yes" altdistance="0.025" altunitdist="inch" altunit="inch"/>
+<grid distance="0.0125" unitdist="inch" unit="inch" style="lines" multiple="8" display="yes" altdistance="0.025" altunitdist="inch" altunit="inch"/>
 <layers>
 <layer number="1" name="Top" color="4" fill="1" visible="yes" active="yes"/>
@@
 </variantdefs>
 <classes>
-<class number="0" name="default" width="0" drill="0">
+<class number="0" name="default" width="0.8128" drill="0">
 </class>
 </classes>
@@
 <element name="C1" library="c" package="C050-020X044" value="330pF" x="12.7" y="35.56"/>
 <element name="C2" library="c" package="C075-035X050" value="100nF" x="11.43" y="33.02" rot="R180"/>
-<element name="C3" library="c" package="C075-035X050" value="220nF" x="11.43" y="17.78"/>
+<element name="C3" library="c" package="C050-020X044" value="220nF" x="10.16" y="17.4625"/>
 <element name="E" library="pad" package="SPAD" value="SPAD" x="5.08" y="15.24"/>
 <element name="GND" library="pad" package="SPAD" value="SPAD" x="17.78" y="15.24" rot="R180"/>
@@
 <contactref element="C1" pad="1"/>
 <contactref element="IC1" pad="1"/>
-<wire x1="7.62" y1="30.48" x2="5.842" y2="30.48" width="0.4064" layer="16"/>
-<wire x1="5.842" y1="30.48" x2="5.842" y2="35.56" width="0.4064" layer="16"/>
-<wire x1="5.842" y1="35.56" x2="10.16" y2="35.56" width="0.4064" layer="16"/>
+<wire x1="7.62" y1="30.48" x2="6.985" y2="30.48" width="0.8128" layer="16"/>
+<wire x1="6.985" y1="30.48" x2="5.5245" y2="31.75" width="0.8128" layer="16" curve="-83.974394"/>
+<wire x1="5.5245" y1="31.75" x2="5.5245" y2="34.0995" width="0.8128" layer="16"/>
+<wire x1="5.5245" y1="34.0995" x2="7.3025" y2="35.56" width="0.8128" layer="16" curve="-90"/>
+<wire x1="7.3025" y1="35.56" x2="7.112" y2="35.56" width="0.8128" layer="16"/>
+<wire x1="7.3025" y1="35.56" x2="10.16" y2="35.56" width="0.8128" layer="16"/>
 </signal>
 <signal name="N$3">
@@
 <contactref element="R1" pad="2"/>
 <contactref element="A" pad="1"/>
-<wire x1="18.415" y1="22.86" x2="18.415" y2="20.32" width="0.4064" layer="16"/>
-<wire x1="18.415" y1="20.32" x2="16.51" y2="20.32" width="0.4064" layer="16"/>
-<wire x1="15.24" y1="22.86" x2="18.415" y2="22.86" width="0.4064" layer="16"/>
-<wire x1="18.415" y1="25.4" x2="18.415" y2="35.56" width="0.4064" layer="16"/>
-<wire x1="18.415" y1="35.56" x2="15.24" y2="35.56" width="0.4064" layer="16"/>
-<wire x1="18.415" y1="22.86" x2="18.415" y2="25.4" width="0.4064" layer="16"/>
-<wire x1="18.415" y1="25.4" x2="17.78" y2="25.4" width="0.4064" layer="16"/>
+<wire x1="18.415" y1="22.86" x2="18.415" y2="21.59" width="0.8128" layer="16"/>
+<wire x1="18.415" y1="21.59" x2="17.4625" y2="20.32" width="0.8128" layer="16" curve="-73.739839"/>
+<wire x1="17.4625" y1="20.32" x2="16.51" y2="20.32" width="0.8128" layer="16"/>
+<wire x1="15.24" y1="22.86" x2="18.415" y2="22.86" width="0.8128" layer="16"/>
+<wire x1="18.415" y1="25.4" x2="18.415" y2="34.29" width="0.8128" layer="16"/>
+<wire x1="18.415" y1="34.29" x2="17.145" y2="35.56" width="0.8128" layer="16" curve="90"/>
+<wire x1="17.145" y1="35.56" x2="15.24" y2="35.56" width="0.8128" layer="16"/>
+<wire x1="18.415" y1="22.86" x2="18.415" y2="25.4" width="0.8128" layer="16"/>
+<wire x1="18.415" y1="25.4" x2="17.78" y2="25.4" width="0.8128" layer="16"/>
 </signal>
 <signal name="N$6">
 <contactref element="R1" pad="1"/>
 <contactref element="C3" pad="1"/>
-<wire x1="7.62" y1="17.78" x2="7.62" y2="20.32" width="0.4064" layer="16"/>
-<wire x1="7.62" y1="20.32" x2="6.35" y2="20.32" width="0.4064" layer="16"/>
+<wire x1="7.62" y1="17.4625" x2="7.62" y2="19.685" width="0.8128" layer="16"/>
+<wire x1="7.62" y1="19.685" x2="6.985" y2="20.32" width="0.8128" layer="16" curve="90"/>
+<wire x1="6.985" y1="20.32" x2="6.35" y2="20.32" width="0.8128" layer="16"/>
 </signal>
 <signal name="N$5">
 <contactref element="IC1" pad="3"/>
 <contactref element="E" pad="1"/>
-<wire x1="5.08" y1="15.24" x2="4.445" y2="15.24" width="0.4064" layer="16"/>
-<wire x1="4.445" y1="15.24" x2="4.445" y2="25.4" width="0.4064" layer="16"/>
-<wire x1="4.445" y1="25.4" x2="5.08" y2="25.4" width="0.4064" layer="16"/>
-<wire x1="5.08" y1="25.4" x2="7.62" y2="25.4" width="0.4064" layer="16"/>
+<wire x1="5.08" y1="15.24" x2="4.1275" y2="16.1925" width="0.8128" layer="16" curve="-90"/>
+<wire x1="4.1275" y1="16.1925" x2="4.1275" y2="23.8125" width="0.8128" layer="16"/>
+<wire x1="4.1275" y1="23.8125" x2="6.0325" y2="25.4" width="0.8128" layer="16" curve="-90"/>
+<wire x1="6.0325" y1="25.4" x2="7.62" y2="25.4" width="0.8128" layer="16"/>
 </signal>
 <signal name="N$7">
 <contactref element="IC1" pad="2"/>
 <contactref element="V" pad="1"/>
-<wire x1="7.62" y1="27.94" x2="5.08" y2="27.94" width="0.4064" layer="16"/>
-<wire x1="5.08" y1="27.94" x2="4.445" y2="27.94" width="0.4064" layer="16"/>
-<wire x1="4.445" y1="27.94" x2="4.445" y2="38.1" width="0.4064" layer="16"/>
-<wire x1="4.445" y1="38.1" x2="5.08" y2="38.1" width="0.4064" layer="16"/>
+<wire x1="7.62" y1="27.94" x2="6.35" y2="27.94" width="0.8128" layer="16"/>
+<wire x1="6.35" y1="27.94" x2="3.81" y2="30.48" width="0.8128" layer="16" curve="-90"/>
+<wire x1="3.81" y1="30.48" x2="3.81" y2="36.195" width="0.8128" layer="16"/>
+<wire x1="3.81" y1="36.195" x2="5.08" y2="38.1" width="0.8128" layer="16" curve="-67.380135"/>
 </signal>
 <signal name="GND">
@@
 <contactref element="GND" pad="1"/>
 <contactref element="C3" pad="2"/>
-<wire x1="7.62" y1="33.02" x2="10.16" y2="33.02" width="0.4064" layer="16"/>
-<wire x1="10.16" y1="33.02" x2="10.16" y2="22.86" width="0.4064" layer="16"/>
-<wire x1="10.16" y1="22.86" x2="10.16" y2="17.78" width="0.4064" layer="16"/>
-<wire x1="10.16" y1="17.78" x2="15.24" y2="17.78" width="0.4064" layer="16"/>
-<wire x1="7.62" y1="22.86" x2="10.16" y2="22.86" width="0.4064" layer="16"/>
-<wire x1="10.16" y1="17.78" x2="10.16" y2="15.24" width="0.4064" layer="16"/>
-<wire x1="10.16" y1="15.24" x2="17.78" y2="15.24" width="0.4064" layer="16"/>
+<wire x1="7.62" y1="33.02" x2="8.89" y2="33.02" width="0.8128" layer="16"/>
+<wire x1="8.89" y1="33.02" x2="10.16" y2="31.75" width="0.8128" layer="16" curve="-90"/>
+<wire x1="10.16" y1="31.75" x2="10.16" y2="22.86" width="0.8128" layer="16"/>
+<wire x1="17.78" y1="15.24" x2="12.7" y2="17.4625" width="0.8128" layer="16" curve="-22.339007"/>
+<wire x1="12.7" y1="17.4625" x2="10.16" y2="22.86" width="0.8128" layer="16" curve="-60"/>
+<wire x1="10.16" y1="22.86" x2="7.62" y2="22.86" width="0.8128" layer="16"/>
 </signal>
 <signal name="VCC">
@@
 <contactref element="C2" pad="1"/>
 <contactref element="VCC" pad="1"/>
-<wire x1="12.7" y1="27.94" x2="12.7" y2="33.02" width="0.4064" layer="16"/>
-<wire x1="15.24" y1="25.4" x2="12.7" y2="25.4" width="0.4064" layer="16"/>
-<wire x1="12.7" y1="25.4" x2="12.7" y2="27.94" width="0.4064" layer="16"/>
-<wire x1="12.7" y1="27.94" x2="15.24" y2="27.94" width="0.4064" layer="16"/>
-<wire x1="15.24" y1="33.02" x2="12.7" y2="33.02" width="0.4064" layer="16"/>
-<wire x1="12.7" y1="33.02" x2="12.7" y2="38.1" width="0.4064" layer="16"/>
-<wire x1="12.7" y1="38.1" x2="17.78" y2="38.1" width="0.4064" layer="16"/>
+<wire x1="12.7" y1="27.94" x2="12.7" y2="33.02" width="0.8128" layer="16"/>
+<wire x1="15.24" y1="25.4" x2="14.2875" y2="25.4" width="0.8128" layer="16"/>
+<wire x1="14.2875" y1="25.4" x2="12.7" y2="26.67" width="0.8128" layer="16" curve="-102.680383"/>
+<wire x1="12.7" y1="26.67" x2="12.7" y2="27.94" width="0.8128" layer="16"/>
+<wire x1="12.7" y1="27.94" x2="15.24" y2="27.94" width="0.8128" layer="16"/>
+<wire x1="15.24" y1="33.02" x2="12.7" y2="33.02" width="0.8128" layer="16"/>
+<wire x1="12.7" y1="33.02" x2="12.7" y2="36.83" width="0.8128" layer="16"/>
+<wire x1="12.7" y1="36.83" x2="13.97" y2="38.1" width="0.8128" layer="16" curve="-90"/>
+<wire x1="13.97" y1="38.1" x2="17.78" y2="38.1" width="0.8128" layer="16"/>
 </signal>
 </signals>
