File: eagle/Pink-Noise-Generator-Thomas-Henry.brd (EAGLE design)
At the start: 84.1 x 45.7 mm, 25 parts, among them IC1 TL072P, J1 SPAD+-+-, T1 BC547

Commit message: ...
Parts:
- C1: device c:E2,5-4 -> c:E2,5-5
Changed lines of the file:
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@@
 </autorouter>
 <elements>
-<element name="C1" library="c" package="E2,5-4" value="10µF" x="10.16" y="7.62"/>
+<element name="C1" library="c" package="E2,5-5" value="10µF" x="10.16" y="7.62"/>
 <element name="C10" library="c" package="C050-020X044/V" value="100nF" x="73.66" y="38.1"/>
 <element name="C11" library="c" package="C050-020X044/V" value="100nF" x="71.12" y="33.02"/>
