File: eagle/VCF-LM324-Stereo-LFO-PinHdr.brd (EAGLE design)
At the start: 63.5 x 66 mm, 50 parts, among them IC1 LM324, J1 A_IN, J2 A_OUT, J3 CONN-2P2P/H

Commit message: ...
Parts:
- moved R13 2.54 mm to (43.2, 26.7)
- moved R21 2.54 mm to (48.3, 27.9)
- moved R5 2.54 mm to (25.4, 26.7)
- moved R6 2.54 mm to (17.8, 27.9)
- moved R7 2.54 mm to (20.3, 33.0)
- moved C9 2.54 mm to (43.5, 17.8)
- moved LED2 2.54 mm to (16.5, 15.2)
- moved J3 2.54 mm to (15.2, 5.08)
- moved LED1 2.54 mm to (16.5, 10.2)
- moved R18 2.54 mm to (33.0, 7.62)
- moved R20 2.54 mm to (48.3, 7.62)
- moved R23 2.54 mm to (22.9, 10.2)
- moved TRI 2.54 mm to (20.3, 5.08)
- moved +5V 2.54 mm to (48.3, 35.6)
- moved C1 2.54 mm to (12.7, 36.8)
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Routing:
- net GND: track 201.6 -> 186.6 mm
- net N$9: track 25.0 -> 17.3 mm
- net N$5: track 57.2 -> 51.9 mm
- net VCC: track 74.1 -> 73.3 mm
- net N$12: track 69.6 -> 68.9 mm
Other:
- board size 63.5 x 66 mm -> 58.4 x 63.5 mm

Commit message: ...
Parts:
- moved C9 0.32 mm to (43.2, 17.8)
Routing:
- net GND: track 186.6 -> 182.2 mm
- net N$3: track 2.54 -> 5.08 mm
- net N$4: track 51.9 -> 50.4 mm
- net N$2: track 31.3 -> 30.0 mm
- net VCC: track 73.3 -> 72.0 mm
Other:
- board size 58.4 x 63.5 mm -> 58.4 x 61 mm
